File: projects/usb-dac-amplifier-rev-a/smartstand-usb-dac-amplifier-rev-a.brd (EAGLE design)
At the start: 174.7 x 136 mm, 224 parts, among them J1 PJ-002A, J2 292304-1, J3 NRJ6HH, J4 PJRAN2XIU01AUX, J5 T1M-5POS, U1 XUF208-256-TQ64, U10 TPS3702, U11 PCM5102A, U12 SZNUD3124, U13 NJM2068M, U14 NJM4556AM, U15 NJM4556AM, U16 TS5A3159DBV, U17 SN74LVC3G34, U2 TPD4E02B04, U3 TPS563200DDC, U4 TPS7A8300RGW, U5 TPS563200DDC, U6 TPS7A8300RGW, U7 TPS7A8300RGW, U8 TPS7A4701RGW, U9 TPS7A3301RGW, X1 24MHz, X2 22.5792MHz, X3 24.576MHz

Commit message: Ensure all resistors and capacitors in audio path are spec'd correctly.
Basically just went through and made sure we had 0.1% tolerance on the
resistors, with the exception of 1% on the outout resistors because
percision ones (aka current sense resistors ) are $xx.xx, and made sure
that our capacitors are C0G/NP0.  I switched to film capacitors for the
DC blocking input capacitors on the output stage because values that
large for C0G/NP0 ceramics don't exist on Mouser.

Also added ESD protection to the headphone output and line output,
specifically using the TPD2E007, which is specified for AC signals like
ours, and won't activate with our -/+10V rails.
Parts:
- added U18, U19: TPD2E007DCK, texas-instruments:R-PDSO-G3
- C101, C102: device rcl:C0603 -> rcl:KEMET-5MM-6.0-7.2
- C83, C84: value 2.2nF -> 2.2nF, C0G
- C91, C92, C93, C94: value 220pF -> 220pF, C0G
- R22, R23: value 470 -> 470, 0.1%
- R24, R28: value 243 -> 243, 0.1%
- R25, R29, R46: value 10K -> 10K, 0.1%
- R26, R30: value 1.5K -> 1.5K, 0.1%
- R31, R32: value 243 -> 243, 0.1%; device rcl:R0603 -> rcl:R0402
- R33, R34: value 715 -> 715, 0.1%; device rcl:R0603 -> rcl:R0402
- R36, R39: value 40.2K, 1% -> 40.2K, 0.1%
- moved C102 9.87 mm to (34.0, 25.3)
- moved C101 8.51 mm to (26.0, 25.3)
- moved R39 1.20 mm to (38.7, 34.8), turned to 0 degrees
- moved R36 1.20 mm to (25.5, 34.9), turned to 0 degrees
- moved C83 0.51 mm to (-8.38, -16.5)
- moved C84 0.51 mm to (-8.38, -20.1)
- moved R22 0.51 mm to (-8.38, -17.7)
- moved R23 0.51 mm to (-8.38, -18.9)
Connections:
- net ADJUSTED_LEFT: now also C101.P$1; no longer C101.1
- net ADJUSTED_RIGHT: now also C102.P$1; no longer C102.1
- net AGND: now also U18.3, U19.3
- net LINE_OUT_LEFT: now also U19.2
- net LINE_OUT_RIGHT: now also U19.1
- net N$19: now also C101.P$2; no longer C101.2
- net N$20: now also C102.P$2; no longer C102.2
- net N$27: now also U18.2
- net N$29: now also U18.1
Routing:
- net ADJUSTED_LEFT: track 123.4 -> 107.5 mm
- net ADJUSTED_RIGHT: track 127.1 -> 116.1 mm
- net N$20: track 19.7 -> 27.8 mm
- net N$19: track 19.7 -> 24.5 mm
- net LINE_OUT_LEFT: track 146.2 -> 150.4 mm
- net N$29: track 42.1 -> 45.1 mm
- net N$79: track 86.6 -> 83.9 mm
- net AGND: track 103.9 -> 106.2 mm, vias 141 -> 143
- net RAW_RIGHT: track 17.5 -> 17.0 mm
- net RAW_LEFT: track 8.92 -> 8.41 mm
- net N$6: track 8.15 -> 8.65 mm
- net N$5: track 8.16 -> 8.67 mm

Commit message: Adding part numbers for major components.
Parts:
- J4: value PJRAN2XIU01AUX -> PJRAN2X1U01AUX
- U17: value SN74LVC3G34 -> SN74LVC3G34DCU; device texas-instruments:R-PDSO-G8 -> texas-instruments:R-PDSO-G8-DCU
- U2: value TPD4E02B04 -> TPD4E02B04DQA
