File: projects/usb-dac-amplifier-rev-a/smartstand-usb-dac-amplifier-rev-a.brd (EAGLE design)
At the start: 174.7 x 136 mm, 226 parts, among them J1 PJ-002A, J2 292304-1, J3 NRJ6HH, J4 PJRAN2X1U01AUX, J5 T1M-5POS, U1 XUF208-256-TQ64, U10 TPS3702, U11 PCM5102A, U12 SZNUD3124, U13 NJM2068M, U14 NJM4556AM, U15 NJM4556AM, U16 TS5A3159DBV, U17 SN74LVC3G34DCU, U18 TPD2E007DCK, U19 TPD2E007DCK, U2 TPD4E02B04DQA, U3 TPS563200DDC, U4 TPS7A8300RGW, U5 TPS563200DDC, U6 TPS7A8300RGW, U7 TPS7A8300RGW, U8 TPS7A4701RGW, U9 TPS7A3301RGW, X1 24MHz, X2 22.5792MHz, X3 24.576MHz

Commit message: Minor board layout tweaks.
Adjusted how we route the USB signals to better take advantage of the
type B connector, which now lets us avoid a layer transition.  We're
about 37mils difference between the pair lengths which is well within
bounds of the 100ps skew allowed by the USB specification.

Also, I mistakenly forgot to route power into the pigtail between the
main board and the headphone detection daughterboard, which is now
rectified.  We're sending it DVDD (3V3) so that it needs no regulator of
its own.  We'll need to make sure that we do have a lot of bulk
capacitance since the pigtail will be 8-12 inches long, and the
measurement current can be large, and thus high di/dt, with frequent
measurements.
Parts:
- moved C7 3.14 mm to (72.1, -28.8)
- moved U2 3.07 mm to (72.6, -31.4)
Connections:
- net AGND: no longer J5.3
- net DVDD: now also J5.3
- net USB_D_N: now also U2.P$4, U2.P$7; no longer U2.P$2, U2.P$9
- net USB_D_P: now also U2.P$2, U2.P$9; no longer U2.P$4, U2.P$7
Routing:
- net USB_D_P: track 64.1 -> 69.4 mm, vias 2 -> 0
- net USB_D_N: track 64.2 -> 68.5 mm, vias 2 -> 0
- net USB_VBUS: track 73.8 -> 76.2 mm
- net DVDD: track 284.5 -> 286.3 mm, vias 27 -> 28
- net AGND: track 106.2 -> 106.4 mm, vias 143 -> 144
- removed copper zone on layer 1, net N$78

Commit message: Adjust the I2C pinout on the daughterboard connector.
This will let us have cleaner routing on the small daughterboard which
houses the proximity sensor.
Connections:
- net DVDD: now also J5.2; no longer J5.3
- net I2C_SCL: now also J5.4, R18.1; no longer J5.2, R17.1
- net I2C_SDA: now also J5.3, R17.1; no longer J5.4, R18.1
Routing:
- net I2C_SDA: track 33.1 -> 35.5 mm
- net I2C_SCL: track 34.6 -> 33.0 mm
Changed lines of the file:
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@@
 <class number="0" name="default" width="0.1524" drill="0.254">
 </class>
-<class number="1" name="USB" width="0.3048" drill="0.254">
+<class number="1" name="USB" width="0.2794" drill="0.254">
 </class>
 </classes>
-<designrules name="OSHPark-4layer">
+<designrules name="OSHPark-4Layer">
 <description language="de">&lt;b&gt;EAGLE Design Rules&lt;/b&gt;
 &lt;p&gt;
@@
 <wire x1="42.799" y1="-20.193" x2="42.799" y2="-12.7" width="1.016" layer="1"/>
 <wire x1="37.084" y1="-6.985" x2="36.957" y2="-6.858" width="1.016" layer="1"/>
-<wire x1="54.328" y1="-17.78" x2="54.328" y2="-16.919" width="0.1524" layer="1"/>
-<via x="54.328" y="-16.919" extent="1-16" drill="0.254"/>
 <via x="43.942" y="-20.066" extent="1-16" drill="0.254"/>
 <wire x1="43.942" y1="-20.066" x2="42.926" y2="-20.066" width="0.4064" layer="1"/>
@@
 <wire x1="45.085" y1="-21.209" x2="43.942" y2="-20.066" width="0.4064" layer="16"/>
 <wire x1="51.308" y1="-16.891" x2="51.336" y2="-16.863" width="0.254" layer="16"/>
-<wire x1="52.832" y1="-16.863" x2="54.272" y2="-16.863" width="0.254" layer="16"/>
-<wire x1="54.272" y1="-16.863" x2="54.328" y2="-16.919" width="0.1524" layer="16"/>
+<wire x1="52.832" y1="-16.863" x2="54.272" y2="-16.863" width="0.4064" layer="16"/>
 <wire x1="73.152" y1="-10.884" x2="73.152" y2="-10.16" width="0.1524" layer="1"/>
 <wire x1="73.152" y1="-10.16" x2="72.898" y2="-9.906" width="0.1524" layer="1"/>
@@
 <vertex x="36.449" y="-7.62"/>
 </polygon>
-<contactref element="J5" pad="3"/>
-<wire x1="52.832" y1="-15.354" x2="52.832" y2="-16.863" width="0.254" layer="1"/>
 <via x="52.832" y="-16.863" extent="1-16" drill="0.254"/>
 <wire x1="52.832" y1="-16.863" x2="51.336" y2="-16.863" width="0.254" layer="16"/>
@@
 <wire x1="27.975" y1="-2.806" x2="26.658" y2="-2.806" width="0.2794" layer="1"/>
 <wire x1="26.658" y1="-2.806" x2="26.543" y2="-2.921" width="0.2794" layer="1"/>
+<contactref element="J5" pad="2"/>
+<via x="54.272" y="-16.863" extent="1-16" drill="0.254"/>
+<wire x1="54.272" y1="-16.863" x2="54.272" y2="-17.724" width="0.1524" layer="1"/>
+<wire x1="54.272" y1="-17.724" x2="54.328" y2="-17.78" width="0.1524" layer="1"/>
+<wire x1="53.832" y1="-15.354" x2="53.832" y2="-16.423" width="0.4064" layer="1"/>
+<wire x1="53.832" y1="-16.423" x2="54.272" y2="-16.863" width="0.4064" layer="1"/>
 </signal>
 <signal name="+1V4">
@@
 <signal name="I2C_SDA">
 <contactref element="U1" pad="P$16"/>
-<contactref element="R18" pad="1"/>
-<contactref element="J5" pad="4"/>
-<wire x1="51.816" y1="-15.37" x2="51.832" y2="-15.354" width="0.1524" layer="1"/>
-<wire x1="52.324" y1="-17.808" x2="52.296" y2="-17.78" width="0.1524" layer="1"/>
-<wire x1="52.324" y1="-17.752" x2="52.296" y2="-17.78" width="0.1524" layer="1"/>
-<wire x1="52.296" y1="-17.78" x2="52.296" y2="-18.824" width="0.1524" layer="1"/>
-<wire x1="52.296" y1="-18.824" x2="51.816" y2="-19.304" width="0.1524" layer="1"/>
-<wire x1="47.752" y1="-18.288" x2="47.752" y2="-10.795" width="0.1524" layer="1"/>
-<wire x1="47.752" y1="-10.795" x2="46.99" y2="-10.033" width="0.1524" layer="1"/>
-<wire x1="46.99" y1="-10.033" x2="44.196" y2="-10.033" width="0.1524" layer="1"/>
 <via x="44.196" y="-10.033" extent="1-16" drill="0.254"/>
 <wire x1="37.405" y1="-9.236" x2="37.405" y2="-9.846" width="0.1524" layer="1"/>
@@
 <via x="38.735" y="-13.716" extent="1-16" drill="0.254"/>
 <wire x1="40.513" y1="-13.716" x2="44.196" y2="-10.033" width="0.1524" layer="16"/>
-<wire x1="52.296" y1="-17.78" x2="52.296" y2="-16.99" width="0.1524" layer="1"/>
-<wire x1="52.296" y1="-16.99" x2="51.832" y2="-16.526" width="0.1524" layer="1"/>
-<wire x1="51.832" y1="-15.354" x2="51.832" y2="-16.526" width="0.1524" layer="1"/>
 <wire x1="38.735" y1="-13.716" x2="40.513" y2="-13.716" width="0.1524" layer="16"/>
 <wire x1="38.354" y1="-10.16" x2="39.243" y2="-11.049" width="0.1524" layer="1"/>
 <wire x1="39.243" y1="-11.049" x2="39.243" y2="-11.811" width="0.1524" layer="1"/>
 <wire x1="39.243" y1="-11.811" x2="38.735" y2="-12.319" width="0.1524" layer="1"/>
-<wire x1="51.816" y1="-19.304" x2="48.768" y2="-19.304" width="0.1524" layer="1"/>
-<wire x1="48.768" y1="-19.304" x2="47.752" y2="-18.288" width="0.1524" layer="1"/>
+<contactref element="J5" pad="3"/>
+<contactref element="R17" pad="1"/>
+<wire x1="52.832" y1="-15.354" x2="52.832" y2="-15.875" width="0.1524" layer="1"/>
+<wire x1="52.832" y1="-15.875" x2="53.34" y2="-16.383" width="0.1524" layer="1"/>
+<wire x1="53.34" y1="-16.383" x2="53.34" y2="-17.752" width="0.1524" layer="1"/>
+<wire x1="53.34" y1="-17.752" x2="53.368" y2="-17.78" width="0.1524" layer="1"/>
+<wire x1="44.196" y1="-10.033" x2="43.561" y2="-10.668" width="0.1524" layer="1"/>
+<wire x1="43.561" y1="-10.668" x2="43.561" y2="-11.43" width="0.1524" layer="1"/>
+<wire x1="43.561" y1="-11.43" x2="44.196" y2="-12.065" width="0.1524" layer="1"/>
+<wire x1="44.196" y1="-12.065" x2="46.228" y2="-12.065" width="0.1524" layer="1"/>
+<wire x1="46.228" y1="-12.065" x2="46.99" y2="-12.827" width="0.1524" layer="1"/>
+<wire x1="46.99" y1="-12.827" x2="46.99" y2="-18.669" width="0.1524" layer="1"/>
+<wire x1="46.99" y1="-18.669" x2="48.26" y2="-19.939" width="0.1524" layer="1"/>
+<wire x1="48.26" y1="-19.939" x2="52.451" y2="-19.939" width="0.1524" layer="1"/>
+<wire x1="52.451" y1="-19.939" x2="53.368" y2="-19.022" width="0.1524" layer="1"/>
+<wire x1="53.368" y1="-17.78" x2="53.368" y2="-19.022" width="0.1524" layer="1"/>
 </signal>
 <signal name="I2C_SCL">
 <contactref element="U1" pad="P$14"/>
-<contactref element="R17" pad="1"/>
-<contactref element="J5" pad="2"/>
-<wire x1="53.848" y1="-15.37" x2="53.832" y2="-15.354" width="0.1524" layer="1"/>
-<wire x1="53.34" y1="-17.752" x2="53.368" y2="-17.78" width="0.1524" layer="1"/>
-<wire x1="53.368" y1="-17.78" x2="53.368" y2="-18.387" width="0.1524" layer="1"/>
-<wire x1="53.368" y1="-18.387" x2="52.07" y2="-19.685" width="0.1524" layer="1"/>
-<wire x1="52.07" y1="-19.685" x2="48.641" y2="-19.685" width="0.1524" layer="1"/>
-<wire x1="47.371" y1="-18.415" x2="47.371" y2="-11.303" width="0.1524" layer="1"/>
-<wire x1="47.371" y1="-11.303" x2="46.99" y2="-10.922" width="0.1524" layer="1"/>
-<wire x1="46.99" y1="-10.922" x2="44.069" y2="-10.922" width="0.1524" layer="1"/>
 <via x="44.069" y="-10.922" extent="1-16" drill="0.254"/>
 <wire x1="36.405" y1="-9.236" x2="36.405" y2="-10.37" width="0.1524" layer="1"/>
@@
 <via x="38.1" y="-14.351" extent="1-16" drill="0.254"/>
 <wire x1="40.64" y1="-14.351" x2="44.069" y2="-10.922" width="0.1524" layer="16"/>
-<wire x1="53.368" y1="-17.78" x2="53.368" y2="-16.99" width="0.1524" layer="1"/>
-<wire x1="53.368" y1="-16.99" x2="53.832" y2="-16.526" width="0.1524" layer="1"/>
-<wire x1="53.832" y1="-15.354" x2="53.832" y2="-16.526" width="0.1524" layer="1"/>
 <wire x1="38.1" y1="-14.351" x2="40.64" y2="-14.351" width="0.1524" layer="16"/>
-<wire x1="48.641" y1="-19.685" x2="47.371" y2="-18.415" width="0.1524" layer="1"/>
+<contactref element="J5" pad="4"/>
+<contactref element="R18" pad="1"/>
+<wire x1="51.832" y1="-15.354" x2="51.832" y2="-16.399" width="0.1524" layer="1"/>
+<wire x1="51.832" y1="-16.399" x2="52.296" y2="-16.863" width="0.1524" layer="1"/>
+<wire x1="52.296" y1="-17.78" x2="52.296" y2="-16.863" width="0.1524" layer="1"/>
+<wire x1="44.069" y1="-10.922" x2="45.847" y2="-10.922" width="0.1524" layer="1"/>
+<wire x1="45.847" y1="-10.922" x2="47.498" y2="-12.573" width="0.1524" layer="1"/>
+<wire x1="47.498" y1="-12.573" x2="47.498" y2="-18.542" width="0.1524" layer="1"/>
+<wire x1="47.498" y1="-18.542" x2="48.387" y2="-19.431" width="0.1524" layer="1"/>
+<wire x1="48.387" y1="-19.431" x2="51.943" y2="-19.431" width="0.1524" layer="1"/>
+<wire x1="52.296" y1="-17.78" x2="52.296" y2="-19.078" width="0.1524" layer="1"/>
+<wire x1="52.296" y1="-19.078" x2="51.943" y2="-19.431" width="0.1524" layer="1"/>
 </signal>
 <signal name="JACK_ENABLE">

Commit message: Add fiducials and fix ERC/DRC errors.
Parts:
- added U$1, U$10, U$11, U$12, U$13, U$2, U$3, U$4, U$5, U$6, U$7, U$8, U$9: FIDUCIAL-1MM, fiducials:FIDUCIAL_1MM
Connections:
- removed net +3V3: U17.8
- net DVDD: now also U17.8
Changed lines of the file:
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@@
 <layer number="29" name="tStop" color="7" fill="3" visible="no" active="yes"/>
 <layer number="30" name="bStop" color="7" fill="6" visible="no" active="yes"/>
-<layer number="31" name="tCream" color="7" fill="4" visible="yes" active="yes"/>
-<layer number="32" name="bCream" color="7" fill="5" visible="yes" active="yes"/>
+<layer number="31" name="tCream" color="7" fill="4" visible="no" active="yes"/>
+<layer number="32" name="bCream" color="7" fill="5" visible="no" active="yes"/>
 <layer number="33" name="tFinish" color="6" fill="3" visible="no" active="yes"/>
 <layer number="34" name="bFinish" color="6" fill="6" visible="no" active="yes"/>
@@
 <layer number="44" name="Drills" color="7" fill="1" visible="no" active="yes"/>
 <layer number="45" name="Holes" color="7" fill="1" visible="yes" active="yes"/>
-<layer number="46" name="Milling" color="3" fill="1" visible="no" active="yes"/>
+<layer number="46" name="Milling" color="3" fill="1" visible="yes" active="yes"/>
 <layer number="47" name="Measures" color="7" fill="1" visible="yes" active="yes"/>
 <layer number="48" name="Document" color="7" fill="1" visible="yes" active="yes"/>
@@
 </classes>
 <designrules name="OSHPark-4Layer">
-<description language="de">&lt;b&gt;EAGLE Design Rules&lt;/b&gt;
-&lt;p&gt;
-Die Standard-Design-Rules sind so gewählt, dass sie für
-die meisten Anwendungen passen. Sollte ihre Platine
-besondere Anforderungen haben, treffen Sie die erforderlichen
-Einstellungen hier und speichern die Design Rules unter
-einem neuen Namen ab.</description>
-<description language="en">&lt;b&gt;Laen's PCB Order Design Rules&lt;/b&gt;
+<description language="en">&lt;b&gt;OSH Park Design Rules (4 layers)&lt;/b&gt;
 &lt;p&gt;
 Please make sure your boards conform to these design rules.</description>
@@
 <param name="slThermalIsolate" value="10mil"/>
 <param name="slThermalsForVias" value="0"/>
-<param name="dpMaxLengthDifference" value="10mm"/>
+<param name="dpMaxLengthDifference" value="1mm"/>
 <param name="dpGapFactor" value="2.5"/>
 <param name="checkGrid" value="0"/>
@@
 <attribute name="PN" value="TPD2E007DCKR" x="75.819" y="8.89" size="1.778" layer="27" rot="R270" display="off"/>
 </element>
+<element name="U$1" library="fiducials" package="FIDUCIAL_1MM" value="FIDUCIAL-1MM" x="-76.327" y="0"/>
+<element name="U$2" library="fiducials" package="FIDUCIAL_1MM" value="FIDUCIAL-1MM" x="22.86" y="-13.208"/>
+<element name="U$3" library="fiducials" package="FIDUCIAL_1MM" value="FIDUCIAL-1MM" x="42.926" y="5.334"/>
+<element name="U$4" library="fiducials" package="FIDUCIAL_1MM" value="FIDUCIAL-1MM" x="14.224" y="56.388"/>
+<element name="U$5" library="fiducials" package="FIDUCIAL_1MM" value="FIDUCIAL-1MM" x="13.716" y="-57.15"/>
+<element name="U$6" library="fiducials" package="FIDUCIAL_1MM" value="FIDUCIAL-1MM" x="36.576" y="17.907"/>
+<element name="U$7" library="fiducials" package="FIDUCIAL_1MM" value="FIDUCIAL-1MM" x="66.421" y="-40.767"/>
+<element name="U$8" library="fiducials" package="FIDUCIAL_1MM" value="FIDUCIAL-1MM" x="65.151" y="29.972"/>
+<element name="U$9" library="fiducials" package="FIDUCIAL_1MM" value="FIDUCIAL-1MM" x="-7.747" y="-22.352"/>
+<element name="U$10" library="fiducials" package="FIDUCIAL_1MM" value="FIDUCIAL-1MM" x="13.208" y="-12.192"/>
+<element name="U$11" library="fiducials" package="FIDUCIAL_1MM" value="FIDUCIAL-1MM" x="22.86" y="-39.497"/>
+<element name="U$12" library="fiducials" package="FIDUCIAL_1MM" value="FIDUCIAL-1MM" x="8.128" y="-30.607"/>
+<element name="U$13" library="fiducials" package="FIDUCIAL_1MM" value="FIDUCIAL-1MM" x="58.42" y="-27.559"/>
 </elements>
 <signals>
@@
 <wire x1="53.832" y1="-15.354" x2="53.832" y2="-16.423" width="0.4064" layer="1"/>
 <wire x1="53.832" y1="-16.423" x2="54.272" y2="-16.863" width="0.4064" layer="1"/>
+<contactref element="U17" pad="8"/>
+<wire x1="70.104" y1="-9.271" x2="61.734" y2="-11.658" width="0" layer="19" extent="1-1"/>
 </signal>
 <signal name="+1V4">
@@
 <signal name="AUDIO_STREAMING">
 <contactref element="U1" pad="P$17"/>
-<contactref element="U17" pad="3"/>
 <wire x1="39.335" y1="-7.306" x2="40.707" y2="-7.306" width="0.1524" layer="1"/>
 <wire x1="40.707" y1="-7.306" x2="40.894" y2="-7.493" width="0.1524" layer="1"/>
@@
 <wire x1="62.484" y1="-13.208" x2="62.738" y2="-13.462" width="0.1524" layer="1"/>
 <wire x1="62.738" y1="-13.462" x2="62.738" y2="-14.754" width="0.1524" layer="1"/>
-<wire x1="62.738" y1="-14.754" x2="62.734" y2="-14.758" width="0.1524" layer="1"/>
+<contactref element="U17" pad="3"/>
+<wire x1="62.734" y1="-14.758" x2="62.738" y2="-14.754" width="0.1524" layer="1"/>
 </signal>
 <signal name="USB_CONNECTED">
@@
 <wire x1="64.897" y1="-12.484" x2="64.897" y2="-14.125" width="0.2032" layer="1"/>
 </signal>
-<signal name="+3V3">
-<contactref element="U17" pad="8"/>
-</signal>
 <signal name="N$39">

Commit message: Switch everything to vector fonts and add LEDs for knob illumination.
We added LEDs around the volume control potentiometer so that we could
get an underlighting effect on the volume knob.  The base now has
corresponding holes inside the support structure/cavity that the volume
knob sits around, and since we engineered it so that the knob has a
small gap from the base, the new holes added will allow light to escape
all the way out, and under the volume knob, providing a soft white glow
when powered up.

We also switched all text on the board layout to be vector, to better
represent what the actual board will look like.
Parts:
- added D10, D11, D12, D13, D14, D9: CLM3C, cree:PLCC-2
- added R27, R44: 150, passives:R1206
Connections:
- new net N$62: D10.ANODE, D9.CATHODE
- new net N$78: D10.CATHODE, D11.ANODE
- new net N$80: D11.CATHODE, R27.2
- new net N$81: D12.CATHODE, D13.ANODE
- new net N$82: D13.CATHODE, D14.ANODE
- new net N$83: D14.CATHODE, R44.2
- net +12V: now also D12.ANODE, D9.ANODE
- net AGND: now also R27.1, R44.1
Routing:
- net N$64: track 207.0 -> 188.5 mm, vias 1 -> 3
- net N$78: track 0.00 -> 13.9 mm
- net N$81: track 0.00 -> 12.8 mm
- net N$62: track 0.00 -> 12.8 mm
- net N$82: track 0.00 -> 12.2 mm
- net DVDD: track 286.5 -> 295.8 mm, vias 28 -> 30
- net +12V: track 9.52 -> 13.3 mm, vias 49 -> 51
- net AGND: track 106.4 -> 110.0 mm, vias 144 -> 146
- net N$80: track 0.00 -> 3.00 mm
- net N$83: track 0.00 -> 2.87 mm
- net V+: track 172.1 -> 173.8 mm
- net V-: track 192.8 -> 194.4 mm
- net JACK_DETECT: track 8.44 -> 9.26 mm
