File: projects/usb-dac-amplifier-rev-a/smartstand-usb-dac-amplifier-rev-a.brd (EAGLE design)
At the start: 174.7 x 136 mm, 247 parts, among them J1 PJ-002A, J2 292304-1, J3 NRJ6HH, J4 PJRAN2X1U01AUX, J5 T1M-5POS, U1 XUF208-256-TQ64, U10 TPS3702, U11 PCM5102A, U12 SZNUD3124, U13 NJM2068M, U14 NJM4556AM, U15 NJM4556AM, U16 TS5A3159DBV, U17 SN74LVC3G34DCU, U18 TPD2E007DCK, U19 TPD2E007DCK, U2 TPD4E02B04DQA, U3 TPS563200DDC, U4 TPS7A8300RGW, U5 TPS563200DDC, U6 TPS7A8300RGW, U7 TPS7A8300RGW, U8 TPS7A4701RGW, U9 TPS7A3301RGW, X1 24MHz, X2 22.5792MHz, X3 24.576MHz

Commit message: Adjust power jack footprint and placement.
After getting the test boards back, the PTH fitment is super loose, and
because of that, it's hard to tell if things are positioned correctly.

I went and back took real measurements of the pins, cross-referenced
with what the datasheet says, and ran the numbers again using the IPC
specification for the tightest fit.

I also adjusted the footprint to better account for the centerline of
the part.  Now that the origin of the part is better situated, I
positioned it such that it should yield the optimal board extension of
1mm, letting it sit flush against the enclosure when installed.
Parts:
- moved J1 4.70 mm to (84.0, -49.5)
Changed lines of the file:
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@@
 <attribute name="VALUE" x="77.089" y="-52.07" size="1.27" layer="27" rot="R180"/>
 </element>
-<element name="J1" library="cui" package="PJ-002A" value="PJ-002A" x="83.82" y="-44.831" smashed="yes">
-<attribute name="PN" value="PJ-002A" x="83.82" y="-44.831" size="1.778" layer="27" display="off"/>
-<attribute name="VALUE" x="78.74" y="-42.545" size="1.27" layer="27"/>
-<attribute name="NAME" x="78.613" y="-42.926" size="1.27" layer="25" font="vector" ratio="12"/>
+<element name="J1" library="cui" package="PJ-002A" value="PJ-002A" x="83.9978" y="-49.53" smashed="yes">
+<attribute name="PN" value="PJ-002A" x="83.9978" y="-49.53" size="1.778" layer="27" display="off"/>
+<attribute name="VALUE" x="78.9178" y="-47.244" size="1.27" layer="27"/>
+<attribute name="NAME" x="79.1718" y="-42.799" size="1.27" layer="25" font="vector" ratio="12"/>
 </element>
 <element name="J3" library="neutrik" package="NRJ6HH" value="NRJ6HH" x="77.724" y="46.609" smashed="yes">

Commit message: Adjust RCA jack placement.
After measuring with the test boards, we had about 1mm worth of distance
from the front face of the RCA jacks to the edge of the board.

Now the jack is shifted over to sit flush with the board edge, exposing
that extra 1mm outside of the enclosure.  This gets us to a more
comfortable 6mm of exposed jack, for better plug seating.
Parts:
- moved J4 1.09 mm to (89.7, 16.5)
Routing:
- net LINE_OUT_RIGHT: track 131.3 -> 132.4 mm
- net LINE_OUT_LEFT: track 150.4 -> 151.5 mm
Changed lines of the file:
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@@
 <attribute name="VALUE" x="-28.321" y="17.907" size="1.27" layer="27"/>
 </element>
-<element name="J4" library="switchcraft" package="PJRAN2X1U" value="PJRAN2X1U01AUX" x="88.646" y="16.51" smashed="yes" rot="R90">
-<attribute name="VALUE" x="78.646" y="0.51" size="1.27" layer="27" rot="R90"/>
-<attribute name="NAME" x="80.202" y="1.78" size="1.27" layer="25" font="vector" ratio="12" rot="R90"/>
-<attribute name="PN" value="PJRAN2X1U01AUX" x="88.646" y="16.51" size="1.778" layer="27" rot="R90" display="off"/>
+<element name="J4" library="switchcraft" package="PJRAN2X1U" value="PJRAN2X1U01AUX" x="89.7382" y="16.51" smashed="yes" rot="R90">
+<attribute name="VALUE" x="79.7382" y="0.51" size="1.27" layer="27" rot="R90"/>
+<attribute name="NAME" x="81.2942" y="1.78" size="1.27" layer="25" font="vector" ratio="12" rot="R90"/>
+<attribute name="PN" value="PJRAN2X1U01AUX" x="89.7382" y="16.51" size="1.778" layer="27" rot="R90" display="off"/>
 </element>
 <element name="L1" library="rcl" package="TDK-VLP8040" value="2.2uH" x="20.066" y="-46.863" smashed="yes" rot="R270">
@@
 <wire x1="80.264" y1="11.811" x2="80.264" y2="18.669" width="0.1524" layer="1"/>
 <wire x1="80.264" y1="18.669" x2="81.855" y2="20.26" width="0.1524" layer="1"/>
-<wire x1="84.946" y1="20.26" x2="81.855" y2="20.26" width="0.1524" layer="1"/>
+<wire x1="86.0382" y1="20.26" x2="81.855" y2="20.26" width="0.1524" layer="1"/>
 </signal>
 <signal name="LINE_OUT_RIGHT">
@@
 <wire x1="76.744" y1="8.24" x2="76.744" y2="8.164" width="0.1524" layer="1"/>
 <wire x1="76.744" y1="8.164" x2="76.708" y2="8.128" width="0.1524" layer="1"/>
-<wire x1="76.708" y1="8.128" x2="82.078" y2="8.128" width="0.1524" layer="1"/>
-<wire x1="82.078" y1="8.128" x2="84.946" y2="5.26" width="0.1524" layer="1"/>
+<wire x1="76.708" y1="8.128" x2="83.1702" y2="8.128" width="0.1524" layer="1"/>
+<wire x1="83.1702" y1="8.128" x2="86.0382" y2="5.26" width="0.1524" layer="1"/>
 </signal>
 <signal name="N$23">
