File: projects/usb-dac-amplifier-rev-a/smartstand-usb-dac-amplifier-rev-a.brd (EAGLE design)
At the start: 174.7 x 136 mm, 247 parts, among them J1 PJ-002A, J2 292304-1, J3 NRJ6HH, J4 PJRAN2X1U01AUX, J5 T1M-5POS, U1 XUF208-256-TQ64, U10 TPS3702, U11 PCM5102A, U12 SZNUD3124, U13 NJM2068M, U14 NJM4556AM, U15 NJM4556AM, U16 TS5A3159DBV, U17 SN74LVC3G34DCU, U18 TPD2E007DCK, U19 TPD2E007DCK, U2 TPD4E02B04DQA, U3 TPS563200DDC, U4 TPS7A8300RGW, U5 TPS563200DDC, U6 TPS7A8300RGW, U7 TPS7A8300RGW, U8 TPS7A4701RGW, U9 TPS7A3301RGW, X1 24MHz, X2 22.5792MHz, X3 24.576MHz

Commit message: Tightening up fiducial to processor.
Parts:
- moved U$2 1.40 mm to (24.3, -13.2)
- moved R19 0.81 mm to (31.4, -14.9)
- moved R20 0.81 mm to (31.4, -16.0)
Routing:
- net I2S_MCLK: track 34.0 -> 31.7 mm
- net I2S_MCLK_SEL: track 30.0 -> 31.7 mm
- net AUDIO_ENABLE: track 48.2 -> 49.1 mm
- net LINK_UP1: track 73.3 -> 74.1 mm

Commit message: Clean up some routing of the relay control lines.
Routing:
- net N$64: track 188.5 -> 175.4 mm
- net AGND: track 110.2 -> 111.0 mm
- net LINE_OUT_SEL: track 171.2 -> 170.8 mm, vias 6 -> 4
Changed lines of the file:
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@@
 <wire x1="34.671" y1="-12.672" x2="34.671" y2="-13.462" width="0.2794" layer="1"/>
 <via x="34.671" y="-13.462" extent="1-16" drill="0.254"/>
-<wire x1="-54.032" y1="-17.465" x2="-54.925" y2="-17.465" width="0.4064" layer="1"/>
-<via x="-54.925" y="-17.465" extent="1-16" drill="0.254"/>
+<wire x1="-54.032" y1="-17.465" x2="-55.306" y2="-17.465" width="0.4064" layer="1"/>
+<via x="-55.306" y="-17.465" extent="1-16" drill="0.254"/>
 <wire x1="-55.306" y1="-16.825" x2="-55.245" y2="-16.764" width="0.4064" layer="2"/>
-<wire x1="-51.632" y1="-19.365" x2="-50.734" y2="-19.365" width="0.4064" layer="1"/>
-<via x="-50.734" y="-19.365" extent="1-16" drill="0.254"/>
+<wire x1="-51.632" y1="-19.365" x2="-50.353" y2="-19.365" width="0.4064" layer="1"/>
+<via x="-50.353" y="-19.365" extent="1-16" drill="0.254"/>
 <via x="24.483" y="4.544" extent="1-16" drill="0.254"/>
 <wire x1="24.483" y1="4.671" x2="24.511" y2="4.699" width="0.2794" layer="2"/>
@@
 <wire x1="-6.223" y1="-24.257" x2="-52.197" y2="-24.257" width="0.1524" layer="1"/>
 <wire x1="-52.197" y1="-24.257" x2="-55.88" y2="-20.574" width="0.1524" layer="1"/>
-<via x="-55.88" y="-20.574" extent="1-16" drill="0.254"/>
-<wire x1="-55.88" y1="-20.574" x2="-55.88" y2="-18.415" width="0.1524" layer="16"/>
-<via x="-55.88" y="-18.415" extent="1-16" drill="0.254"/>
-<wire x1="-55.88" y1="-18.415" x2="-54.032" y2="-18.415" width="0.1524" layer="1"/>
 <wire x1="61.976" y1="-7.874" x2="62.738" y2="-8.636" width="0.1524" layer="16"/>
 <via x="62.738" y="-8.636" extent="1-16" drill="0.254"/>
@@
 <wire x1="41.783" y1="-8.89" x2="45.085" y2="-8.89" width="0.1524" layer="1"/>
 <wire x1="45.085" y1="-8.89" x2="46.101" y2="-7.874" width="0.1524" layer="1"/>
+<wire x1="-55.88" y1="-20.574" x2="-55.88" y2="-19.05" width="0.1524" layer="1"/>
+<wire x1="-55.88" y1="-19.05" x2="-55.245" y2="-18.415" width="0.1524" layer="1"/>
+<wire x1="-55.245" y1="-18.415" x2="-54.032" y2="-18.415" width="0.1524" layer="1"/>
 </signal>
 <signal name="AUDIO_STREAMING">
@@
 <wire x1="-31.877" y1="-16.51" x2="-33.401" y2="-14.986" width="0.2032" layer="1"/>
 <wire x1="-33.401" y1="-14.986" x2="-47.879" y2="-14.986" width="0.2032" layer="1"/>
-<wire x1="-47.879" y1="-14.986" x2="-50.292" y2="-17.399" width="0.2032" layer="1"/>
-<wire x1="-50.292" y1="-17.399" x2="-51.566" y2="-17.399" width="0.2032" layer="1"/>
-<wire x1="-51.566" y1="-17.399" x2="-51.632" y2="-17.465" width="0.1524" layer="1"/>
+<wire x1="-47.879" y1="-14.986" x2="-50.358" y2="-17.465" width="0.2032" layer="1"/>
+<wire x1="-51.632" y1="-17.465" x2="-50.358" y2="-17.465" width="0.2032" layer="1"/>
 </signal>
 <signal name="N$19">
@@
 <wire x1="7.62" y1="15.621" x2="-34.417" y2="15.621" width="0.2032" layer="1"/>
 <wire x1="-34.417" y1="15.621" x2="-39.243" y2="10.795" width="0.2032" layer="1"/>
-<wire x1="-60.833" y1="-19.431" x2="-54.098" y2="-19.431" width="0.2032" layer="1"/>
-<wire x1="-54.098" y1="-19.431" x2="-54.032" y2="-19.365" width="0.1524" layer="1"/>
-<via x="-60.833" y="-19.431" extent="1-16" drill="0.254"/>
-<wire x1="-60.833" y1="-19.431" x2="-60.833" y2="-17.526" width="0.2032" layer="16"/>
 <via x="-39.243" y="10.795" extent="1-16" drill="0.254"/>
 <wire x1="-39.243" y1="10.795" x2="-39.243" y2="-9.271" width="0.2032" layer="16"/>
 <wire x1="-39.243" y1="-9.271" x2="-44.196" y2="-14.224" width="0.2032" layer="16"/>
-<wire x1="-44.196" y1="-14.224" x2="-57.531" y2="-14.224" width="0.2032" layer="16"/>
-<wire x1="-57.531" y1="-14.224" x2="-60.833" y2="-17.526" width="0.2032" layer="16"/>
+<wire x1="-44.196" y1="-14.224" x2="-50.927" y2="-14.224" width="0.2032" layer="16"/>
+<wire x1="-50.927" y1="-14.224" x2="-52.832" y2="-16.129" width="0.2032" layer="16"/>
+<wire x1="-52.832" y1="-16.129" x2="-52.832" y2="-18.542" width="0.2032" layer="16"/>
+<via x="-52.832" y="-18.542" extent="1-16" drill="0.254"/>
+<wire x1="-52.832" y1="-18.542" x2="-52.832" y2="-19.05" width="0.2032" layer="1"/>
+<wire x1="-52.832" y1="-19.05" x2="-53.147" y2="-19.365" width="0.2032" layer="1"/>
+<wire x1="-54.032" y1="-19.365" x2="-53.147" y2="-19.365" width="0.2032" layer="1"/>
 </signal>
 <signal name="N$38">
