File: projects/usb-dac-amplifier-rev-a/smartstand-usb-dac-amplifier-rev-a.sch (EAGLE design)
At the start: 224 parts, among them J1 PJ-002A, J2 292304-1, J3 NRJ6HH, J4 PJRAN2XIU01AUX, J5 T1M-5POS, U1 XUF208-256-TQ64, U10 TPS3702, U11 PCM5102A, U12 SZNUD3124, U13 NJM2068M, U14 NJM4556AM, U15 NJM4556AM, U16 TS5A3159DBV, U17 SN74LVC3G34, U2 TPD4E02B04, U3 TPS563200DDC, U4 TPS7A8300RGW, U5 TPS563200DDC, U6 TPS7A8300RGW, U7 TPS7A8300RGW, U8 TPS7A4701RGW, U9 TPS7A3301RGW, X1 24MHz, X2 22.5792MHz, X3 24.576MHz

Commit message: Ensure all resistors and capacitors in audio path are spec'd correctly.
Basically just went through and made sure we had 0.1% tolerance on the
resistors, with the exception of 1% on the outout resistors because
percision ones (aka current sense resistors ) are $xx.xx, and made sure
that our capacitors are C0G/NP0.  I switched to film capacitors for the
DC blocking input capacitors on the output stage because values that
large for C0G/NP0 ceramics don't exist on Mouser.

Also added ESD protection to the headphone output and line output,
specifically using the TPD2E007, which is specified for AC signals like
ours, and won't activate with our -/+10V rails.
Parts:
- added U18, U19: TPD2E007DCK, texas-instruments:TPD2E007DCK
- C101, C102: device rcl:CAPACITOR-HORIZONTAL-0603 -> rcl:CAPACITOR-HORIZONTAL-KEMET-5MM-6.0-7.2; PN (none) -> RSBCC4220Z310K
- C83, C84: value 2.2nF -> 2.2nF, C0G; PN (none) -> C0402C222J3GACTU
- C91, C92, C93, C94: value 220pF -> 220pF, C0G; PN (none) -> GRM1555C1H221JA01J
- R22, R23: value 470 -> 470, 0.1%; PN (none) -> RG1005P-471-B-T5
- R24, R28: value 243 -> 243, 0.1%; PN (none) -> ERA-2AEB2430X
- R25, R29, R46: value 10K -> 10K, 0.1%; PN (none) -> ERA-2AEB103X
- R26, R30: value 1.5K -> 1.5K, 0.1%; PN (none) -> RG1005P-152-B-T5
- R31, R32: value 243 -> 243, 0.1%; device rcl:R-US_R0603 -> rcl:R-US_R0402; PN (none) -> ERA-2AEB2430X
- R33, R34: value 715 -> 715, 0.1%; device rcl:R-US_R0603 -> rcl:R-US_R0402; PN (none) -> ERA-2AEB7150X
- R35, R37, R38, R40: PN (none) -> MCA12060C1008FP500
- R36, R39: value 40.2K, 1% -> 40.2K, 0.1%; PN (none) -> RG1005P-4022-B-T5
Connections:
- net AGND: now also U18.GND, U19.GND
- net LINE_OUT_LEFT: now also U19.IO2
- net LINE_OUT_RIGHT: now also U19.IO1
- net N$27: now also U18.IO2
- net N$29: now also U18.IO1
Other:
- moved on the sheet: C101, C102, C122, C83, C84, C91, C92, C93, C94, R24, R25, R26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

Commit message: Adding part numbers for major components.
Parts:
- J3: PN (none) -> NRJ6HH
- J4: value PJRAN2XIU01AUX -> PJRAN2X1U01AUX; PN (none) -> PJRAN2X1U01AUX
- J5: PN (none) -> T1M-05-T-S-RA-TR
- L1: PN (none) -> VLP8040T-2R2N
- L2: PN (none) -> VLP8040T-1R5N
- RL1, RL2: PN (none) -> TQ2-12V
- U11: PN (none) -> PCM5102APWR
- U12: PN (none) -> SZNUD3124DMT1G
- U13: PN (none) -> NJM2068M-TE1
- U14, U15: PN (none) -> NJM4556AM-TE1
- U16: PN (none) -> TS5A3159DBVR
- U17: value SN74LVC3G34 -> SN74LVC3G34DCU; device texas-instruments:SN74LVC3G34 -> texas-instruments:SN74LVC3G34DCU; PN (none) -> SN74LVC3G34DCUT
- U18, U19: PN (none) -> TPD2E007DCKR
- U2: value TPD4E02B04 -> TPD4E02B04DQA; device texas-instruments:TPD4E02B04 -> texas-instruments:TPD4E02B04DQA; PN (none) -> TPD4E02B04DQAR
- U3, U5: PN (none) -> TPS563200DDCR
- U4, U6, U7: PN (none) -> TPS7A8300RGWR
- U8: PN (none) -> TPS7A4701RGWR
- U9: PN (none) -> TPS7A3301RGWR
- VR1: PN (none) -> RK14K1240A4S
- X2: PN (none) -> KC2520K22.5792C1GE00
- X3: PN (none) -> KC2520K24.5760C1GE00
Other:
- moved on the sheet: D4, D6, D7, R49, R51, R52

Commit message: Adding more part numbers and fixing incorrect ones.
Parts:
- J2: PN (none) -> 292304-1
- JP1: PN (none) -> 961206-6404-AR
- U10: PN TPS3702CX10DDC -> TPS3702CX10DDCT
Changed lines of the file:
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@@
 <part name="AGND24" library="supply1" deviceset="AGND" device=""/>
 <part name="U10" library="texas-instruments" deviceset="TPS3702" device="CX10DDC" value="TPS3702">
-<attribute name="PN" value="TPS3702CX10DDC"/>
+<attribute name="PN" value="TPS3702CX10DDCT"/>
 </part>
 <part name="AGND18" library="supply1" deviceset="AGND" device=""/>
@@
 <attribute name="PN" value="T1M-05-T-S-RA-TR"/>
 </part>
-<part name="JP1" library="pinhead" deviceset="PINHD-2X3" device=""/>
+<part name="JP1" library="pinhead" deviceset="PINHD-2X3" device="">
+<attribute name="PN" value="961206-6404-AR"/>
+</part>
 <part name="C76" library="rcl" deviceset="C-EU" device="C0402" value="100nF">
 <attribute name="PN" value="GRM155R71C104KA88D"/>
@@
 <part name="AGND69" library="supply1" deviceset="AGND" device=""/>
 <part name="+1V07" library="supply1" deviceset="+1V0" device=""/>
-<part name="J2" library="te-connectivity" deviceset="292304" device="-1"/>
+<part name="J2" library="te-connectivity" deviceset="292304" device="-1">
+<attribute name="PN" value="292304-1"/>
+</part>
 <part name="U18" library="texas-instruments" deviceset="TPD2E007" device="DCK">
 <attribute name="PN" value="TPD2E007DCKR"/>
@@
 <instance part="AGND5" gate="VR1" x="177.8" y="106.68"/>
 <instance part="AGND6" gate="VR1" x="190.5" y="106.68"/>
-<instance part="J2" gate="G$1" x="53.34" y="52.07"/>
+<instance part="J2" gate="G$1" x="53.34" y="52.07">
+<attribute name="PN" x="53.34" y="52.07" size="1.778" layer="96" display="off"/>
+</instance>
 </instances>
 <busses>
@@
 <instance part="C98" gate="G$1" x="205.74" y="33.02"/>
 <instance part="C100" gate="G$1" x="233.68" y="33.02"/>
-<instance part="JP1" gate="A" x="71.12" y="36.83"/>
+<instance part="JP1" gate="A" x="71.12" y="36.83">
+<attribute name="PN" x="71.12" y="36.83" size="1.778" layer="96" display="off"/>
+</instance>
 </instances>
 <busses>
