File: projects/usb-dac-amplifier-rev-a/smartstand-usb-dac-amplifier-rev-a.sch (EAGLE design)
At the start: 226 parts, among them J1 PJ-002A, J2 292304-1, J3 NRJ6HH, J4 PJRAN2X1U01AUX, J5 T1M-5POS, U1 XUF208-256-TQ64, U10 TPS3702, U11 PCM5102A, U12 SZNUD3124, U13 NJM2068M, U14 NJM4556AM, U15 NJM4556AM, U16 TS5A3159DBV, U17 SN74LVC3G34DCU, U18 TPD2E007DCK, U19 TPD2E007DCK, U2 TPD4E02B04DQA, U3 TPS563200DDC, U4 TPS7A8300RGW, U5 TPS563200DDC, U6 TPS7A8300RGW, U7 TPS7A8300RGW, U8 TPS7A4701RGW, U9 TPS7A3301RGW, X1 24MHz, X2 22.5792MHz, X3 24.576MHz

Commit message: Some housekeeping tasks to keep up the schematic.
Switched from R_US/R_US-VERTICAL to RESISTOR and RESISTOR-HORIZONTAL,
which brings up in line with our usage of CAPACITOR and
CAPACITOR-HORIZONTAL.  Ultimately, our likelihood of using through-hole
passives is very, very low, so I'm trying to commit to pruning down our
rcl (to eventually be named 'passives') library to the most basic/common
SMD passives footprints and nothing more

Also added part numbers, en masse, for many passives.  This is taking
advantage of our new tooling for finding inconsistencies in the
schematic, such as parts missing a part number or identical parts
(device and value) with different part numbers attached to them.  That
still needs to be put into its own repo, and eventually, we'll run it as
part of an automated test against this repository for a continual
feedback loop.  Until then...
Parts:
- C10, C23: PN (none) -> 12063D226KAT2A
- C100, C105, C108, C111, C114, C97: PN (none) -> GRM1555C1H330JA01D
- C103, C106, C109, C112, C12, C122, C16, C25, C29, C37, C42, C45, C48, C49, C50, C53, C56, C57, C95, C98: PN (none) -> GRM155R71H104KE14D
- C104, C107, C110, C113, C20, C22, C33, C34, C41, C9, C96, C99: PN (none) -> GRM15XR71C103KA86D
- C11, C15, C24, C28, C36, C44, C47, C52, C55: PN (none) -> GCM188R71E105KA64D
- C115, C118: device rcl:C-EUC0603 -> rcl:CAPACITOR-0603; PN (none) -> GCM188R71E105KA64D
- C116, C119, C121: device rcl:C-EUC0402 -> rcl:CAPACITOR-0402; PN (none) -> GRM155R71H104KE14D
- C117, C120: device rcl:C-EUC0402 -> rcl:CAPACITOR-0402; PN (none) -> GRM15XR71C103KA86D
- C14, C17, C18, C19, C27, C30, C31, C32, C35, C38, C39, C40, C43, C46, C51, C54: PN (none) -> GRM21BR61E106KA73L
- C21, C8: PN (none) -> C0805C104K5RACTU
- C79, C85, C87, C89: PN GRM155R71C104KA88D -> GRM155R71H104KE14D
- C80, C86, C88, C90: PN EEE-1CA100SR -> GRM21BR61E106KA73L
- R1, R19, R20, R22, R23, R24, R26, R28, R30, R31, R32, R33, R34: device rcl:R-US_R0402 -> rcl:RESISTOR-HORIZONTAL-0402
- R10: device rcl:R-US-VERTICALR0402 -> rcl:RESISTOR-0402; PN (none) -> RC0402FR-079K76L
- R11: device rcl:R-US-VERTICALR0402 -> rcl:RESISTOR-0402; PN (none) -> RK73H1ETTP1154F
- R12: device rcl:R-US-VERTICALR0402 -> rcl:RESISTOR-0402; PN (none) -> RC0402FR-07137KL
- R13, R14, R25, R29, R36, R39, R46, R48, R49, R50, R51, R52, R53: device rcl:R-US-VERTICALR0402 -> rcl:RESISTOR-0402
- R15, R21, R41, R42: device rcl:R-US_R0402 -> rcl:RESISTOR-HORIZONTAL-0402; PN (none) -> ERJ-2GE0R00X
- R17, R18: device rcl:R-US-VERTICALR0402 -> rcl:RESISTOR-0402; PN (none) -> RC0402FR-074K7L
- R2, R4, R5, R7, R8: device rcl:R-US-VERTICALR0402 -> rcl:RESISTOR-0402; PN (none) -> RK73B1ETTP103J
- R3: device rcl:R-US-VERTICALR0402 -> rcl:RESISTOR-0402; PN (none) -> RK73H1ETTP4022F
- R35, R37, R38, R40: device rcl:R-US_R1206 -> rcl:RESISTOR-HORIZONTAL-1206
- R43, R45: device rcl:R-US-VERTICALR0402 -> rcl:RESISTOR-0402; PN (none) -> RK73H1ETTP1003F
- R47: device rcl:R-US_R0402 -> rcl:RESISTOR-HORIZONTAL-0402; PN (none) -> RC0402FR-0749K9L
- R6: device rcl:R-US-VERTICALR0402 -> rcl:RESISTOR-0402; PN (none) -> RC0402FR-078K45L
- R9: device rcl:R-US-VERTICALR0402 -> rcl:RESISTOR-0402; PN (none) -> RK73H1ETTP6652F

Commit message: testing the tests :P
Parts:
- C60: PN GRM155R71C104KA88D -> GRM155R71C104KA88D-X
Changed lines of the file:
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@@
 <part name="SHEET5" library="frames" deviceset="A4L-NODOC" device=""/>
 <part name="C60" library="rcl" deviceset="C-EU" device="C0402" value="100nF">
-<attribute name="PN" value="GRM155R71C104KA88D"/>
+<attribute name="PN" value="GRM155R71C104KA88D-X"/>
 </part>
 <part name="C61" library="rcl" deviceset="C-EU" device="C0402" value="100nF">

Commit message: Alright, tests catch failures properly so going back to clean.
Parts:
- C60: PN GRM155R71C104KA88D-X -> GRM155R71C104KA88D
Changed lines of the file:
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@@
 <part name="SHEET5" library="frames" deviceset="A4L-NODOC" device=""/>
 <part name="C60" library="rcl" deviceset="C-EU" device="C0402" value="100nF">
-<attribute name="PN" value="GRM155R71C104KA88D-X"/>
+<attribute name="PN" value="GRM155R71C104KA88D"/>
 </part>
 <part name="C61" library="rcl" deviceset="C-EU" device="C0402" value="100nF">
