File: projects/usb-dac-amplifier-rev-a/smartstand-usb-dac-amplifier-rev-a.sch (EAGLE design)
At the start: 226 parts, among them J1 PJ-002A, J2 292304-1, J3 NRJ6HH, J4 PJRAN2X1U01AUX, J5 T1M-5POS, U1 XUF208-256-TQ64, U10 TPS3702, U11 PCM5102A, U12 SZNUD3124, U13 NJM2068M, U14 NJM4556AM, U15 NJM4556AM, U16 TS5A3159DBV, U17 SN74LVC3G34DCU, U18 TPD2E007DCK, U19 TPD2E007DCK, U2 TPD4E02B04DQA, U3 TPS563200DDC, U4 TPS7A8300RGW, U5 TPS563200DDC, U6 TPS7A8300RGW, U7 TPS7A8300RGW, U8 TPS7A4701RGW, U9 TPS7A3301RGW, X1 24MHz, X2 22.5792MHz, X3 24.576MHz

Commit message: Switch over to renamed libraries.
Parts:
- C1, C2, C3, C4, C5, C6: device rcl:CPOL-EUCHEMICON_F55 -> passives:CPOL-EUCHEMICON_F55
- C10, C13, C23, C26: device rcl:CAPACITOR-1206 -> passives:CAPACITOR-1206
- C100, C103, C104, C105, C106, C107, C108, C109, C110, C111, C112, C113, C114, C116, C117, C119, C12, C120, C121, C122, C16, C20, C22, C25, C29, C33, C34, C37, C41, C42, C45, C48, C49, C50, C53, C56, C57, C79, C83, C84, C85, C87, C89, C9, C91, C93, C95, C96, C97, C98, C99: device rcl:CAPACITOR-0402 -> passives:CAPACITOR-0402
- C101, C102: device rcl:CAPACITOR-HORIZONTAL-KEMET-5MM-6.0-7.2 -> passives:CAPACITOR-HORIZONTAL-KEMET-5MM-6.0-7.2
- C11, C115, C118, C15, C24, C28, C36, C44, C47, C52, C55, C81, C82: device rcl:CAPACITOR-0603 -> passives:CAPACITOR-0603
- C14, C17, C18, C19, C27, C30, C31, C32, C35, C38, C39, C40, C43, C46, C51, C54, C80, C86, C88, C90: device rcl:CAPACITOR-0805 -> passives:CAPACITOR-0805
- C21, C8: device rcl:CAPACITOR-HORIZONTAL-0805 -> passives:CAPACITOR-HORIZONTAL-0805
- C58, C59, C60, C61, C62, C63, C64, C65, C66, C67, C68, C69, C70, C71, C72, C73, C74, C75, C76, C77, C78: device rcl:C-EUC0402 -> passives:C-EUC0402
- C7: device rcl:C-EUC0603 -> passives:C-EUC0603
- C92, C94: device rcl:CAPACITOR-HORIZONTAL-0402 -> passives:CAPACITOR-HORIZONTAL-0402
- JP1: device pinhead:PINHD-2X3 -> pin-headers:PINHD-2X3
- JP2: device pinhead:PINHD-2X10 -> pin-headers:PINHD-2X10
- L1, L2: device rcl:L-USVLP8040 -> passives:L-USVLP8040
- R1, R15, R19, R20, R21, R22, R23, R24, R26, R28, R30, R31, R32, R33, R34, R41, R42, R47: device rcl:RESISTOR-HORIZONTAL-0402 -> passives:RESISTOR-HORIZONTAL-0402
- R10, R11, R12, R13, R14, R17, R18, R2, R25, R29, R3, R36, R39, R4, R43, R45, R46, R48, R49, R5, R50, R51, R52, R53, R6, R7, R8, R9: device rcl:RESISTOR-0402 -> passives:RESISTOR-0402
- R16: device rcl:R-US_R0402 -> passives:R-US_R0402
- R35, R37, R38, R40: device rcl:RESISTOR-HORIZONTAL-1206 -> passives:RESISTOR-HORIZONTAL-1206

Commit message: Converting over to our simplified passives.
Parts:
- C1, C2, C3, C4, C5, C6: device passives:CPOL-EUCHEMICON_F55 -> passives:CAPACITOR-POLARIZEDCHEMICON_F55
- C58, C59, C60, C61, C62, C63, C64, C65, C66, C67, C68, C69, C70, C71, C72, C73, C74, C75, C76, C77, C78: device passives:C-EUC0402 -> passives:CAPACITOR-0402
- C7: device passives:C-EUC0603 -> passives:CAPACITOR-0603
- L1, L2: device passives:L-USVLP8040 -> passives:INDUCTOR-HORIZONTALVLP8040
- R16: device passives:R-US_R0402 -> passives:RESISTOR-HORIZONTAL-0402
Changed lines of the file:
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@@
 <attribute name="PN" value="PMEG3050BEP,115"/>
 </part>
-<part name="C1" library="passives" deviceset="CPOL-EU" device="CHEMICON_F55" value="47uF">
+<part name="C1" library="passives" deviceset="CAPACITOR-POLARIZED" device="CHEMICON_F55" value="47uF">
 <attribute name="PN" value="EMVA250ADA470MF55G"/>
 </part>
-<part name="C2" library="passives" deviceset="CPOL-EU" device="CHEMICON_F55" value="47uF">
+<part name="C2" library="passives" deviceset="CAPACITOR-POLARIZED" device="CHEMICON_F55" value="47uF">
 <attribute name="PN" value="EMVA250ADA470MF55G"/>
 </part>
-<part name="C3" library="passives" deviceset="CPOL-EU" device="CHEMICON_F55" value="47uF">
+<part name="C3" library="passives" deviceset="CAPACITOR-POLARIZED" device="CHEMICON_F55" value="47uF">
 <attribute name="PN" value="EMVA250ADA470MF55G"/>
 </part>
-<part name="C4" library="passives" deviceset="CPOL-EU" device="CHEMICON_F55" value="47uF">
+<part name="C4" library="passives" deviceset="CAPACITOR-POLARIZED" device="CHEMICON_F55" value="47uF">
 <attribute name="PN" value="EMVA250ADA470MF55G"/>
 </part>
@@
 </part>
 <part name="AGND22" library="supplies" deviceset="AGND" device=""/>
-<part name="C77" library="passives" deviceset="C-EU" device="C0402" value="100nF">
+<part name="C77" library="passives" deviceset="CAPACITOR" device="-0402" value="100nF">
 <attribute name="PN" value="GRM155R71C104KA88D"/>
 </part>
@@
 <attribute name="PN" value="SG73P1ETTP4R7J"/>
 </part>
-<part name="C78" library="passives" deviceset="C-EU" device="C0402" value="100nF">
-<attribute name="PN" value="GRM155R71C104KA88D"/>
-</part>
-<part name="R16" library="passives" deviceset="R-US_" device="R0402" value="1K">
+<part name="C78" library="passives" deviceset="CAPACITOR" device="-0402" value="100nF">
+<attribute name="PN" value="GRM155R71C104KA88D"/>
+</part>
+<part name="R16" library="passives" deviceset="RESISTOR-HORIZONTAL" device="-0402" value="1K">
 <attribute name="PN" value="RK73B1ETTP102J"/>
 </part>
-<part name="C71" library="passives" deviceset="C-EU" device="C0402" value="100nF">
-<attribute name="PN" value="GRM155R71C104KA88D"/>
-</part>
-<part name="C72" library="passives" deviceset="C-EU" device="C0402" value="100nF">
-<attribute name="PN" value="GRM155R71C104KA88D"/>
-</part>
-<part name="C73" library="passives" deviceset="C-EU" device="C0402" value="100nF">
+<part name="C71" library="passives" deviceset="CAPACITOR" device="-0402" value="100nF">
+<attribute name="PN" value="GRM155R71C104KA88D"/>
+</part>
+<part name="C72" library="passives" deviceset="CAPACITOR" device="-0402" value="100nF">
+<attribute name="PN" value="GRM155R71C104KA88D"/>
+</part>
+<part name="C73" library="passives" deviceset="CAPACITOR" device="-0402" value="100nF">
 <attribute name="PN" value="GRM155R71C104KA88D"/>
 </part>
 <part name="AGND21" library="supplies" deviceset="AGND" device=""/>
 <part name="SHEET5" library="frames" deviceset="A4L-NODOC" device=""/>
-<part name="C60" library="passives" deviceset="C-EU" device="C0402" value="100nF">
-<attribute name="PN" value="GRM155R71C104KA88D"/>
-</part>
-<part name="C61" library="passives" deviceset="C-EU" device="C0402" value="100nF">
-<attribute name="PN" value="GRM155R71C104KA88D"/>
-</part>
-<part name="C62" library="passives" deviceset="C-EU" device="C0402" value="100nF">
-<attribute name="PN" value="GRM155R71C104KA88D"/>
-</part>
-<part name="C63" library="passives" deviceset="C-EU" device="C0402" value="100nF">
-<attribute name="PN" value="GRM155R71C104KA88D"/>
-</part>
-<part name="C64" library="passives" deviceset="C-EU" device="C0402" value="100nF">
-<attribute name="PN" value="GRM155R71C104KA88D"/>
-</part>
-<part name="C65" library="passives" deviceset="C-EU" device="C0402" value="100nF">
-<attribute name="PN" value="GRM155R71C104KA88D"/>
-</part>
-<part name="C66" library="passives" deviceset="C-EU" device="C0402" value="100nF">
-<attribute name="PN" value="GRM155R71C104KA88D"/>
-</part>
-<part name="C67" library="passives" deviceset="C-EU" device="C0402" value="100nF">
-<attribute name="PN" value="GRM155R71C104KA88D"/>
-</part>
-<part name="C68" library="passives" deviceset="C-EU" device="C0402" value="100nF">
-<attribute name="PN" value="GRM155R71C104KA88D"/>
-</part>
-<part name="C69" library="passives" deviceset="C-EU" device="C0402" value="100nF">
-<attribute name="PN" value="GRM155R71C104KA88D"/>
-</part>
-<part name="C70" library="passives" deviceset="C-EU" device="C0402" value="100nF">
+<part name="C60" library="passives" deviceset="CAPACITOR" device="-0402" value="100nF">
+<attribute name="PN" value="GRM155R71C104KA88D"/>
+</part>
+<part name="C61" library="passives" deviceset="CAPACITOR" device="-0402" value="100nF">
+<attribute name="PN" value="GRM155R71C104KA88D"/>
+</part>
+<part name="C62" library="passives" deviceset="CAPACITOR" device="-0402" value="100nF">
+<attribute name="PN" value="GRM155R71C104KA88D"/>
+</part>
+<part name="C63" library="passives" deviceset="CAPACITOR" device="-0402" value="100nF">
+<attribute name="PN" value="GRM155R71C104KA88D"/>
+</part>
+<part name="C64" library="passives" deviceset="CAPACITOR" device="-0402" value="100nF">
+<attribute name="PN" value="GRM155R71C104KA88D"/>
+</part>
+<part name="C65" library="passives" deviceset="CAPACITOR" device="-0402" value="100nF">
+<attribute name="PN" value="GRM155R71C104KA88D"/>
+</part>
+<part name="C66" library="passives" deviceset="CAPACITOR" device="-0402" value="100nF">
+<attribute name="PN" value="GRM155R71C104KA88D"/>
+</part>
+<part name="C67" library="passives" deviceset="CAPACITOR" device="-0402" value="100nF">
+<attribute name="PN" value="GRM155R71C104KA88D"/>
+</part>
+<part name="C68" library="passives" deviceset="CAPACITOR" device="-0402" value="100nF">
+<attribute name="PN" value="GRM155R71C104KA88D"/>
+</part>
+<part name="C69" library="passives" deviceset="CAPACITOR" device="-0402" value="100nF">
+<attribute name="PN" value="GRM155R71C104KA88D"/>
+</part>
+<part name="C70" library="passives" deviceset="CAPACITOR" device="-0402" value="100nF">
 <attribute name="PN" value="GRM155R71C104KA88D"/>
 </part>
 <part name="AGND20" library="supplies" deviceset="AGND" device=""/>
-<part name="C7" library="passives" deviceset="C-EU" device="C0603" value="1uF">
+<part name="C7" library="passives" deviceset="CAPACITOR" device="-0603" value="1uF">
 <attribute name="PN" value="GRM188R61C225KE15D"/>
 </part>
-<part name="C74" library="passives" deviceset="C-EU" device="C0402" value="100nF">
-<attribute name="PN" value="GRM155R71C104KA88D"/>
-</part>
-<part name="C75" library="passives" deviceset="C-EU" device="C0402" value="100nF">
+<part name="C74" library="passives" deviceset="CAPACITOR" device="-0402" value="100nF">
+<attribute name="PN" value="GRM155R71C104KA88D"/>
+</part>
+<part name="C75" library="passives" deviceset="CAPACITOR" device="-0402" value="100nF">
 <attribute name="PN" value="GRM155R71C104KA88D"/>
 </part>
@@
 <part name="+1V06" library="supplies" deviceset="+1V0" device=""/>
 <part name="+1V03" library="supplies" deviceset="+1V0" device=""/>
-<part name="C58" library="passives" deviceset="C-EU" device="C0402" value="10nF">
-<attribute name="PN" value="GRM15XR71C103KA86D"/>
-</part>
-<part name="C59" library="passives" deviceset="C-EU" device="C0402" value="10nF">
+<part name="C58" library="passives" deviceset="CAPACITOR" device="-0402" value="10nF">
+<attribute name="PN" value="GRM15XR71C103KA86D"/>
+</part>
+<part name="C59" library="passives" deviceset="CAPACITOR" device="-0402" value="10nF">
 <attribute name="PN" value="GRM15XR71C103KA86D"/>
 </part>
@@
 </part>
 <part name="SHEET2" library="frames" deviceset="A4L-NODOC" device=""/>
-<part name="C5" library="passives" deviceset="CPOL-EU" device="CHEMICON_F55" value="47uF">
+<part name="C5" library="passives" deviceset="CAPACITOR-POLARIZED" device="CHEMICON_F55" value="47uF">
 <attribute name="PN" value="EMVA250ADA470MF55G"/>
 </part>
-<part name="C6" library="passives" deviceset="CPOL-EU" device="CHEMICON_F55" value="47uF">
+<part name="C6" library="passives" deviceset="CAPACITOR-POLARIZED" device="CHEMICON_F55" value="47uF">
 <attribute name="PN" value="EMVA250ADA470MF55G"/>
 </part>
@@
 <attribute name="PN" value="EMVA250ADA470MF55G"/>
 </part>
-<part name="L1" library="passives" deviceset="L-US" device="VLP8040" value="2.2uH">
+<part name="L1" library="passives" deviceset="INDUCTOR-HORIZONTAL" device="VLP8040" value="2.2uH">
 <attribute name="PN" value="VLP8040T-2R2N"/>
 </part>
@@
 <attribute name="PN" value="EMVA250ADA470MF55G"/>
 </part>
-<part name="L2" library="passives" deviceset="L-US" device="VLP8040" value="1.5uH">
+<part name="L2" library="passives" deviceset="INDUCTOR-HORIZONTAL" device="VLP8040" value="1.5uH">
 <attribute name="PN" value="VLP8040T-1R5N"/>
 </part>
@@
 <attribute name="PN" value="961206-6404-AR"/>
 </part>
-<part name="C76" library="passives" deviceset="C-EU" device="C0402" value="100nF">
-<attribute name="PN" value="GRM155R71C104KA88D"/>
-</part>
+<part name="C76" library="passives" deviceset="CAPACITOR" device="-0402" value="100nF">
+<attribute name="PN" value="GRM155R71C104KA88D"/>
+</part>
