File: projects/usb-dac-amplifier-rev-a/smartstand-usb-dac-amplifier-rev-a.sch (EAGLE design)
At the start: 226 parts, among them J1 PJ-002A, J2 292304-1, J3 NRJ6HH, J4 PJRAN2X1U01AUX, J5 T1M-5POS, U1 XUF208-256-TQ64, U10 TPS3702, U11 PCM5102A, U12 SZNUD3124, U13 NJM2068M, U14 NJM4556AM, U15 NJM4556AM, U16 TS5A3159DBV, U17 SN74LVC3G34DCU, U18 TPD2E007DCK, U19 TPD2E007DCK, U2 TPD4E02B04DQA, U3 TPS563200DDC, U4 TPS7A8300RGW, U5 TPS563200DDC, U6 TPS7A8300RGW, U7 TPS7A8300RGW, U8 TPS7A4701RGW, U9 TPS7A3301RGW, X1 24MHz, X2 22.5792MHz, X3 24.576MHz

Commit message: Fix some part number issues.
Parts:
- C11, C115, C118, C15, C24, C28, C36, C44, C47, C52, C55: PN GCM188R71E105KA64D -> GRM188R61E105KA12D
- C60, C61, C62, C63, C64, C65, C66, C67, C68, C69, C70, C71, C72, C73, C74, C75, C76, C77, C78: PN GRM155R71C104KA88D -> GRM155R71H104KE14D
- C7: PN GRM188R61C225KE15D -> GRM188R61E105KA12D

Commit message: Minor board layout tweaks.
Adjusted how we route the USB signals to better take advantage of the
type B connector, which now lets us avoid a layer transition.  We're
about 37mils difference between the pair lengths which is well within
bounds of the 100ps skew allowed by the USB specification.

Also, I mistakenly forgot to route power into the pigtail between the
main board and the headphone detection daughterboard, which is now
rectified.  We're sending it DVDD (3V3) so that it needs no regulator of
its own.  We'll need to make sure that we do have a lot of bulk
capacitance since the pigtail will be 8-12 inches long, and the
measurement current can be large, and thus high di/dt, with frequent
measurements.
Connections:
- net AGND: no longer J5.3
- net DVDD: now also J5.3
- net USB_D_N: now also U2.IO3; no longer U2.IO2
- net USB_D_P: now also U2.IO2; no longer U2.IO3
Other:
- note added: "Headphone Detection Link"
- note added: "This I2C link goes off to the headphone detection daughterboard which provides the proximity sensor to detect when the headphones are on the stand or not."
- moved on the sheet: J5
Changed lines of the file:
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@@
 <setting verticaltext="up"/>
 </settings>
-<grid distance="0.1" unitdist="inch" unit="inch" style="lines" multiple="1" display="no" altdistance="0.01" altunitdist="inch" altunit="inch"/>
+<grid distance="0.05" unitdist="inch" unit="inch" style="lines" multiple="1" display="no" altdistance="0.01" altunitdist="inch" altunit="inch"/>
 <layers>
 <layer number="1" name="Top" color="4" fill="1" visible="no" active="no"/>
@@
 <part name="AGND74" library="supplies" deviceset="AGND" device=""/>
 <part name="AGND75" library="supplies" deviceset="AGND" device=""/>
+<part name="DVDD18" library="supplies" deviceset="DVDD" device=""/>
 </parts>
 <sheets>
@@
 <net name="USB_D_N" class="1">
 <segment>
-<wire x1="66.04" y1="46.99" x2="86.36" y2="46.99" width="0.1524" layer="91"/>
 <pinref part="U1" gate="USB" pin="USB_D-"/>
-<wire x1="184.15" y1="46.99" x2="86.36" y2="46.99" width="0.1524" layer="91"/>
-<pinref part="U2" gate="G$1" pin="IO2"/>
-<wire x1="86.36" y1="39.37" x2="86.36" y2="46.99" width="0.1524" layer="91"/>
-<junction x="86.36" y="46.99"/>
+<wire x1="184.15" y1="46.99" x2="91.44" y2="46.99" width="0.1524" layer="91"/>
 <pinref part="J2" gate="G$1" pin="DM"/>
+<pinref part="U2" gate="G$1" pin="IO3"/>
+<wire x1="91.44" y1="46.99" x2="66.04" y2="46.99" width="0.1524" layer="91"/>
+<wire x1="91.44" y1="39.37" x2="91.44" y2="46.99" width="0.1524" layer="91"/>
+<junction x="91.44" y="46.99"/>
 </segment>
 </net>
 <net name="USB_D_P" class="1">
 <segment>
-<wire x1="91.44" y1="44.45" x2="66.04" y2="44.45" width="0.1524" layer="91"/>
 <pinref part="U1" gate="USB" pin="USB_D+"/>
-<wire x1="91.44" y1="44.45" x2="184.15" y2="44.45" width="0.1524" layer="91"/>
-<pinref part="U2" gate="G$1" pin="IO3"/>
-<wire x1="91.44" y1="39.37" x2="91.44" y2="44.45" width="0.1524" layer="91"/>
-<junction x="91.44" y="44.45"/>
+<wire x1="66.04" y1="44.45" x2="86.36" y2="44.45" width="0.1524" layer="91"/>
 <pinref part="J2" gate="G$1" pin="DP"/>
+<pinref part="U2" gate="G$1" pin="IO2"/>
+<wire x1="86.36" y1="44.45" x2="184.15" y2="44.45" width="0.1524" layer="91"/>
+<wire x1="86.36" y1="39.37" x2="86.36" y2="44.45" width="0.1524" layer="91"/>
+<junction x="86.36" y="44.45"/>
 </segment>
 </net>
@@
 It uses two xLINK connections to provide a high-speed
 connection for taking xSCOPE measurements.</text>
+<text x="137.16" y="68.58" size="5.08" layer="112">Headphone Detection Link</text>
+<text x="137.16" y="52.07" size="3.302" layer="113">This I2C link goes off to the headphone detection
+daughterboard which provides the proximity sensor to
+detect when the headphones are on the stand or not.</text>
 </plain>
 <instances>
@@
 <instance part="P+16" gate="1" x="19.05" y="41.91"/>
 <instance part="P-8" gate="1" x="43.18" y="41.91" rot="R180"/>
-<instance part="AGND70" gate="VR1" x="170.18" y="35.56"/>
-<instance part="J5" gate="G$1" x="181.61" y="50.8">
-<attribute name="PN" x="181.61" y="50.8" size="1.778" layer="96" display="off"/>
+<instance part="AGND70" gate="VR1" x="172.72" y="17.78"/>
+<instance part="J5" gate="G$1" x="184.15" y="30.48">
+<attribute name="PN" x="184.15" y="30.48" size="1.778" layer="96" display="off"/>
 </instance>
 <instance part="TP2" gate="G$1" x="25.4" y="125.73"/>
@@
 <instance part="AGND69" gate="VR1" x="41.91" y="53.34"/>
 <instance part="+1V07" gate="G$1" x="41.91" y="73.66"/>
+<instance part="DVDD18" gate="G$1" x="175.26" y="44.45"/>
 </instances>
 <busses>
@@
 <segment>
 <pinref part="AGND70" gate="VR1" pin="AGND"/>
-<wire x1="181.61" y1="45.72" x2="170.18" y2="45.72" width="0.1524" layer="91"/>
-<wire x1="170.18" y1="45.72" x2="170.18" y2="38.1" width="0.1524" layer="91"/>
-<wire x1="181.61" y1="50.8" x2="170.18" y2="50.8" width="0.1524" layer="91"/>
-<wire x1="170.18" y1="50.8" x2="170.18" y2="45.72" width="0.1524" layer="91"/>
-<junction x="170.18" y="45.72"/>
-<pinref part="J5" gate="G$1" pin="3"/>
+<wire x1="184.15" y1="25.4" x2="172.72" y2="25.4" width="0.1524" layer="91"/>
+<wire x1="172.72" y1="25.4" x2="172.72" y2="20.32" width="0.1524" layer="91"/>
+<junction x="172.72" y="25.4"/>
 <pinref part="J5" gate="G$1" pin="5"/>
 <pinref part="J5" gate="G$1" pin="1"/>
-<wire x1="181.61" y1="55.88" x2="170.18" y2="55.88" width="0.1524" layer="91"/>
-<wire x1="170.18" y1="55.88" x2="170.18" y2="50.8" width="0.1524" layer="91"/>
-<junction x="170.18" y="50.8"/>
+<wire x1="184.15" y1="35.56" x2="172.72" y2="35.56" width="0.1524" layer="91"/>
+<wire x1="172.72" y1="35.56" x2="172.72" y2="25.4" width="0.1524" layer="91"/>
 </segment>
 <segment>
@@
 <net name="I2C_SCL" class="0">
 <segment>
-<wire x1="181.61" y1="53.34" x2="165.1" y2="53.34" width="0.1524" layer="91"/>
-<label x="165.1" y="53.34" size="2.54" layer="95" rot="R180" xref="yes"/>
+<wire x1="184.15" y1="33.02" x2="167.64" y2="33.02" width="0.1524" layer="91"/>
+<label x="167.64" y="33.02" size="2.54" layer="95" rot="R180" xref="yes"/>
 <pinref part="J5" gate="G$1" pin="2"/>
 </segment>
@@
 <net name="I2C_SDA" class="0">
 <segment>
-<wire x1="181.61" y1="48.26" x2="165.1" y2="48.26" width="0.1524" layer="91"/>
-<label x="165.1" y="48.26" size="2.54" layer="95" rot="R180" xref="yes"/>
+<wire x1="184.15" y1="27.94" x2="167.64" y2="27.94" width="0.1524" layer="91"/>
+<label x="167.64" y="27.94" size="2.54" layer="95" rot="R180" xref="yes"/>
 <pinref part="J5" gate="G$1" pin="4"/>
 </segment>
@@
 <wire x1="41.91" y1="95.25" x2="41.91" y2="102.87" width="0.1524" layer="91"/>
 </segment>
+<segment>
+<pinref part="J5" gate="G$1" pin="3"/>
+<wire x1="184.15" y1="30.48" x2="175.26" y2="30.48" width="0.1524" layer="91"/>
+<wire x1="175.26" y1="30.48" x2="175.26" y2="41.91" width="0.1524" layer="91"/>
+<pinref part="DVDD18" gate="G$1" pin="DVDD"/>
+</segment>
 </net>

Commit message: Adjust the I2C pinout on the daughterboard connector.
This will let us have cleaner routing on the small daughterboard which
houses the proximity sensor.
Connections:
- net DVDD: now also J5.2; no longer J5.3
- net I2C_SCL: now also J5.4, R18.1; no longer J5.2, R17.1
- net I2C_SDA: now also J5.3, R17.1; no longer J5.4, R18.1
Changed lines of the file:
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@@
 <class number="0" name="default" width="0.1524" drill="0.254">
 </class>
-<class number="1" name="USB" width="0.3048" drill="0.254">
+<class number="1" name="USB" width="0.2794" drill="0.254">
 </class>
 </classes>
@@
 <segment>
 <pinref part="U1" gate="IO" pin="X0D11"/>
-<wire x1="88.9" y1="41.91" x2="62.23" y2="41.91" width="0.1524" layer="91"/>
+<wire x1="88.9" y1="41.91" x2="52.07" y2="41.91" width="0.1524" layer="91"/>
 <label x="45.72" y="41.91" size="2.54" layer="95" rot="R180" xref="yes"/>
-<pinref part="R18" gate="G$1" pin="1"/>
-<wire x1="62.23" y1="41.91" x2="45.72" y2="41.91" width="0.1524" layer="91"/>
-<wire x1="62.23" y1="49.53" x2="62.23" y2="41.91" width="0.1524" layer="91"/>
-<junction x="62.23" y="41.91"/>
+<pinref part="R17" gate="G$1" pin="1"/>
+<wire x1="52.07" y1="41.91" x2="45.72" y2="41.91" width="0.1524" layer="91"/>
+<wire x1="52.07" y1="49.53" x2="52.07" y2="41.91" width="0.1524" layer="91"/>
+<junction x="52.07" y="41.91"/>
 </segment>
 </net>
@@
 <wire x1="88.9" y1="59.69" x2="73.66" y2="59.69" width="0.1524" layer="91"/>
 <wire x1="73.66" y1="59.69" x2="73.66" y2="46.99" width="0.1524" layer="91"/>
-<wire x1="73.66" y1="46.99" x2="52.07" y2="46.99" width="0.1524" layer="91"/>
+<wire x1="73.66" y1="46.99" x2="62.23" y2="46.99" width="0.1524" layer="91"/>
 <label x="45.72" y="46.99" size="2.54" layer="95" rot="R180" xref="yes"/>
-<pinref part="R17" gate="G$1" pin="1"/>
-<wire x1="52.07" y1="46.99" x2="45.72" y2="46.99" width="0.1524" layer="91"/>
-<wire x1="52.07" y1="49.53" x2="52.07" y2="46.99" width="0.1524" layer="91"/>
-<junction x="52.07" y="46.99"/>
+<pinref part="R18" gate="G$1" pin="1"/>
+<wire x1="62.23" y1="46.99" x2="45.72" y2="46.99" width="0.1524" layer="91"/>
+<wire x1="62.23" y1="49.53" x2="62.23" y2="46.99" width="0.1524" layer="91"/>
+<junction x="62.23" y="46.99"/>
 </segment>
 </net>
@@
 <net name="I2C_SCL" class="0">
 <segment>
-<wire x1="184.15" y1="33.02" x2="167.64" y2="33.02" width="0.1524" layer="91"/>
-<label x="167.64" y="33.02" size="2.54" layer="95" rot="R180" xref="yes"/>
-<pinref part="J5" gate="G$1" pin="2"/>
+<label x="167.64" y="27.94" size="2.54" layer="95" rot="R180" xref="yes"/>
+<pinref part="J5" gate="G$1" pin="4"/>
+<wire x1="167.64" y1="27.94" x2="184.15" y2="27.94" width="0.1524" layer="91"/>
 </segment>
 </net>
 <net name="I2C_SDA" class="0">
 <segment>
-<wire x1="184.15" y1="27.94" x2="167.64" y2="27.94" width="0.1524" layer="91"/>
-<label x="167.64" y="27.94" size="2.54" layer="95" rot="R180" xref="yes"/>
-<pinref part="J5" gate="G$1" pin="4"/>
+<wire x1="170.18" y1="33.02" x2="167.64" y2="33.02" width="0.1524" layer="91"/>
+<label x="167.64" y="33.02" size="2.54" layer="95" rot="R180" xref="yes"/>
+<pinref part="J5" gate="G$1" pin="3"/>
+<wire x1="184.15" y1="30.48" x2="170.18" y2="30.48" width="0.1524" layer="91"/>
+<wire x1="170.18" y1="30.48" x2="170.18" y2="33.02" width="0.1524" layer="91"/>
 </segment>
 </net>
@@
 </segment>
 <segment>
-<pinref part="J5" gate="G$1" pin="3"/>
-<wire x1="184.15" y1="30.48" x2="175.26" y2="30.48" width="0.1524" layer="91"/>
-<wire x1="175.26" y1="30.48" x2="175.26" y2="41.91" width="0.1524" layer="91"/>
+<wire x1="175.26" y1="33.02" x2="175.26" y2="41.91" width="0.1524" layer="91"/>
 <pinref part="DVDD18" gate="G$1" pin="DVDD"/>
+<pinref part="J5" gate="G$1" pin="2"/>
+<wire x1="184.15" y1="33.02" x2="175.26" y2="33.02" width="0.1524" layer="91"/>
 </segment>
 </net>

Commit message: Updated component choice to better alternative.
Parts:
- R13, R2, R4, R5, R7, R8: PN RK73B1ETTP103J -> RC0402FR-0710KL
Changed lines of the file:
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@@
 <setting verticaltext="up"/>
 </settings>
-<grid distance="0.05" unitdist="inch" unit="inch" style="lines" multiple="1" display="no" altdistance="0.01" altunitdist="inch" altunit="inch"/>
+<grid distance="0.1" unitdist="inch" unit="inch" style="lines" multiple="1" display="no" altdistance="0.01" altunitdist="inch" altunit="inch"/>
 <layers>
 <layer number="1" name="Top" color="4" fill="1" visible="no" active="no"/>
@@
 <part name="+1V02" library="supplies" deviceset="+1V0" device=""/>
 <part name="R13" library="passives" deviceset="RESISTOR" device="-0402" value="10K">
-<attribute name="PN" value="RK73B1ETTP103J"/>
+<attribute name="PN" value="RC0402FR-0710KL"/>
 </part>
 <part name="R14" library="passives" deviceset="RESISTOR" device="-0402" value="4.7">
@@
 </part>
 <part name="R4" library="passives" deviceset="RESISTOR" device="-0402" value="10K">
-<attribute name="PN" value="RK73B1ETTP103J"/>
+<attribute name="PN" value="RC0402FR-0710KL"/>
 </part>
 <part name="C13" library="passives" deviceset="CAPACITOR" device="-1206" value="47uF">
@@
 </part>
 <part name="R7" library="passives" deviceset="RESISTOR" device="-0402" value="10K">
-<attribute name="PN" value="RK73B1ETTP103J"/>
+<attribute name="PN" value="RC0402FR-0710KL"/>
 </part>
 <part name="C26" library="passives" deviceset="CAPACITOR" device="-1206" value="47uF">
@@
 </part>
 <part name="R5" library="passives" deviceset="RESISTOR" device="-0402" value="10K">
-<attribute name="PN" value="RK73B1ETTP103J"/>
+<attribute name="PN" value="RC0402FR-0710KL"/>
 </part>
 <part name="C30" library="passives" deviceset="CAPACITOR" device="-0805" value="10uF">
@@
 </part>
 <part name="R2" library="passives" deviceset="RESISTOR" device="-0402" value="10K">
-<attribute name="PN" value="RK73B1ETTP103J"/>
+<attribute name="PN" value="RC0402FR-0710KL"/>
 </part>
 <part name="C17" library="passives" deviceset="CAPACITOR" device="-0805" value="10uF">
@@
 </part>
 <part name="R8" library="passives" deviceset="RESISTOR" device="-0402" value="10K">
-<attribute name="PN" value="RK73B1ETTP103J"/>
+<attribute name="PN" value="RC0402FR-0710KL"/>
 </part>
 <part name="C38" library="passives" deviceset="CAPACITOR" device="-0805" value="10uF">

Commit message: Add BOM exclusions to frames/testpoints.
Parts:
- TP1, TP10, TP2, TP3, TP4, TP5, TP6, TP7, TP8, TP9: BOM (none) -> EXCLUDE

Commit message: Add fiducials and fix ERC/DRC errors.
Parts:
- added U$1, U$10, U$11, U$12, U$13, U$2, U$3, U$4, U$5, U$6, U$7, U$8, U$9: FIDUCIAL-1MM, fiducials:FIDUCIAL-1MM
Connections:
- removed net +3V3: U17PWR.VDD
- net DVDD: now also U17PWR.VDD
Other:
- note added: "Fiducials"
- note added: "Fiducials provide a means for automated pick-and-place machines to orient themselves to a board and ensure that they are aligned, delivering accurate placement."
- moved on the sheet: U17B

Commit message: Add BOM exclude to fiducials.
Parts:
- U$1, U$10, U$11, U$12, U$13, U$2, U$3, U$4, U$5, U$6, U$7, U$8, U$9: BOM (none) -> EXCLUDE
Changed lines of the file:
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@@
 <setting verticaltext="up"/>
 </settings>
-<grid distance="0.05" unitdist="inch" unit="inch" style="lines" multiple="1" display="no" altdistance="0.01" altunitdist="inch" altunit="inch"/>
+<grid distance="0.1" unitdist="inch" unit="inch" style="lines" multiple="1" display="no" altdistance="0.01" altunitdist="inch" altunit="inch"/>
 <layers>
 <layer number="1" name="Top" color="4" fill="1" visible="no" active="no"/>
@@
 <part name="AGND75" library="supplies" deviceset="AGND" device=""/>
 <part name="DVDD18" library="supplies" deviceset="DVDD" device=""/>
-<part name="U$1" library="fiducials" deviceset="FIDUCIAL" device="-1MM"/>
-<part name="U$2" library="fiducials" deviceset="FIDUCIAL" device="-1MM"/>
-<part name="U$3" library="fiducials" deviceset="FIDUCIAL" device="-1MM"/>
-<part name="U$4" library="fiducials" deviceset="FIDUCIAL" device="-1MM"/>
-<part name="U$5" library="fiducials" deviceset="FIDUCIAL" device="-1MM"/>
-<part name="U$6" library="fiducials" deviceset="FIDUCIAL" device="-1MM"/>
-<part name="U$7" library="fiducials" deviceset="FIDUCIAL" device="-1MM"/>
-<part name="U$8" library="fiducials" deviceset="FIDUCIAL" device="-1MM"/>
-<part name="U$9" library="fiducials" deviceset="FIDUCIAL" device="-1MM"/>
-<part name="U$10" library="fiducials" deviceset="FIDUCIAL" device="-1MM"/>
-<part name="U$11" library="fiducials" deviceset="FIDUCIAL" device="-1MM"/>
-<part name="U$12" library="fiducials" deviceset="FIDUCIAL" device="-1MM"/>
-<part name="U$13" library="fiducials" deviceset="FIDUCIAL" device="-1MM"/>
+<part name="U$1" library="fiducials" deviceset="FIDUCIAL" device="-1MM">
+<attribute name="BOM" value="EXCLUDE"/>
+</part>
+<part name="U$2" library="fiducials" deviceset="FIDUCIAL" device="-1MM">
+<attribute name="BOM" value="EXCLUDE"/>
+</part>
+<part name="U$3" library="fiducials" deviceset="FIDUCIAL" device="-1MM">
+<attribute name="BOM" value="EXCLUDE"/>
+</part>
+<part name="U$4" library="fiducials" deviceset="FIDUCIAL" device="-1MM">
+<attribute name="BOM" value="EXCLUDE"/>
+</part>
+<part name="U$5" library="fiducials" deviceset="FIDUCIAL" device="-1MM">
+<attribute name="BOM" value="EXCLUDE"/>
+</part>
+<part name="U$6" library="fiducials" deviceset="FIDUCIAL" device="-1MM">
+<attribute name="BOM" value="EXCLUDE"/>
+</part>
+<part name="U$7" library="fiducials" deviceset="FIDUCIAL" device="-1MM">
+<attribute name="BOM" value="EXCLUDE"/>
+</part>
+<part name="U$8" library="fiducials" deviceset="FIDUCIAL" device="-1MM">
+<attribute name="BOM" value="EXCLUDE"/>
+</part>
+<part name="U$9" library="fiducials" deviceset="FIDUCIAL" device="-1MM">
+<attribute name="BOM" value="EXCLUDE"/>
+</part>
+<part name="U$10" library="fiducials" deviceset="FIDUCIAL" device="-1MM">
+<attribute name="BOM" value="EXCLUDE"/>
+</part>
+<part name="U$11" library="fiducials" deviceset="FIDUCIAL" device="-1MM">
+<attribute name="BOM" value="EXCLUDE"/>
+</part>
+<part name="U$12" library="fiducials" deviceset="FIDUCIAL" device="-1MM">
+<attribute name="BOM" value="EXCLUDE"/>
+</part>
+<part name="U$13" library="fiducials" deviceset="FIDUCIAL" device="-1MM">
+<attribute name="BOM" value="EXCLUDE"/>
+</part>
 </parts>
 <sheets>
@@
 <attribute name="PN" x="90.17" y="27.94" size="1.778" layer="96" display="off"/>
 </instance>
-<instance part="U$1" gate="G$1" x="137.16" y="130.81"/>
-<instance part="U$2" gate="G$1" x="146.05" y="130.81"/>
-<instance part="U$3" gate="G$1" x="154.94" y="130.81"/>
-<instance part="U$4" gate="G$1" x="163.83" y="130.81"/>
-<instance part="U$5" gate="G$1" x="172.72" y="130.81"/>
-<instance part="U$6" gate="G$1" x="181.61" y="130.81"/>
-<instance part="U$7" gate="G$1" x="190.5" y="130.81"/>
-<instance part="U$8" gate="G$1" x="199.39" y="130.81"/>
-<instance part="U$9" gate="G$1" x="208.28" y="130.81"/>
-<instance part="U$10" gate="G$1" x="217.17" y="130.81"/>
-<instance part="U$11" gate="G$1" x="226.06" y="130.81"/>
-<instance part="U$12" gate="G$1" x="234.95" y="130.81"/>
-<instance part="U$13" gate="G$1" x="137.16" y="121.92"/>
+<instance part="U$1" gate="G$1" x="137.16" y="130.81">
+<attribute name="BOM" x="137.16" y="130.81" size="1.778" layer="96" display="off"/>
+</instance>
+<instance part="U$2" gate="G$1" x="146.05" y="130.81">
+<attribute name="BOM" x="146.05" y="130.81" size="1.778" layer="96" display="off"/>
+</instance>
+<instance part="U$3" gate="G$1" x="154.94" y="130.81">
+<attribute name="BOM" x="154.94" y="130.81" size="1.778" layer="96" display="off"/>
+</instance>
+<instance part="U$4" gate="G$1" x="163.83" y="130.81">
+<attribute name="BOM" x="163.83" y="130.81" size="1.778" layer="96" display="off"/>
+</instance>
+<instance part="U$5" gate="G$1" x="172.72" y="130.81">
+<attribute name="BOM" x="172.72" y="130.81" size="1.778" layer="96" display="off"/>
+</instance>
+<instance part="U$6" gate="G$1" x="181.61" y="130.81">
+<attribute name="BOM" x="181.61" y="130.81" size="1.778" layer="96" display="off"/>
+</instance>
+<instance part="U$7" gate="G$1" x="190.5" y="130.81">
+<attribute name="BOM" x="190.5" y="130.81" size="1.778" layer="96" display="off"/>
+</instance>
+<instance part="U$8" gate="G$1" x="199.39" y="130.81">
+<attribute name="BOM" x="199.39" y="130.81" size="1.778" layer="96" display="off"/>
+</instance>
+<instance part="U$9" gate="G$1" x="208.28" y="130.81">
+<attribute name="BOM" x="208.28" y="130.81" size="1.778" layer="96" display="off"/>
+</instance>
+<instance part="U$10" gate="G$1" x="217.17" y="130.81">
+<attribute name="BOM" x="217.17" y="130.81" size="1.778" layer="96" display="off"/>
+</instance>
+<instance part="U$11" gate="G$1" x="226.06" y="130.81">
+<attribute name="BOM" x="226.06" y="130.81" size="1.778" layer="96" display="off"/>
+</instance>
+<instance part="U$12" gate="G$1" x="234.95" y="130.81">
+<attribute name="BOM" x="234.95" y="130.81" size="1.778" layer="96" display="off"/>
+</instance>
+<instance part="U$13" gate="G$1" x="137.16" y="121.92">
+<attribute name="BOM" x="137.16" y="121.92" size="1.778" layer="96" display="off"/>
+</instance>
 </instances>
 <busses>
