File: projects/usb-dac-amplifier-rev-a/smartstand-usb-dac-amplifier-rev-a.sch (EAGLE design)
At the start: 239 parts, among them J1 PJ-002A, J2 292304-1, J3 NRJ6HH, J4 PJRAN2X1U01AUX, J5 T1M-5POS, U1 XUF208-256-TQ64, U10 TPS3702, U11 PCM5102A, U12 SZNUD3124, U13 NJM2068M, U14 NJM4556AM, U15 NJM4556AM, U16 TS5A3159DBV, U17 SN74LVC3G34DCU, U18 TPD2E007DCK, U19 TPD2E007DCK, U2 TPD4E02B04DQA, U3 TPS563200DDC, U4 TPS7A8300RGW, U5 TPS563200DDC, U6 TPS7A8300RGW, U7 TPS7A8300RGW, U8 TPS7A4701RGW, U9 TPS7A3301RGW, X1 24MHz, X2 22.5792MHz, X3 24.576MHz

Commit message: Switch everything to vector fonts and add LEDs for knob illumination.
We added LEDs around the volume control potentiometer so that we could
get an underlighting effect on the volume knob.  The base now has
corresponding holes inside the support structure/cavity that the volume
knob sits around, and since we engineered it so that the knob has a
small gap from the base, the new holes added will allow light to escape
all the way out, and under the volume knob, providing a soft white glow
when powered up.

We also switched all text on the board layout to be vector, to better
represent what the actual board will look like.
Parts:
- added D10, D11, D12, D13, D14, D9: CLM3C, cree:CLM3C
- added R27, R44: 150, passives:RESISTOR-1206
Connections:
- new net N$62: D10.A, D9.C
- new net N$78: D10.C, D11.A
- new net N$80: D11.C, R27.2
- new net N$81: D12.C, D13.A
- new net N$82: D13.C, D14.A
- new net N$83: D14.C, R44.2
- net +12V: now also D12.A, D9.A
- net AGND: now also R27.1, R44.1
Changed lines of the file:
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@@
 <setting verticaltext="up"/>
 </settings>
-<grid distance="0.1" unitdist="inch" unit="inch" style="lines" multiple="1" display="no" altdistance="0.01" altunitdist="inch" altunit="inch"/>
+<grid distance="0.05" unitdist="inch" unit="inch" style="lines" multiple="1" display="no" altdistance="0.01" altunitdist="inch" altunit="inch"/>
 <layers>
 <layer number="1" name="Top" color="4" fill="1" visible="no" active="no"/>
@@
 <attribute name="BOM" value="EXCLUDE"/>
 </part>
+<part name="SHEET13" library="frames" deviceset="A4L-NODOC" device="">
+<attribute name="BOM" value="EXCLUDE"/>
+</part>
+<part name="D9" library="cree" deviceset="CLM3C" device="">
+<attribute name="PN" value="CLM3C-WKW-CWBYA453"/>
+</part>
+<part name="P+17" library="supplies" deviceset="+12V" device=""/>
+<part name="AGND73" library="supplies" deviceset="AGND" device=""/>
+<part name="R27" library="passives" deviceset="RESISTOR" device="-1206" value="150">
+<attribute name="PN" value="RK73H2BTTD1500F"/>
+</part>
+<part name="D10" library="cree" deviceset="CLM3C" device="">
+<attribute name="PN" value="CLM3C-WKW-CWBYA453"/>
+</part>
+<part name="D11" library="cree" deviceset="CLM3C" device="">
+<attribute name="PN" value="CLM3C-WKW-CWBYA453"/>
+</part>
+<part name="D12" library="cree" deviceset="CLM3C" device="">
+<attribute name="PN" value="CLM3C-WKW-CWBYA453"/>
+</part>
+<part name="P+18" library="supplies" deviceset="+12V" device=""/>
+<part name="AGND76" library="supplies" deviceset="AGND" device=""/>
+<part name="R44" library="passives" deviceset="RESISTOR" device="-1206" value="150">
+<attribute name="PN" value="RK73H2BTTD1500F"/>
+</part>
+<part name="D13" library="cree" deviceset="CLM3C" device="">
+<attribute name="PN" value="CLM3C-WKW-CWBYA453"/>
+</part>
+<part name="D14" library="cree" deviceset="CLM3C" device="">
+<attribute name="PN" value="CLM3C-WKW-CWBYA453"/>
+</part>
 </parts>
 <sheets>
@@
 </segment>
 </net>
+</nets>
+</sheet>
+<sheet>
+<plain>
+</plain>
+<instances>
+<instance part="SHEET13" gate="G$1" x="0" y="0">
+<attribute name="BOM" x="0" y="0" size="1.778" layer="96" display="off"/>
+</instance>
+<instance part="D9" gate="G$1" x="106.68" y="127">
+<attribute name="PN" x="106.68" y="127" size="1.778" layer="96" display="off"/>
+</instance>
+<instance part="P+17" gate="1" x="92.71" y="143.51"/>
+<instance part="AGND73" gate="VR1" x="144.78" y="102.87"/>
+<instance part="R27" gate="G$1" x="144.78" y="116.84">
+<attribute name="PN" x="144.78" y="116.84" size="1.778" layer="96" display="off"/>
+</instance>
+<instance part="D10" gate="G$1" x="120.65" y="127">
+<attribute name="PN" x="120.65" y="127" size="1.778" layer="96" display="off"/>
+</instance>
+<instance part="D11" gate="G$1" x="134.62" y="127">
+<attribute name="PN" x="134.62" y="127" size="1.778" layer="96" display="off"/>
+</instance>
+<instance part="D12" gate="G$1" x="106.68" y="78.74">
+<attribute name="PN" x="106.68" y="78.74" size="1.778" layer="96" display="off"/>
+</instance>
+<instance part="P+18" gate="1" x="92.71" y="95.25"/>
+<instance part="AGND76" gate="VR1" x="144.78" y="54.61"/>
+<instance part="R44" gate="G$1" x="144.78" y="68.58">
+<attribute name="PN" x="144.78" y="68.58" size="1.778" layer="96" display="off"/>
+</instance>
+<instance part="D13" gate="G$1" x="120.65" y="78.74">
+<attribute name="PN" x="120.65" y="78.74" size="1.778" layer="96" display="off"/>
+</instance>
+<instance part="D14" gate="G$1" x="134.62" y="78.74">
+<attribute name="PN" x="134.62" y="78.74" size="1.778" layer="96" display="off"/>
+</instance>
+</instances>
+<busses>
+</busses>
+<nets>
+<net name="+12V" class="0">
+<segment>
+<pinref part="D9" gate="G$1" pin="A"/>
+<pinref part="P+17" gate="1" pin="+12V"/>
+<wire x1="102.87" y1="127" x2="92.71" y2="127" width="0.1524" layer="91"/>
+<wire x1="92.71" y1="127" x2="92.71" y2="140.97" width="0.1524" layer="91"/>
+</segment>
+<segment>
+<pinref part="D12" gate="G$1" pin="A"/>
+<pinref part="P+18" gate="1" pin="+12V"/>
+<wire x1="102.87" y1="78.74" x2="92.71" y2="78.74" width="0.1524" layer="91"/>
+<wire x1="92.71" y1="78.74" x2="92.71" y2="92.71" width="0.1524" layer="91"/>
+</segment>
+</net>
+<net name="N$62" class="0">
+<segment>
+<pinref part="D9" gate="G$1" pin="C"/>
+<pinref part="D10" gate="G$1" pin="A"/>
+<wire x1="110.49" y1="127" x2="116.84" y2="127" width="0.1524" layer="91"/>
+</segment>
+</net>
+<net name="N$78" class="0">
+<segment>
+<pinref part="D10" gate="G$1" pin="C"/>
+<pinref part="D11" gate="G$1" pin="A"/>
+<wire x1="124.46" y1="127" x2="130.81" y2="127" width="0.1524" layer="91"/>
+</segment>
+</net>
+<net name="N$80" class="0">
+<segment>
+<pinref part="D11" gate="G$1" pin="C"/>
+<pinref part="R27" gate="G$1" pin="2"/>
+<wire x1="138.43" y1="127" x2="144.78" y2="127" width="0.1524" layer="91"/>
+<wire x1="144.78" y1="127" x2="144.78" y2="121.92" width="0.1524" layer="91"/>
+</segment>
+</net>
+<net name="AGND" class="0">
+<segment>
+<pinref part="AGND73" gate="VR1" pin="AGND"/>
+<pinref part="R27" gate="G$1" pin="1"/>
+<wire x1="144.78" y1="105.41" x2="144.78" y2="111.76" width="0.1524" layer="91"/>
+</segment>
+<segment>
+<pinref part="AGND76" gate="VR1" pin="AGND"/>
+<pinref part="R44" gate="G$1" pin="1"/>
+<wire x1="144.78" y1="57.15" x2="144.78" y2="63.5" width="0.1524" layer="91"/>
+</segment>
+</net>
+<net name="N$81" class="0">
+<segment>
+<pinref part="D12" gate="G$1" pin="C"/>
+<pinref part="D13" gate="G$1" pin="A"/>
+<wire x1="110.49" y1="78.74" x2="116.84" y2="78.74" width="0.1524" layer="91"/>
+</segment>
+</net>
+<net name="N$82" class="0">
+<segment>
+<pinref part="D13" gate="G$1" pin="C"/>
+<pinref part="D14" gate="G$1" pin="A"/>
+<wire x1="124.46" y1="78.74" x2="130.81" y2="78.74" width="0.1524" layer="91"/>
+</segment>
+</net>
+<net name="N$83" class="0">
+<segment>
+<pinref part="D14" gate="G$1" pin="C"/>
+<pinref part="R44" gate="G$1" pin="2"/>
+<wire x1="138.43" y1="78.74" x2="144.78" y2="78.74" width="0.1524" layer="91"/>
+<wire x1="144.78" y1="78.74" x2="144.78" y2="73.66" width="0.1524" layer="91"/>
+</segment>
+</net>
