File: projects/amplifier-rev-a/smartstand-amplifier-rev-a.sch (EAGLE design)
At the start: 86 parts, among them J1 PJ-002A, J2 NRJ6HH, Q1 60V, U1 TPS7A4701RGW, U2 TPS7A4701RGW, U3 TPS7A4701RGW, U4 PCM5102A, U5 TPS7A3301RGW, U6 NJM2068M, U7 NJM4556AM, U8 NJM4556AM

Commit message: Switch over to renamed libraries.
Parts:
- C1, C2: device rcl:CAPACITOR-0603 -> passives:CAPACITOR-0603
- C10, C7, C8, C9: device rcl:CPOL-EUB -> passives:CPOL-EUB
- C11, C12, C19, C20, C23, C27, C29, C3, C30, C33, C34, C37, C38, C39, C4, C40, C5, C6: device rcl:CAPACITOR-0402 -> passives:CAPACITOR-0402
- C13, C14, C15, C16: device rcl:CPOL-EUCHEMICON_F55 -> passives:CPOL-EUCHEMICON_F55
- C17, C18, C21, C22, C24, C25, C26, C28: device rcl:CAPACITOR-0805 -> passives:CAPACITOR-0805
- C31, C32: device rcl:CAPACITOR-HORIZONTAL-0402 -> passives:CAPACITOR-HORIZONTAL-0402
- C35, C36: device rcl:CAPACITOR-HORIZONTAL-0603 -> passives:CAPACITOR-HORIZONTAL-0603
- R1, R11, R12, R15, R16, R2, R24: device rcl:R-US_R0402 -> passives:R-US_R0402
- R10, R13, R14, R21, R22, R25, R3, R4, R5, R6, R7, R8, R9: device rcl:R-US-VERTICALR0402 -> passives:R-US-VERTICALR0402
- R17, R18, R19, R20: device rcl:R-US_R1206 -> passives:R-US_R1206
- R26, R27, R28, R29: device rcl:R-US_R0805 -> passives:R-US_R0805
