File: projects/clock-source-rev-a/smartstand-clock-source-rev-a.sch (EAGLE design)
At the start: 5 parts, among them J1 RECE-20279-001E-01, X1 KC2520K

Commit message: Switch over to renamed libraries.
Parts:
- C1: device rcl:C-EUC0402 -> passives:C-EUC0402
- C2: device rcl:C-EUC0603 -> passives:C-EUC0603
- JP1: device pinhead:PINHD-1X5 -> pin-headers:PINHD-1X5
Changed lines of the file:
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@@
 <parts>
 <part name="U$1" library="frames" deviceset="A4L-NODOC" device=""/>
-<part name="JP1" library="pinhead" deviceset="PINHD-1X5" device="">
+<part name="JP1" library="pin-headers" deviceset="PINHD-1X5" device="">
 <attribute name="PN" value="90120-0125"/>
 </part>
@@
 <attribute name="PN" value="KC3225K24.5760C1GE00"/>
 </part>
-<part name="+3V1" library="supply1" deviceset="+3V3" device=""/>
-<part name="AGND1" library="supply1" deviceset="AGND" device=""/>
-<part name="+3V2" library="supply1" deviceset="+3V3" device=""/>
-<part name="AGND2" library="supply1" deviceset="AGND" device=""/>
-<part name="AGND3" library="supply1" deviceset="AGND" device=""/>
-<part name="+3V3" library="supply1" deviceset="+3V3" device=""/>
-<part name="AGND4" library="supply1" deviceset="AGND" device=""/>
-<part name="C1" library="rcl" deviceset="C-EU" device="C0402" value="100nF">
+<part name="+3V1" library="supplies" deviceset="+3V3" device=""/>
+<part name="AGND1" library="supplies" deviceset="AGND" device=""/>
+<part name="+3V2" library="supplies" deviceset="+3V3" device=""/>
+<part name="AGND2" library="supplies" deviceset="AGND" device=""/>
+<part name="AGND3" library="supplies" deviceset="AGND" device=""/>
+<part name="+3V3" library="supplies" deviceset="+3V3" device=""/>
+<part name="AGND4" library="supplies" deviceset="AGND" device=""/>
+<part name="C1" library="passives" deviceset="C-EU" device="C0402" value="100nF">
 <attribute name="PN" value="GRM155R71C104KA88D"/>
 </part>
-<part name="C2" library="rcl" deviceset="C-EU" device="C0603" value="1uF">
+<part name="C2" library="passives" deviceset="C-EU" device="C0603" value="1uF">
 <attribute name="PN" value="GRM188R61C105KA93D"/>
 </part>
