File: projects/usb-dac-rev-b/smartstand-usb-dac-i2s-rev-b.sch (EAGLE design)
At the start: 69 parts, among them J1 DX4R005H91R1500, J7 RECE-20279-001E-01, U1 TPD4E02B04, U2 XUF208-256-TQ64, U3 LP5912-3.3, U4 LP3879MR-1.0, U5 TPS3702, U6 SN74LVC3G34, X1 24MHz

Commit message: Switch over to renamed libraries.
Parts:
- C1, C10, C11, C12, C13, C14, C15, C16, C17, C18, C19, C20, C21, C22, C23, C28, C30, C6, C7, C8, C9: device rcl:C-EUC0402 -> passives:C-EUC0402
- C2, C24, C3, C4, C5: device rcl:C-EUC0603 -> passives:C-EUC0603
- J2: device pinhead:PINHD-2X10 -> pin-headers:PINHD-2X10
- J3: device pinhead:PINHD-2X3 -> pin-headers:PINHD-2X3
- J4: device pinhead:PINHD-1X4 -> pin-headers:PINHD-1X4
- J5: device pinhead:PINHD-1X7 -> pin-headers:PINHD-1X7
- J6: device pinhead:PINHD-1X5 -> pin-headers:PINHD-1X5
- R1, R2, R3, R7: device rcl:R-US_R0402 -> passives:R-US_R0402
- R10, R11, R12, R13, R14, R4, R5, R6, R8, R9: device rcl:R-US-VERTICALR0402 -> passives:R-US-VERTICALR0402
