File: projects/headphone-detection-rev-a/headphone-detection-rev-a.sch (EAGLE design)
At the start: 9 parts, among them J1 T1M-5POS, U1 VCNL4010

Commit message: Big updates to the headphone detection daughterboard.
In no particular order:

- we're now using the VL6180X (micro LIDAR, basically)
- which needs 2V8 so we have an on-board regulator
- which means we need to interface with 3V3 I2C logic so we
- added level translation FETs for each I2C line
- added test points for the two supply rails
Parts:
- removed C1, C2: 10uF, passives:CAPACITOR-0603
- removed C4: 1uF, passives:CAPACITOR-0402
- added C5, C6: 10uF, passives:CAPACITOR-0603
- added C7: 4.7uF, passives:CAPACITOR-0402
- added R1, R2: 47K, passives:RESISTOR-0402
- added R3, R4, R5, R6: 10K, passives:RESISTOR-0402
- added TP2: TESTPOINT-WITH-GND, test:TESTPOINT-WITH-GND
- added U2: LP5907MFX-2.8, texas-instruments:LP5907MFX-2.8
- added U3, U4: BSS138, on-semiconductor:BSS138LT3G
- C3: value 1uF -> 100nF
- U1: value VCNL4010 -> VL6180XV0NR; device vishay:VCNL4010 -> st-microelectronics:VL6180XV0NR
Connections:
- removed net N$4: J1.4, U1.SCL
- removed net N$6: J1.3, U1.SDA
- new net +2V8: C3.1, C6.1, C7.1, R1.2, R2.2, R3.2, R4.2, TP2.S, U1.AVDD, U1.AVDD_VCSEL, U2.OUT, U3.G, U4.G
- new net LOCAL_SCL: R4.1, U1.SCL, U3.S
- new net LOCAL_SDA: R3.1, U1.SDA, U4.S
- new net N$3: R2.1, U1.GPIO1
- new net N$5: R1.1, U1.GPIO0
- new net SCL: J1.4, R5.1, U3.D
- new net SDA: J1.3, R6.1, U4.D
- net +3V3: now also C5.1, R5.2, R6.2, U2.EN, U2.IN; no longer C1.1, C2.1, C3.1, C4.1, U1.IR_A, U1.VDD
- net AGND: now also C5.2, C6.2, C7.2, TP2.G, U1.AVSS, U1.AVSS_VCSEL, U2.GND; no longer C1.2, C2.2, C4.2, U1.GND
Other:
- moved on the sheet: C3, J1, TP1
