File: projects/headphone-detection-rev-a/smartstand-headphone-detection-rev-a.brd (EAGLE design)
At the start: 22 x 23 mm, 19 parts, among them J1 T1M-5POS, U1 VL6180XV0NR, U2 LP5907MFX-2.8, U3 BSS138, U4 BSS138

Commit message: Adding part numbers to schematic.
Routing:
- net +3V3: track 40.8 -> 41.0 mm, vias 0 -> 1

Commit message: DFM tweaks to the headphone detection daughterboard.
Switched to vector fonts to better repicate what will end up on our
actual boards, and tweaked net label sizes.

Also switched one capacitor to a different package/PN for cost reasons.
Parts:
- removed R2: 47K, passives:R0402
- C7: device passives:C0402 -> passives:C0603
- moved C7 0.81 mm to (13.8, 14.9)
Connections:
- removed net N$3: R2.1, U1.1
- net +2V8: no longer R2.2
Routing:
- net N$3: track 8.34 -> 0.00 mm
- net AGND: track 15.3 -> 17.0 mm
- net +2V8: track 52.7 -> 51.6 mm
- net +3V3: track 41.0 -> 40.9 mm, vias 1 -> 0
