File: projects/headphone-detection-rev-a/smartstand-headphone-detection-rev-a.sch (EAGLE design)
At the start: 19 parts, among them J1 T1M-5POS, U1 VL6180XV0NR, U2 LP5907MFX-2.8, U3 BSS138, U4 BSS138

Commit message: Adding part numbers to schematic.
Parts:
- J1: PN (none) -> T1M-05-T-S-RA-TR
- R1, R2: PN (none) -> RC0402FR-0747KL
- R3, R4, R5, R6: PN (none) -> RC0402FR-0710KL
- U1: PN (none) -> VL6180XV0NR/1
- U3, U4: PN (none) -> BSS138LT3G
Changed lines of the file:
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@@
 <setting verticaltext="up"/>
 </settings>
-<grid distance="0.05" unitdist="inch" unit="inch" style="lines" multiple="1" display="no" altdistance="0.01" altunitdist="inch" altunit="inch"/>
+<grid distance="0.1" unitdist="inch" unit="inch" style="lines" multiple="1" display="no" altdistance="0.01" altunitdist="inch" altunit="inch"/>
 <layers>
 <layer number="1" name="Top" color="4" fill="1" visible="no" active="no"/>
@@
 <attribute name="BOM" value="EXCLUDE"/>
 </part>
-<part name="J1" library="samtec" deviceset="T1M-5POS" device=""/>
+<part name="J1" library="samtec" deviceset="T1M-5POS" device="">
+<attribute name="PN" value="T1M-05-T-S-RA-TR"/>
+</part>
 <part name="+3V1" library="supplies" deviceset="+3V3" device=""/>
 <part name="AGND1" library="supplies" deviceset="AGND" device=""/>
@@
 <part name="AGND8" library="supplies" deviceset="AGND" device=""/>
 <part name="+2V2" library="supplies" deviceset="+2V8" device=""/>
-<part name="U1" library="st-microelectronics" deviceset="VL6180X" device="V0NR"/>
+<part name="U1" library="st-microelectronics" deviceset="VL6180X" device="V0NR">
+<attribute name="PN" value="VL6180XV0NR/1"/>
+</part>
 <part name="+2V3" library="supplies" deviceset="+2V8" device=""/>
 <part name="AGND2" library="supplies" deviceset="AGND" device=""/>
@@
 <attribute name="PN" value="GRM155R60J475ME87D"/>
 </part>
-<part name="R1" library="passives" deviceset="RESISTOR" device="-0402" value="47K"/>
-<part name="R2" library="passives" deviceset="RESISTOR" device="-0402" value="47K"/>
+<part name="R1" library="passives" deviceset="RESISTOR" device="-0402" value="47K">
+<attribute name="PN" value="RC0402FR-0747KL"/>
+</part>
+<part name="R2" library="passives" deviceset="RESISTOR" device="-0402" value="47K">
+<attribute name="PN" value="RC0402FR-0747KL"/>
+</part>
 <part name="+2V5" library="supplies" deviceset="+2V8" device=""/>
 <part name="+2V6" library="supplies" deviceset="+2V8" device=""/>
-<part name="U4" library="on-semiconductor" deviceset="BSS138" device="LT3G" value="BSS138"/>
-<part name="R3" library="passives" deviceset="RESISTOR" device="-0402" value="10K"/>
-<part name="R4" library="passives" deviceset="RESISTOR" device="-0402" value="10K"/>
-<part name="R5" library="passives" deviceset="RESISTOR" device="-0402" value="10K"/>
-<part name="R6" library="passives" deviceset="RESISTOR" device="-0402" value="10K"/>
-<part name="U3" library="on-semiconductor" deviceset="BSS138" device="LT3G" value="BSS138"/>
+<part name="U4" library="on-semiconductor" deviceset="BSS138" device="LT3G" value="BSS138">
+<attribute name="PN" value="BSS138LT3G"/>
+</part>
+<part name="R3" library="passives" deviceset="RESISTOR" device="-0402" value="10K">
+<attribute name="PN" value="RC0402FR-0710KL"/>
+</part>
+<part name="R4" library="passives" deviceset="RESISTOR" device="-0402" value="10K">
+<attribute name="PN" value="RC0402FR-0710KL"/>
+</part>
+<part name="R5" library="passives" deviceset="RESISTOR" device="-0402" value="10K">
+<attribute name="PN" value="RC0402FR-0710KL"/>
+</part>
+<part name="R6" library="passives" deviceset="RESISTOR" device="-0402" value="10K">
+<attribute name="PN" value="RC0402FR-0710KL"/>
+</part>
+<part name="U3" library="on-semiconductor" deviceset="BSS138" device="LT3G" value="BSS138">
+<attribute name="PN" value="BSS138LT3G"/>
+</part>
 <part name="+2V7" library="supplies" deviceset="+2V8" device=""/>
 <part name="+3V2" library="supplies" deviceset="+3V3" device=""/>
@@
 <attribute name="BOM" x="0" y="0" size="1.778" layer="96" display="off"/>
 </instance>
-<instance part="J1" gate="G$1" x="36.83" y="96.52" rot="R180"/>
+<instance part="J1" gate="G$1" x="36.83" y="96.52" rot="R180">
+<attribute name="PN" x="36.83" y="96.52" size="1.778" layer="96" rot="R180" display="off"/>
+</instance>
 <instance part="+3V1" gate="G$1" x="45.72" y="123.19"/>
 <instance part="AGND1" gate="VR1" x="48.26" y="78.74"/>
@@
 <instance part="AGND8" gate="VR1" x="217.17" y="20.32"/>
 <instance part="+2V2" gate="G$1" x="217.17" y="36.83"/>
-<instance part="U1" gate="G$1" x="128.27" y="97.79"/>
+<instance part="U1" gate="G$1" x="128.27" y="97.79">
+<attribute name="PN" x="128.27" y="97.79" size="1.778" layer="96" display="off"/>
+</instance>
 <instance part="+2V3" gate="G$1" x="106.68" y="120.65"/>
 <instance part="AGND2" gate="VR1" x="106.68" y="78.74"/>
@@
 <attribute name="PN" x="180.34" y="105.41" size="1.778" layer="96" display="off"/>
 </instance>
-<instance part="R1" gate="G$1" x="149.86" y="111.76"/>
-<instance part="R2" gate="G$1" x="160.02" y="111.76"/>
+<instance part="R1" gate="G$1" x="149.86" y="111.76">
+<attribute name="PN" x="149.86" y="111.76" size="1.778" layer="96" display="off"/>
+</instance>
+<instance part="R2" gate="G$1" x="160.02" y="111.76">
+<attribute name="PN" x="160.02" y="111.76" size="1.778" layer="96" display="off"/>
+</instance>
 <instance part="+2V5" gate="G$1" x="149.86" y="120.65"/>
 <instance part="+2V6" gate="G$1" x="160.02" y="120.65"/>
-<instance part="U4" gate="G$1" x="156.21" y="21.59" rot="R270"/>
-<instance part="R3" gate="G$1" x="109.22" y="43.18"/>
-<instance part="R4" gate="G$1" x="119.38" y="43.18"/>
-<instance part="R5" gate="G$1" x="173.99" y="43.18"/>
-<instance part="R6" gate="G$1" x="184.15" y="43.18"/>
-<instance part="U3" gate="G$1" x="144.78" y="35.56" rot="R270"/>
+<instance part="U4" gate="G$1" x="156.21" y="21.59" rot="R270">
+<attribute name="PN" x="156.21" y="21.59" size="1.778" layer="96" rot="R270" display="off"/>
+</instance>
+<instance part="R3" gate="G$1" x="109.22" y="43.18">
+<attribute name="PN" x="109.22" y="43.18" size="1.778" layer="96" display="off"/>
+</instance>
+<instance part="R4" gate="G$1" x="119.38" y="43.18">
+<attribute name="PN" x="119.38" y="43.18" size="1.778" layer="96" display="off"/>
+</instance>
+<instance part="R5" gate="G$1" x="173.99" y="43.18">
+<attribute name="PN" x="173.99" y="43.18" size="1.778" layer="96" display="off"/>
+</instance>
+<instance part="R6" gate="G$1" x="184.15" y="43.18">
+<attribute name="PN" x="184.15" y="43.18" size="1.778" layer="96" display="off"/>
+</instance>
+<instance part="U3" gate="G$1" x="144.78" y="35.56" rot="R270">
+<attribute name="PN" x="144.78" y="35.56" size="1.778" layer="96" rot="R270" display="off"/>
+</instance>
 <instance part="+2V7" gate="G$1" x="109.22" y="57.15"/>
 <instance part="+3V2" gate="G$1" x="184.15" y="59.69"/>

Commit message: DFM tweaks to the headphone detection daughterboard.
Switched to vector fonts to better repicate what will end up on our
actual boards, and tweaked net label sizes.

Also switched one capacitor to a different package/PN for cost reasons.
Parts:
- removed R2: 47K, passives:RESISTOR-0402
- C3: PN GRM155R61A105KE15D -> GRM155R71H104KE14D
- C7: device passives:CAPACITOR-0402 -> passives:CAPACITOR-0603; PN GRM155R60J475ME87D -> GRM188R60J475ME19J
Connections:
- removed net N$3: R2.1, U1.GPIO1
- net +2V8: no longer R2.2
Changed lines of the file:
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@@
 <part name="AGND3" library="supplies" deviceset="AGND" device=""/>
 <part name="C3" library="passives" deviceset="CAPACITOR" device="-0402" value="100nF">
-<attribute name="PN" value="GRM155R61A105KE15D"/>
+<attribute name="PN" value="GRM155R71H104KE14D"/>
 </part>
 <part name="U$1" library="fiducials" deviceset="FIDUCIAL" device="-1MM">
@@
 <part name="AGND2" library="supplies" deviceset="AGND" device=""/>
 <part name="+2V4" library="supplies" deviceset="+2V8" device=""/>
-<part name="C7" library="passives" deviceset="CAPACITOR" device="-0402" value="4.7uF">
-<attribute name="PN" value="GRM155R60J475ME87D"/>
+<part name="C7" library="passives" deviceset="CAPACITOR" device="-0603" value="4.7uF">
+<attribute name="PN" value="GRM188R60J475ME19J"/>
 </part>
 <part name="R1" library="passives" deviceset="RESISTOR" device="-0402" value="47K">
 <attribute name="PN" value="RC0402FR-0747KL"/>
 </part>
-<part name="R2" library="passives" deviceset="RESISTOR" device="-0402" value="47K">
-<attribute name="PN" value="RC0402FR-0747KL"/>
-</part>
 <part name="+2V5" library="supplies" deviceset="+2V8" device=""/>
-<part name="+2V6" library="supplies" deviceset="+2V8" device=""/>
 <part name="U4" library="on-semiconductor" deviceset="BSS138" device="LT3G" value="BSS138">
 <attribute name="PN" value="BSS138LT3G"/>
@@
 <attribute name="PN" x="149.86" y="111.76" size="1.778" layer="96" display="off"/>
 </instance>
-<instance part="R2" gate="G$1" x="160.02" y="111.76">
-<attribute name="PN" x="160.02" y="111.76" size="1.778" layer="96" display="off"/>
-</instance>
 <instance part="+2V5" gate="G$1" x="149.86" y="120.65"/>
-<instance part="+2V6" gate="G$1" x="160.02" y="120.65"/>
 <instance part="U4" gate="G$1" x="156.21" y="21.59" rot="R270">
 <attribute name="PN" x="156.21" y="21.59" size="1.778" layer="96" rot="R270" display="off"/>
@@
 <pinref part="+2V5" gate="G$1" pin="+2V8"/>
 <wire x1="149.86" y1="116.84" x2="149.86" y2="120.65" width="0.1524" layer="91"/>
-</segment>
-<segment>
-<pinref part="R2" gate="G$1" pin="2"/>
-<pinref part="+2V6" gate="G$1" pin="+2V8"/>
-<wire x1="160.02" y1="116.84" x2="160.02" y2="120.65" width="0.1524" layer="91"/>
 </segment>
 <segment>
@@
 </segment>
 </net>
-<net name="N$3" class="0">
-<segment>
-<pinref part="U1" gate="G$1" pin="GPIO1"/>
-<pinref part="R2" gate="G$1" pin="1"/>
-<wire x1="144.78" y1="101.6" x2="160.02" y2="101.6" width="0.1524" layer="91"/>
-<wire x1="160.02" y1="101.6" x2="160.02" y2="106.68" width="0.1524" layer="91"/>
-</segment>
-</net>
