File: projects/volume-control-rev-a/volume-control-rev-a.brd (EAGLE design)
At the start: 59.7 x 45.7 mm, 33 parts, among them U1 TPS562200DDC, U2 TLC59116IRHB

Commit message: Lots of updates and tweaks.
This is the locked version for rev A of the volume control board.
Parts:
- L1: value 3.3uH -> 2.2uH
- U1: value TPS562200DDC -> TPS563200DDC
- moved U$4 4.83 mm to (61.0, 41.9)
- moved U$3 4.83 mm to (61.0, 3.81)
- moved JP1 4.83 mm to (62.1, 22.9)
- moved C2 0.92 mm to (49.7, 12.7), turned to 90 degrees
- moved U$2 0.36 mm to (3.81, 41.9)
- moved AGND 0.36 mm to (3.81, 3.81)
Connections:
- net N$1 renamed LEFT_IN
- net N$2 renamed LEFT_OUT
- net N$3 renamed RIGHT_IN
- net N$4 renamed RIGHT_OUT
Routing:
- net +4V0: track 54.4 -> 44.0 mm
- net +3V3: track 27.2 -> 36.8 mm
- net RIGHT_OUT: track 29.0 -> 33.9 mm
- net RIGHT_IN: track 29.5 -> 34.4 mm
- net LEFT_OUT: track 28.5 -> 33.3 mm
- net LEFT_IN: track 29.8 -> 34.7 mm
- net SDA: track 13.0 -> 17.1 mm
- net SCL: track 12.2 -> 16.3 mm
- net N$19: track 12.6 -> 15.5 mm
- net N$13: track 54.7 -> 53.4 mm
- net N$17: track 1.23 -> 0.00 mm, vias 10 -> 11
- net N$12: track 64.1 -> 63.0 mm
- net N$18: track 3.22 -> 2.13 mm
- net N$11: track 76.7 -> 75.8 mm
- net N$7: track 86.5 -> 85.7 mm
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Other:
- board size 59.7 x 45.7 mm -> 64.8 x 45.7 mm
- board text added: "+12V"
- board text added: "+3V3"
- board text added: "GND"
- board text added: "LEFT_IN"
- board text added: "LEFT_OUT"
- board text added: "RIGHT_IN"
- board text added: "RIGHT_OUT"
- board text added: "SCL"
- board text added: "SDA"
