File: projects/volume-control-rev-a/volume-control-rev-a.sch (EAGLE design)
At the start: 32 parts, among them U1 TPS562200DDC, U2 TLC59116IRHB

Commit message: Lots of updates and tweaks.
This is the locked version for rev A of the volume control board.
Parts:
- D1, D10, D11, D12, D2, D3, D4, D5, D6, D7, D8, D9: MPN (none) -> CLM3C-WKW-CXAYA453
- JP1: MPN (none) -> 22-05-3101
- L1: value 3.3uH -> 2.2uH; MPN XFL4020-332MEB -> XFL4020-222MEB
- U1: value TPS562200DDC -> TPS563200DDC; MPN (none) -> TPS563200DDCT
- U2: MPN (none) -> TLC59116IRHB
Connections:
- net N$1 renamed LEFT_IN
- net N$2 renamed LEFT_OUT
- net N$3 renamed RIGHT_IN
- net N$4 renamed RIGHT_OUT
Other:
- note added: "Board Input"
- note added: "LED Control"
- note added: "LED Power Supply"
- note added: "Volume Control"
- moved on the sheet: C4
