File: projects/usb-dac-amplifier-rev-b/smartstand-usb-dac-amplifier-rev-b.brd (EAGLE design)
At the start: 174.7 x 136 mm, 239 parts, among them J1 PJ-002A, J2 292304-1, J3 NRJ6HH, J4 PJRAN2X1U01AUX, J5 T1M-5POS, U1 XUF208-256-TQ64, U10 TPS3702, U11 PCM5102A, U12 SZNUD3124, U13 NJM2068M, U14 NJM4556AM, U15 NJM4556AM, U16 TS5A3159DBV, U17 SN74LVC3G34DCU, U18 TPD2E007DCK, U19 TPD2E007DCK, U2 TPD4E02B04DQA, U3 TPS563200DDC, U4 TPS7A8300RGW, U5 TPS563200DDC, U6 TPS7A8300RGW, U7 TPS7A8300RGW, U8 TPS7A4701RGW, U9 TPS7A3301RGW, X1 24MHz, X2 22.5792MHz, X3 24.576MHz

Commit message: Start shuffling things off into the main section.
Parts:
- moved U12 105.6 mm to (17.1, 60.7)
- moved U$8 99.2 mm to (-7.87, -27.8)
- moved U$6 91.4 mm to (-27.4, -38.9)
- moved R32 75.4 mm to (47.5, 12.8)
- moved R34 75.4 mm to (47.5, 10.3)
- moved JP1 74.9 mm to (53.3, 11.6)
- moved R31 74.3 mm to (59.1, 12.8)
- moved R33 74.3 mm to (59.1, 10.3)
- moved C100 69.3 mm to (41.9, 19.2)
- moved C91 69.3 mm to (54.0, 19.7)
- moved C92 69.3 mm to (48.1, 26.7)
- moved C93 69.3 mm to (40.3, 22.1)
- moved C94 69.3 mm to (44.8, 25.5)
- moved C95 69.3 mm to (54.6, 24.0)
- moved C96 69.3 mm to (53.5, 24.0)
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Routing:
- net N$64: track 175.4 -> 0.00 mm, vias 3 -> 0
- net V-: track 202.0 -> 39.0 mm, vias 6 -> 3
- net LINE_OUT_LEFT: track 151.5 -> 0.00 mm
- net V+: track 181.4 -> 43.3 mm, vias 7 -> 4
- net LINE_OUT_RIGHT: track 132.4 -> 0.00 mm
- net JACK_ENABLE: track 120.1 -> 31.0 mm, vias 4 -> 3
- net N$79: track 82.0 -> 13.4 mm
- net N$47: track 79.6 -> 15.0 mm, vias 3 -> 1
- net ADJUSTED_RIGHT: track 95.6 -> 34.7 mm
- net N$46: track 74.1 -> 15.0 mm, vias 3 -> 1
- net LINE_OUT_SEL: track 170.8 -> 115.1 mm, vias 4 -> 3
- net LINK_UP1: track 74.1 -> 19.2 mm, vias 2 -> 1
- net LINK_DOWN1: track 78.0 -> 23.3 mm
- net N$48: track 65.6 -> 15.0 mm, vias 2 -> 1
- net LINK_UP0: track 68.4 -> 18.7 mm, vias 2 -> 1
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Other:
- board text removed: "3X Gain"
- board text removed: "7X Gain"

Commit message: First rough pass at the slimdown.
I've roughly adjusted the dimensions and shoved everything in there.
The routing isn't half bad, but it's gonna need a lot of tweaks, namely
to get things in a better position, with better trace/space, with
cleaner silkscreen layout.

There's still some angles and airwires and obvious stuff to sort out
but, otherwise, a good first pass.
Parts:
- removed JP1: (no value), pinhead:2X03
- removed R31, R32: 243, 0.1%, rcl:R0402
- moved TP2 122.7 mm to (61.5, 62.4)
- moved U$11 105.1 mm to (-39.0, 45.5)
- moved U$1 93.4 mm to (-61.8, 57.0)
- moved U$10 93.4 mm to (-48.5, 54.1)
- moved U$12 93.4 mm to (-50.8, 56.9)
- moved U$2 93.4 mm to (-55.8, 55.9)
- moved U$6 93.4 mm to (-64.4, 46.9)
- moved U$8 93.4 mm to (-44.8, 57.9)
- moved U$9 93.4 mm to (-53.1, 52.8)
- moved TP9 93.3 mm to (25.1, 36.2), turned to 180 degrees
- moved U$4 60.2 mm to (-45.2, 46.7)
- moved TP10 53.3 mm to (64.8, 36.8), turned to 180 degrees
- moved U12 37.7 mm to (47.4, 38.1), turned to 180 degrees
- moved C112 27.9 mm to (33.8, 37.0), turned to 180 degrees
- moved C103 26.7 mm to (31.1, 65.2), turned to 0 degrees
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Connections:
- removed net N$28: JP1.1, R31.2
- removed net N$30: JP1.5, R33.2
- removed net N$31: JP1.6, R34.1
- removed net N$32: JP1.2, R32.1
- net AGND: now also R33.2, R34.1; no longer JP1.3, JP1.4
- net GAIN_LEFT: no longer R31.1
- net GAIN_RIGHT: no longer R32.2
- net OUT_LEFT: now also R35.2, R37.2; no longer R38.2, R40.2
- net OUT_RIGHT: now also R38.2, R40.2; no longer R35.2, R37.2
Routing:
- net V+: track 43.3 -> 127.5 mm, vias 4 -> 6
- net N$79: track 13.4 -> 94.4 mm
- net LINE_OUT_RIGHT: track 0.00 -> 73.5 mm, vias 0 -> 1
- net LINE_OUT_LEFT: track 0.00 -> 68.4 mm, vias 0 -> 1
- net V-: track 39.0 -> 104.4 mm, vias 3 -> 6
- net I2S_BCLK: track 12.9 -> 61.0 mm
- net I2S_DATA: track 12.3 -> 58.4 mm
- net AVDD: track 131.7 -> 177.3 mm, vias 5 -> 6
- net I2S_LRCLK: track 10.5 -> 54.6 mm
- net I2S_MCLK: track 26.8 -> 69.4 mm
- net N$26: track 57.4 -> 20.4 mm
- net AUDIO_ENABLE: track 34.5 -> 68.8 mm
- net LINE_OUT_SEL: track 115.1 -> 82.9 mm, vias 3 -> 2
- net N$20: track 49.6 -> 25.3 mm
- net JACK_ENABLE: track 31.0 -> 52.4 mm, vias 3 -> 4
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Other:
- board size 174.7 x 136 mm -> 91 x 135.9 mm

Commit message: More fixups and cleaup.
Not too much changed here, but the airwires have been cleaned up.

Still need to make sure that the connector offset from the edge is good,
as well as go through each subsystem and redo functional/design checks.
After that, I think I can properly clean up and tidy up the routing.
Parts:
- removed U$10, U$12, U$4, U$8, U$9: FIDUCIAL-1MM, fiducials:FIDUCIAL_1MM
- moved U$6 153.3 mm to (80.4, -3.56)
- moved U$2 123.4 mm to (57.5, 6.99)
- moved U$11 86.4 mm to (22.5, -15.2)
- moved U$1 77.0 mm to (14.9, 64.3)
Routing:
- net DVDD: track 278.6 -> 301.6 mm
- net AVDD: track 177.3 -> 183.4 mm
- net LINK_UP0: track 37.8 -> 32.7 mm, vias 1 -> 2
- net V-: track 104.4 -> 105.8 mm
- net N$48: vias 2 -> 1

Commit message: Start attributizing things to help develop tooling.
Parts:
- removed JP3: (no value), pin-headers:1X07
- removed R15: 0, rcl:R0402
- removed U$1, U$11, U$13, U$2, U$3, U$5, U$6, U$7: FIDUCIAL-1MM, fiducials:FIDUCIAL_1MM
- added C123: 1uF, passives:C0603
- added C124: 0.1uF, passives:C0402
- added FID1, FID2, FID3, FID4, FID5, FID6: FIDUCIAL_100MIL, MF_Aesthetics:FIDUCIAL_100MIL
- added JP1: (no value), pin-headers:1X10
- added R27: 10K, passives:R0402
- added R31: 18K, passives:R0402
- C10, C23: value 22uF -> 47uF
- C103, C106, C109, C112, C116, C119, C12, C121, C122, C16, C21, C25, C29, C37, C45, C48, C53, C56, C60, C61, C62, C63, C64, C65, C66, C67, C68, C69, C70, C71, C72, C73, C74, C75, C76, C77, C78, C79, C8, C85, C87, C89, C95, C98: value 100nF -> 0.1uF
- C104, C107, C110, C113, C117, C120, C20, C22, C33, C34, C41, C58, C59, C9, C96, C99: value 10nF -> 0.01uF
- C105, C108, C111, C114: value 33pF -> 27pF
- C42, C49, C50, C57: value 100nF -> 0.01uF
- L2: value 1.5uH -> 2.2uH
- R24, R28: value 243, 0.1% -> 270, 1%; device rcl:R0402 -> passives:R0603
- R25, R26, R29, R30: device rcl:R0402 -> passives:R0603
- R3: value 40.2K -> 40.2K, 1%
- R33, R34: value 715, 0.1% -> 1K, 0.1%; device rcl:R0402 -> passives:R0603
- R4, R7: value 10K -> 10K, 1%
- R46: value 10K, 0.1% -> 10K
- R49, R50, R51, R52, R53: value 150 -> 220
- R6: value 8.45K -> 9.53K, 1%
- U3, U5: value TPS563200DDC -> TPS563201DDC
- moved J2 8.89 mm to (89.3, -21.8)
- moved C122 5.43 mm to (19.1, 6.48), turned to 0 degrees
- moved R47 5.32 mm to (19.1, 7.62), turned to 180 degrees
- moved TP4 4.89 mm to (13.6, 1.65), turned to 180 degrees
- moved R25 3.56 mm to (45.6, 13.8)
- moved R29 3.30 mm to (47.0, 25.7)
- moved C73 3.05 mm to (22.0, -2.41)
- moved R45 2.98 mm to (20.7, 7.11), turned to 270 degrees
- moved C93 2.95 mm to (47.4, 27.1)
- moved C91 2.92 mm to (46.2, 15.2)
- moved R24 2.71 mm to (48.1, 14.1)
- moved C74 2.59 mm to (41.4, -6.60)
- moved R28 2.59 mm to (49.4, 26.5)
- moved C7 2.55 mm to (69.6, -28.6)
- moved C32 2.54 mm to (50.4, -39.4)
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Connections:
- removed net N$33: R15.1, X1.P$3
- new net N$231: C123.1, C7.1, J2.P$1, R27.1, R31.2, U2.P$5, U2.P$6
- net +12V: now also JP1.1; no longer JP3.1
- net ADJUSTED_LEFT: now also JP1.6; no longer JP3.6
- net ADJUSTED_RIGHT: now also JP1.5; no longer JP3.5
- net AGND: now also C123.2, C124.2, JP1.2, JP1.7, R31.1; no longer JP3.2, JP3.7
- net CLK: now also X1.P$3; no longer R15.2
- net DVDD: now also JP1.8
- net I2C_SCL: now also JP1.9
- net I2C_SDA: now also JP1.10
- net PREAMP_LEFT: now also JP1.3; no longer JP3.4
- net PREAMP_RIGHT: now also JP1.4; no longer JP3.3
- net USB_VBUS: now also C124.1, R27.2; no longer C7.1, J2.P$1, U2.P$5, U2.P$6
Routing:
- net DVDD: track 301.6 -> 275.7 mm, vias 30 -> 35
- net N$231: track 0.00 -> 22.7 mm
- net USB_VBUS: track 76.2 -> 62.8 mm
- net ADJUSTED_LEFT: track 21.5 -> 28.8 mm
- net AUDIO_ENABLE: track 68.8 -> 63.4 mm
- net JACK_DETECT: track 9.26 -> 14.4 mm, vias 2 -> 0
- net USB_CONNECTED: track 39.4 -> 34.5 mm
- net +1V0: track 113.7 -> 108.8 mm, vias 22 -> 23
- net PREAMP_LEFT: track 69.6 -> 73.6 mm
- net AGND: track 109.6 -> 113.6 mm, vias 146 -> 149
- net PREAMP_RIGHT: track 59.2 -> 63.1 mm
- net LINE_OUT_RIGHT: track 73.5 -> 76.7 mm
- net LINE_OUT_LEFT: track 68.8 -> 72.0 mm
- net N$27: track 25.8 -> 28.4 mm
- net N$29: track 34.4 -> 36.9 mm
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Other:
- board size 91 x 135.9 mm -> 93.3 x 134.6 mm

Commit message: Lots of updates and tweaks.
This is the locked version for rev A of the volume control board.
Connections:
- net I2C_SCL: now also JP1.10; no longer JP1.9
- net I2C_SDA: now also JP1.9; no longer JP1.10
Routing:
- net I2C_SDA: track 35.5 -> 103.0 mm
- net I2C_SCL: track 33.0 -> 98.4 mm
- net DVDD: track 275.7 -> 317.0 mm, vias 35 -> 34
- net I2S_MCLK_SEL: track 33.7 -> 1.85 mm, vias 6 -> 0

Commit message: Lots of cleanup.
Fixing up some incorrect MPNs and package sizes for bulk capacitance, and cleaning up DRC bits.  Also trying to move some bulk capacitance around the board to create a better supply plane.
Parts:
- removed C16, C29: 0.1uF, rcl:C0402
- added D9: 13.6V, diodes:SMA
- C10, C23: device rcl:C1206 -> passives:C1210
- C13, C26: value 47uF -> 22uF; device rcl:C1206 -> passives:C1210
- C14, C27: value 10uF -> 22uF; device rcl:C0805 -> passives:C1210
- moved C6 77.5 mm to (77.5, -6.10)
- moved FID3 23.7 mm to (76.3, -38.0)
- moved FID2 15.9 mm to (75.2, -17.4)
- moved R45 7.11 mm to (27.8, 7.11)
- moved C122 6.10 mm to (25.1, 6.48)
- moved R47 6.10 mm to (25.1, 7.62)
- moved C74 4.44 mm to (37.3, -4.83), flipped to the bottom, turned to 180 degrees
- moved TP10 3.81 mm to (58.4, 36.8)
- moved C76 3.24 mm to (34.0, -9.02), flipped to the bottom
- moved C73 2.92 mm to (24.9, -2.41), flipped to the bottom, turned to 0 degrees
- moved C62 2.84 mm to (37.3, -6.10), flipped to the bottom, turned to 180 degrees
- moved C72 2.62 mm to (34.3, 2.67), flipped to the bottom
- moved C66 2.54 mm to (32.5, 2.67), flipped to the bottom
- moved C67 2.54 mm to (31.4, 2.67), flipped to the bottom
- moved C68 2.54 mm to (30.2, 2.67), flipped to the bottom
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Connections:
- net +1V4: no longer C29.1
- net +4V0: no longer C16.1
- net AGND: now also D9.A; no longer C16.2, C29.2
- net N$8: now also D9.C
Routing:
- net DVDD: track 317.0 -> 284.4 mm, vias 34 -> 33
- net I2S_MCLK_SEL: track 1.85 -> 31.5 mm, vias 0 -> 4
- net AGND: track 113.6 -> 127.1 mm, vias 149 -> 147
- net +1V0: track 108.9 -> 97.7 mm
- net N$79: track 93.1 -> 88.1 mm
- net AUDIO_ENABLE: track 63.4 -> 58.7 mm
- net JACK_DETECT: track 14.4 -> 10.6 mm
- net +12V: track 9.52 -> 13.1 mm, vias 49 -> 47
- net USB_VBUS: track 62.8 -> 59.8 mm
- net V-: track 105.8 -> 108.7 mm
- net I2C_SDA: track 103.0 -> 100.6 mm
- net V+: track 127.6 -> 125.2 mm
- net I2C_SCL: track 98.4 -> 96.1 mm
- net +4V0: track 65.5 -> 63.6 mm, vias 36 -> 37
- net N$231: track 22.7 -> 20.9 mm
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
Commit message: More DFM tune ups.
Just trying to simplify the BOM and make the sourcing easier.
Parts:
- C100, C97: value 33pF -> 27pF
- C17, C18, C19, C30, C31, C32, C35, C38, C39, C40: device rcl:C0805 -> passives:C1206
- moved C30 1.40 mm to (56.4, -39.4)
- moved C40 1.02 mm to (17.3, -28.6)
- moved C31 1.02 mm to (53.7, -39.4)
- moved R5 0.90 mm to (53.7, -31.1)
- moved C39 0.81 mm to (17.3, -31.1)
- moved C22 0.77 mm to (53.7, -33.4)
- moved C18 0.74 mm to (33.5, -31.1)
- moved C19 0.74 mm to (33.5, -28.8)
- moved C32 0.64 mm to (51.1, -39.4)
- moved C38 0.63 mm to (17.3, -33.7)
- moved C35 0.57 mm to (17.3, -36.8)
- moved C36 0.54 mm to (17.1, -39.0)
- moved C37 0.54 mm to (17.1, -40.5)
- moved C17 0.46 mm to (33.5, -33.8)
- moved C27 0.40 mm to (47.4, -39.4)
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Routing:
- net AVDD: track 183.5 -> 182.0 mm
- net +4V0: track 63.6 -> 62.4 mm
- net +1V0: track 97.7 -> 97.1 mm

Commit message: Continuing to optimize the design for DFM.
Parts:
- C21, C8: device rcl:C0805 -> passives:C0603
Changed lines of the file:
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@@
 </element>
 <element name="C1" library="rcl" package="CHEMICON_F55" value="47uF" x="36.83" y="-59.309" smashed="yes" rot="R270">
-<attribute name="MPN" value="EMVA250ADA470MF55G" x="36.83" y="-59.309" size="1.778" layer="27" rot="R270" display="off"/>
 <attribute name="NAME" x="33.147" y="-65.786" size="1.27" layer="25" font="vector" ratio="12"/>
 <attribute name="VALUE" x="40.894" y="-54.483" size="1.27" layer="27" rot="R270"/>
 </element>
 <element name="C2" library="rcl" package="CHEMICON_F55" value="47uF" x="52.578" y="-59.309" smashed="yes" rot="R270">
-<attribute name="MPN" value="EMVA250ADA470MF55G" x="52.578" y="-59.309" size="1.778" layer="27" rot="R270" display="off"/>
 <attribute name="NAME" x="48.895" y="-65.786" size="1.27" layer="25" font="vector" ratio="12"/>
 <attribute name="VALUE" x="56.642" y="-54.483" size="1.27" layer="27" rot="R270"/>
 </element>
 <element name="C3" library="rcl" package="CHEMICON_F55" value="47uF" x="60.452" y="-59.309" smashed="yes" rot="R270">
-<attribute name="MPN" value="EMVA250ADA470MF55G" x="60.452" y="-59.309" size="1.778" layer="27" rot="R270" display="off"/>
 <attribute name="NAME" x="56.769" y="-65.786" size="1.27" layer="25" font="vector" ratio="12"/>
 <attribute name="VALUE" x="64.516" y="-54.483" size="1.27" layer="27" rot="R270"/>
 </element>
 <element name="C4" library="rcl" package="CHEMICON_F55" value="47uF" x="28.956" y="-59.309" smashed="yes" rot="R270">
-<attribute name="MPN" value="EMVA250ADA470MF55G" x="28.956" y="-59.309" size="1.778" layer="27" rot="R270" display="off"/>
 <attribute name="NAME" x="25.273" y="-65.786" size="1.27" layer="25" font="vector" ratio="12"/>
 <attribute name="VALUE" x="33.02" y="-54.483" size="1.27" layer="27" rot="R270"/>
@@
 <element name="C20" library="rcl" package="C0402" value="0.01uF" x="26.67" y="-39.624" smashed="yes" rot="R180">
 <attribute name="NAME" x="25.654" y="-39.37" size="1.27" layer="25" font="vector" ratio="12" rot="R180"/>
-<attribute name="PN" value="GRM15XR71C103KA86D" x="26.67" y="-39.624" size="1.778" layer="27" rot="R180" display="off"/>
 </element>
 <element name="C9" library="rcl" package="C0402" value="0.01uF" x="27.94" y="-30.861" smashed="yes" rot="R180">
 <attribute name="NAME" x="27.432" y="-30.099" size="1.27" layer="25" font="vector" ratio="12"/>
-<attribute name="PN" value="GRM15XR71C103KA86D" x="27.94" y="-30.861" size="1.778" layer="27" rot="R180" display="off"/>
 </element>
 <element name="C45" library="rcl" package="C0402" value="0.1uF" x="71.247" y="6.477" smashed="yes">
@@
 <element name="C7" library="rcl" package="C0603" value="1uF" x="69.596" y="-28.575" smashed="yes" rot="R180">
 <attribute name="NAME" x="67.056" y="-28.067" size="1.27" layer="25" font="vector" ratio="12" rot="R180"/>
-<attribute name="PN" value="GRM188R61E105KA12D" x="69.596" y="-28.575" size="1.778" layer="27" rot="R180" display="off"/>
 </element>
 <element name="C74" library="rcl" package="C0402" value="0.1uF" x="37.338" y="-4.826" smashed="yes" rot="MR180">
@@
 </element>
 <element name="C5" library="rcl" package="CHEMICON_F55" value="47uF" x="44.704" y="-59.309" smashed="yes" rot="R270">
-<attribute name="MPN" value="EMVA250ADA470MF55G" x="44.704" y="-59.309" size="1.778" layer="27" rot="R270" display="off"/>
 <attribute name="NAME" x="41.021" y="-65.786" size="1.27" layer="25" font="vector" ratio="12"/>
 <attribute name="VALUE" x="48.768" y="-54.483" size="1.27" layer="27" rot="R270"/>
 </element>
 <element name="C6" library="rcl" package="CHEMICON_F55" value="47uF" x="77.47" y="-6.096" smashed="yes" rot="R270">
-<attribute name="MPN" value="EMVA250ADA470MF55G" x="77.47" y="-6.096" size="1.778" layer="27" rot="R270" display="off"/>
 <attribute name="NAME" x="73.787" y="-12.573" size="1.27" layer="25" font="vector" ratio="12"/>
 <attribute name="VALUE" x="81.534" y="-1.27" size="1.27" layer="27" rot="R270"/>
@@
 <attribute name="PN" value="GRM188R61E105KA12D" x="27.94" y="-49.276" size="1.778" layer="27" rot="R90" display="off"/>
 </element>
-<element name="C8" library="rcl" package="C0805" value="0.1uF" x="34.544" y="-45.593" smashed="yes" rot="R180">
-<attribute name="MPN" value="C0805C104K5RACTU" x="34.544" y="-45.593" size="1.778" layer="27" rot="R180" display="off"/>
+<element name="C8" library="passives" package="C0603" value="0.1uF" x="34.544" y="-45.593" smashed="yes" rot="R180">
+<attribute name="MPN" value="GCM188R71H104KA57J" x="34.544" y="-45.593" size="1.778" layer="27" rot="R180" display="off"/>
 <attribute name="NAME" x="29.845" y="-46.101" size="1.27" layer="25" font="vector" ratio="12"/>
 </element>
@@
 <element name="C15" library="rcl" package="C0603" value="1uF" x="33.782" y="-39.878" smashed="yes">
 <attribute name="NAME" x="36.449" y="-40.386" size="1.27" layer="25" font="vector" ratio="12"/>
-<attribute name="PN" value="GRM188R61E105KA12D" x="33.782" y="-39.878" size="1.778" layer="27" display="off"/>
 </element>
 <element name="C51" library="rcl" package="C0805" value="10uF" x="71.12" y="22.733" smashed="yes">
@@
 <attribute name="NAME" x="23.749" y="13.335" size="1.27" layer="25" font="vector" ratio="12"/>
 </element>
-<element name="C21" library="rcl" package="C0805" value="0.1uF" x="60.452" y="-45.593" smashed="yes" rot="R180">
-<attribute name="MPN" value="C0805C104K5RACTU" x="60.452" y="-45.593" size="1.778" layer="27" rot="R180" display="off"/>
+<element name="C21" library="passives" package="C0603" value="0.1uF" x="60.452" y="-45.593" smashed="yes" rot="R180">
+<attribute name="MPN" value="GCM188R71H104KA57J" x="60.452" y="-45.593" size="1.778" layer="27" rot="R180" display="off"/>
 <attribute name="NAME" x="54.737" y="-46.736" size="1.27" layer="25" font="vector" ratio="12"/>
 </element>
@@
 <element name="C33" library="rcl" package="C0402" value="0.01uF" x="44.958" y="-32.512" smashed="yes" rot="R90">
 <attribute name="NAME" x="45.466" y="-31.242" size="1.27" layer="25" font="vector" ratio="12" rot="R90"/>
-<attribute name="PN" value="GRM15XR71C103KA86D" x="44.958" y="-32.512" size="1.778" layer="27" rot="R90" display="off"/>
 </element>
 <element name="C27" library="passives" package="C1210" value="22uF" x="47.371" y="-39.37" smashed="yes" rot="R270">
@@
 <element name="C28" library="rcl" package="C0603" value="1uF" x="44.704" y="-39.37" smashed="yes" rot="R270">
 <attribute name="NAME" x="42.164" y="-41.021" size="1.27" layer="25" font="vector" ratio="12" rot="R90"/>
-<attribute name="PN" value="GRM188R61E105KA12D" x="44.704" y="-39.37" size="1.778" layer="27" rot="R270" display="off"/>
 </element>
 <element name="C22" library="rcl" package="C0402" value="0.01uF" x="53.721" y="-33.401" smashed="yes" rot="R90">
 <attribute name="NAME" x="55.753" y="-34.417" size="1.27" layer="25" font="vector" ratio="12" rot="R90"/>
-<attribute name="PN" value="GRM15XR71C103KA86D" x="53.721" y="-33.401" size="1.778" layer="27" rot="R90" display="off"/>
 </element>
 <element name="C30" library="passives" package="C1206" value="10uF" x="56.388" y="-39.37" smashed="yes" rot="R270">
@@
 <element name="C123" library="passives" package="C0603" value="1uF" x="69.596" y="-26.797" smashed="yes" rot="R180">
 <attribute name="NAME" x="67.056" y="-26.289" size="1.27" layer="25" font="vector" ratio="12" rot="R180"/>
-<attribute name="PN" value="GRM188R61E105KA12D" x="69.596" y="-26.797" size="1.778" layer="27" rot="R180" display="off"/>
 <attribute name="VALUE" x="71.374" y="-27.813" size="1.27" layer="27" rot="R180"/>
 </element>
@@
 <contactref element="C8" pad="1"/>
 <contactref element="U3" pad="6"/>
-<wire x1="35.444" y1="-45.593" x2="35.444" y2="-46.852" width="0.254" layer="1"/>
+<wire x1="35.344" y1="-45.593" x2="35.444" y2="-46.852" width="0.254" layer="1"/>
 <wire x1="35.444" y1="-46.852" x2="35.132" y2="-47.164" width="0.254" layer="1"/>
 <wire x1="35.132" y1="-48.072" x2="35.132" y2="-47.164" width="0.254" layer="1"/>
@@
 <wire x1="61.04" y1="-47.164" x2="61.341" y2="-46.863" width="0.254" layer="1"/>
 <wire x1="61.341" y1="-46.863" x2="61.341" y2="-45.604" width="0.254" layer="1"/>
-<wire x1="61.341" y1="-45.604" x2="61.352" y2="-45.593" width="0.254" layer="1"/>
+<wire x1="61.341" y1="-45.604" x2="61.252" y2="-45.593" width="0.254" layer="1"/>
 </signal>
 <signal name="N$56">
@@
 <wire x1="49.149" y1="-21.209" x2="42.291" y2="-21.209" width="0.4064" layer="16"/>
 <polygon width="0.254" layer="15" thermals="no">
-<vertex x="33.401" y="1.016"/>
-<vertex x="32.131" y="-0.254"/>
-<vertex x="30.861" y="-0.254"/>
-<vertex x="30.607" y="0"/>
-<vertex x="30.48" y="0.127"/>
-<vertex x="30.099" y="0.508"/>
+<vertex x="33.274" y="1.016"/>
+<vertex x="31.877" y="-0.381"/>
+<vertex x="30.861" y="-0.381"/>
+<vertex x="30.48" y="0"/>
+<vertex x="30.353" y="0.127"/>
+<vertex x="29.972" y="0.508"/>
 <vertex x="28.702" y="0.508"/>
 <vertex x="28.657178125" y="0.552825"/>
@@
 <wire x1="34.437" y1="-4.806" x2="34.417" y2="-4.826" width="0.2794" layer="1"/>
 <via x="34.417" y="-4.826" extent="1-16" drill="0.3048"/>
-<polygon width="0.2794" layer="1">
-<vertex x="33.2232" y="-7.1628"/>
-<vertex x="34.6075" y="-5.7785"/>
+<polygon width="0.127" layer="1">
+<vertex x="33.2867" y="-7.2263"/>
+<vertex x="34.671" y="-5.842"/>
 <vertex x="35.179" y="-6.35"/>
 <vertex x="35.179" y="-6.985"/>
@@
 <vertex x="33.6804" y="-7.62"/>
 </polygon>
-<polygon width="0.2794" layer="1">
-<vertex x="33.274" y="-7.239"/>
-<vertex x="34.671" y="-5.842"/>
-<vertex x="35.56" y="-6.731"/>
-<vertex x="35.56" y="-7.493"/>
-<vertex x="35.052" y="-8.001"/>
-<vertex x="34.036" y="-8.001"/>
+<polygon width="0.127" layer="1">
+<vertex x="33.147" y="-7.112"/>
+<vertex x="34.6075" y="-5.6515"/>
+<vertex x="35.56" y="-6.604"/>
+<vertex x="35.56" y="-7.62"/>
+<vertex x="35.052" y="-8.128"/>
+<vertex x="34.163" y="-8.128"/>
 </polygon>
 <via x="34.1122" y="-6.604" extent="1-16" drill="0.3048"/>
