File: projects/usb-dac-amplifier-rev-b/smartstand-usb-dac-amplifier-rev-b.brd (EAGLE design)
At the start: 93.3 x 134.6 mm, 231 parts, among them J1 PJ-002A, J2 292304-1, J3 NRJ6HH, J4 PJRAN2X1U01AUX, J5 T1M-5POS, U1 XUF208-256-TQ64, U10 TPS3702, U11 PCM5102A, U12 SZNUD3124, U13 NJM2068M, U14 NJM4556AM, U15 NJM4556AM, U16 TS5A3159DBV, U17 SN74LVC3G34DCU, U18 TPD2E007DCK, U19 TPD2E007DCK, U2 TPD4E02B04DQA, U3 TPS563201DDC, U4 TPS7A8300RGW, U5 TPS563201DDC, U6 TPS7A8300RGW, U7 TPS7A8300RGW, U8 TPS7A4701RGW, U9 TPS7A3301RGW, X1 24MHz, X2 22.5792MHz, X3 24.576MHz

Commit message: start switching over to simplified bypassing
Parts:
- removed C17, C18, C30, C31: 10uF, passives:C1206
- C10, C23: value 47uF -> 10uF; device passives:C1210 -> passives:C0603
- C11, C24: value 1uF -> 10uF
- C13, C14, C26, C27: device passives:C1210 -> passives:C0603
- C15, C28: value 1uF -> 22uF
- C19, C32: value 10uF -> 22uF; device passives:C1206 -> passives:C0603
- moved C19 5.11 mm to (33.0, -33.9)
- moved C15 1.59 mm to (33.0, -38.5)
- moved C12 0.85 mm to (29.2, -48.6)
- moved C11 0.81 mm to (27.4, -48.6)
- moved C13 0.64 mm to (25.4, -43.7)
- moved C14 0.57 mm to (33.0, -36.7)
- moved C10 0.52 mm to (25.3, -48.6)
Connections:
- net +1V0: no longer C30.1, C31.1
- net AGND: no longer C17.2, C18.2, C30.2, C31.2
- net DVDD: no longer C17.1, C18.1
Routing:
- net DVDD: track 284.5 -> 279.2 mm, vias 33 -> 34
- net PG_DVDD: track 30.7 -> 29.1 mm
- net +4V0: track 62.4 -> 63.1 mm, vias 37 -> 33
- net AGND: vias 147 -> 146
- net +12V: vias 47 -> 48

Commit message: More BOM tweaking.
We had some caps that were not sized properly for their expected voltages, so we've fixed that up, and we've added MPNs where necessary.
Parts:
- removed C23: 10uF, passives:C0603
- removed C24: 10uF, rcl:C0603
- removed C35, C38, C39: 10uF, passives:C1206
- removed C36: 1uF, rcl:C0603
- removed C37: 0.1uF, rcl:C0402
- removed R5, R8: 10K, rcl:R0402
- added C16: 22uF, passives:C0805
- C10: value 10uF -> 22uF; device passives:C0603 -> passives:C1812
- C11: value 10uF -> 22uF; device rcl:C0603 -> passives:C1812
- C13, C14: device passives:C0603 -> passives:C0805
- C15: device rcl:C0603 -> passives:C0805
- C40: value 10uF -> 22uF; device passives:C1206 -> passives:C0603
- moved C10 26.6 mm to (51.8, -50.0)
- moved C40 5.58 mm to (16.1, -34.0)
- moved C11 2.07 mm to (25.9, -50.0)
- moved C28 1.83 mm to (46.2, -38.4)
- moved C27 1.20 mm to (48.0, -38.4)
- moved C32 1.14 mm to (50.5, -38.4)
- moved C26 1.05 mm to (51.2, -43.9)
- moved C25 0.92 mm to (55.0, -48.6)
- moved C19 0.52 mm to (32.5, -34.0)
- moved C34 0.52 mm to (11.0, -31.0)
- moved C15 0.36 mm to (32.8, -38.7)
- moved C14 0.28 mm to (32.8, -36.6)
- moved C13 0.25 mm to (25.4, -43.9)
- moved C12 0.13 mm to (29.1, -48.6)
- moved C9 0.13 mm to (27.9, -31.0)
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Connections:
- removed net PG_1V0: R5.2, U6.P$4
- removed net PG_AVDD: R8.2, U7.P$4
- net +12V: no longer C23.1, C24.1
- net +1V0: no longer R5.1
- net +4V0: now also C16.1; no longer C35.1, C36.1, C37.1
- net AGND: now also C16.2; no longer C23.2, C24.2, C35.2, C36.2, C37.2, C38.2, C39.2
- net AVDD: no longer C38.1, C39.1, R8.1
Routing:
- net +1V4: track 19.9 -> 31.4 mm
- net DVDD: track 279.2 -> 289.2 mm, vias 34 -> 33
- net AVDD: track 182.0 -> 175.2 mm
- net +1V0: track 97.1 -> 91.8 mm
- net AGND: track 126.9 -> 123.1 mm, vias 146 -> 168
- net PG_1V0: track 3.06 -> 0.00 mm
- net PG_AVDD: track 2.85 -> 0.00 mm
- net +4V0: track 63.1 -> 63.2 mm, vias 33 -> 29
- net +12V: vias 48 -> 69

Commit message: Cleaning up some of the power circuitry.
A lot of generic cleanup here:
- capacitor availability is painful, so reworking that
- no need to use the smallest via possible when fewer bigger ones will do
- use ranks to better allow flood pours to coexist
Parts:
- added C17, C18: 10uF, passives:C0603
- C10, C11: value 22uF -> 10uF; device passives:C1812 -> passives:C0603
- C13, C14, C15, C16: device passives:C0805 -> passives:C0603
- C43, C46, C51, C54: value 10uF -> 22uF; device rcl:C0805 -> passives:C0603
- moved C10 1.44 mm to (50.8, -49.0)
- moved C11 1.44 mm to (24.9, -49.0)
- moved R3 0.76 mm to (34.5, -42.9)
- moved R6 0.76 mm to (60.5, -42.9)
- moved R4 0.64 mm to (34.5, -44.1)
- moved R7 0.64 mm to (60.5, -44.1)
- moved C25 0.40 mm to (54.9, -49.0)
- moved C12 0.40 mm to (29.0, -49.0)
- moved C15 0.40 mm to (32.6, -38.4)
- moved C16 0.28 mm to (16.3, -36.6)
- moved C19 0.13 mm to (32.6, -34.0)
- moved C40 0.13 mm to (16.3, -34.0)
- moved C14 0.13 mm to (32.6, -36.6)
Connections:
- net +12V: now also C17.1, C18.1
- net AGND: now also C17.2, C18.2
Routing:
- net +1V4: track 31.4 -> 17.3 mm, vias 9 -> 2
- net AGND: track 123.1 -> 115.5 mm, vias 168 -> 169
- net +4V0: track 63.2 -> 62.4 mm, vias 29 -> 28
- net N$53: track 10.4 -> 9.56 mm
- net +1V0: vias 23 -> 20
- net +12V: vias 69 -> 71
