File: projects/usb-dac-amplifier-rev-b/smartstand-usb-dac-amplifier-rev-b.sch (EAGLE design)
At the start: 239 parts, among them J1 PJ-002A, J2 292304-1, J3 NRJ6HH, J4 PJRAN2X1U01AUX, J5 T1M-5POS, U1 XUF208-256-TQ64, U10 TPS3702, U11 PCM5102A, U12 SZNUD3124, U13 NJM2068M, U14 NJM4556AM, U15 NJM4556AM, U16 TS5A3159DBV, U17 SN74LVC3G34DCU, U18 TPD2E007DCK, U19 TPD2E007DCK, U2 TPD4E02B04DQA, U3 TPS563200DDC, U4 TPS7A8300RGW, U5 TPS563200DDC, U6 TPS7A8300RGW, U7 TPS7A8300RGW, U8 TPS7A4701RGW, U9 TPS7A3301RGW, X1 24MHz, X2 22.5792MHz, X3 24.576MHz

Commit message: First rough pass at the slimdown.
I've roughly adjusted the dimensions and shoved everything in there.
The routing isn't half bad, but it's gonna need a lot of tweaks, namely
to get things in a better position, with better trace/space, with
cleaner silkscreen layout.

There's still some angles and airwires and obvious stuff to sort out
but, otherwise, a good first pass.
Parts:
- removed JP1: (no value), pin-headers:PINHD-2X3
- removed R31, R32: 243, 0.1%, passives:RESISTOR-HORIZONTAL-0402
Connections:
- removed net N$28: JP1.1, R31.2
- removed net N$30: JP1.5, R33.2
- removed net N$31: JP1.6, R34.1
- removed net N$32: JP1.2, R32.1
- net AGND: now also R33.2, R34.1; no longer JP1.3, JP1.4
- net GAIN_LEFT: no longer R31.1
- net GAIN_RIGHT: no longer R32.2
- net OUT_LEFT: now also R35.2, R37.2; no longer R38.2, R40.2
- net OUT_RIGHT: now also R38.2, R40.2; no longer R35.2, R37.2
Other:
- moved on the sheet: R33, R34
Changed lines of the file:
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@@
 <attribute name="PN" value="ERA-2AEB7150X"/>
 </part>
-<part name="R32" library="passives" deviceset="RESISTOR-HORIZONTAL" device="-0402" value="243, 0.1%">
-<attribute name="PN" value="ERA-2AEB2430X"/>
-</part>
 <part name="R34" library="passives" deviceset="RESISTOR-HORIZONTAL" device="-0402" value="715, 0.1%">
 <attribute name="PN" value="ERA-2AEB7150X"/>
 </part>
-<part name="R31" library="passives" deviceset="RESISTOR-HORIZONTAL" device="-0402" value="243, 0.1%">
-<attribute name="PN" value="ERA-2AEB2430X"/>
-</part>
 <part name="AGND35" library="supplies" deviceset="AGND" device=""/>
 <part name="J3" library="neutrik" deviceset="NRJ6HH" device="">
@@
 <attribute name="PN" value="T1M-05-T-S-RA-TR"/>
 </part>
-<part name="JP1" library="pin-headers" deviceset="PINHD-2X3" device="">
-<attribute name="PN" value="961206-6404-AR"/>
-</part>
 <part name="C76" library="passives" deviceset="CAPACITOR" device="-0402" value="100nF">
 <attribute name="PN" value="GRM155R71H104KE14D"/>
@@
 <attribute name="PN" x="71.12" y="82.55" size="1.778" layer="96" display="off"/>
 </instance>
-<instance part="R33" gate="G$1" x="50.8" y="31.75">
-<attribute name="PN" x="50.8" y="31.75" size="1.778" layer="96" display="off"/>
-</instance>
-<instance part="R32" gate="G$1" x="93.98" y="41.91">
-<attribute name="PN" x="93.98" y="41.91" size="1.778" layer="96" display="off"/>
-</instance>
-<instance part="R34" gate="G$1" x="93.98" y="31.75">
-<attribute name="PN" x="93.98" y="31.75" size="1.778" layer="96" display="off"/>
+<instance part="R33" gate="G$1" x="50.8" y="45.72">
+<attribute name="PN" x="50.8" y="45.72" size="1.778" layer="96" display="off"/>
 </instance>
-<instance part="R31" gate="G$1" x="50.8" y="41.91">
-<attribute name="PN" x="50.8" y="41.91" size="1.778" layer="96" display="off"/>
+<instance part="R34" gate="G$1" x="73.66" y="45.72">
+<attribute name="PN" x="73.66" y="45.72" size="1.778" layer="96" display="off"/>
 </instance>
-<instance part="AGND35" gate="VR1" x="72.39" y="20.32"/>
+<instance part="AGND35" gate="VR1" x="62.23" y="34.29"/>
 <instance part="C99" gate="G$1" x="219.71" y="33.02">
 <attribute name="PN" x="219.71" y="33.02" size="1.778" layer="96" display="off"/>
@@
 <attribute name="PN" x="233.68" y="33.02" size="1.778" layer="96" display="off"/>
 </instance>
-<instance part="JP1" gate="A" x="71.12" y="36.83">
-<attribute name="PN" x="71.12" y="36.83" size="1.778" layer="96" display="off"/>
-</instance>
 </instances>
 <busses>
@@
 </segment>
 <segment>
-<pinref part="JP1" gate="A" pin="3"/>
-<wire x1="68.58" y1="36.83" x2="62.23" y2="36.83" width="0.1524" layer="91"/>
-<wire x1="62.23" y1="36.83" x2="62.23" y2="26.67" width="0.1524" layer="91"/>
 <pinref part="AGND35" gate="VR1" pin="AGND"/>
-<wire x1="62.23" y1="26.67" x2="72.39" y2="26.67" width="0.1524" layer="91"/>
-<wire x1="72.39" y1="26.67" x2="72.39" y2="22.86" width="0.1524" layer="91"/>
-<pinref part="JP1" gate="A" pin="4"/>
-<wire x1="76.2" y1="36.83" x2="82.55" y2="36.83" width="0.1524" layer="91"/>
-<wire x1="82.55" y1="36.83" x2="82.55" y2="26.67" width="0.1524" layer="91"/>
-<wire x1="82.55" y1="26.67" x2="72.39" y2="26.67" width="0.1524" layer="91"/>
-<junction x="72.39" y="26.67"/>
+<pinref part="R33" gate="G$1" pin="2"/>
+<wire x1="55.88" y1="45.72" x2="62.23" y2="45.72" width="0.1524" layer="91"/>
+<wire x1="62.23" y1="45.72" x2="62.23" y2="36.83" width="0.1524" layer="91"/>
+<pinref part="R34" gate="G$1" pin="1"/>
+<wire x1="68.58" y1="45.72" x2="62.23" y2="45.72" width="0.1524" layer="91"/>
+<junction x="62.23" y="45.72"/>
 </segment>
 </net>
@@
 </segment>
 <segment>
-<wire x1="45.72" y1="41.91" x2="43.18" y2="41.91" width="0.1524" layer="91"/>
-<label x="39.37" y="41.91" size="2.54" layer="95" rot="R180" xref="yes"/>
-<pinref part="R31" gate="G$1" pin="1"/>
+<label x="39.37" y="45.72" size="2.54" layer="95" rot="R180" xref="yes"/>
 <pinref part="R33" gate="G$1" pin="1"/>
-<wire x1="43.18" y1="41.91" x2="39.37" y2="41.91" width="0.1524" layer="91"/>
-<wire x1="45.72" y1="31.75" x2="43.18" y2="31.75" width="0.1524" layer="91"/>
-<wire x1="43.18" y1="31.75" x2="43.18" y2="41.91" width="0.1524" layer="91"/>
-<junction x="43.18" y="41.91"/>
+<wire x1="45.72" y1="45.72" x2="39.37" y2="45.72" width="0.1524" layer="91"/>
 </segment>
 </net>
@@
 </segment>
 <segment>
-<wire x1="99.06" y1="41.91" x2="101.6" y2="41.91" width="0.1524" layer="91"/>
-<label x="105.41" y="41.91" size="2.54" layer="95" xref="yes"/>
-<pinref part="R32" gate="G$1" pin="2"/>
+<label x="85.09" y="45.72" size="2.54" layer="95" xref="yes"/>
 <pinref part="R34" gate="G$1" pin="2"/>
-<wire x1="101.6" y1="41.91" x2="105.41" y2="41.91" width="0.1524" layer="91"/>
-<wire x1="99.06" y1="31.75" x2="101.6" y2="31.75" width="0.1524" layer="91"/>
-<wire x1="101.6" y1="31.75" x2="101.6" y2="41.91" width="0.1524" layer="91"/>
-<junction x="101.6" y="41.91"/>
+<wire x1="78.74" y1="45.72" x2="85.09" y2="45.72" width="0.1524" layer="91"/>
 </segment>
 </net>
@@
 </segment>
 </net>
-<net name="N$28" class="0">
-<segment>
-<pinref part="JP1" gate="A" pin="1"/>
-<wire x1="68.58" y1="39.37" x2="58.42" y2="39.37" width="0.1524" layer="91"/>
-<wire x1="58.42" y1="39.37" x2="58.42" y2="41.91" width="0.1524" layer="91"/>
-<pinref part="R31" gate="G$1" pin="2"/>
-<wire x1="58.42" y1="41.91" x2="55.88" y2="41.91" width="0.1524" layer="91"/>
-</segment>
-</net>
-<net name="N$30" class="0">
-<segment>
-<pinref part="JP1" gate="A" pin="5"/>
-<wire x1="68.58" y1="34.29" x2="58.42" y2="34.29" width="0.1524" layer="91"/>
-<wire x1="58.42" y1="34.29" x2="58.42" y2="31.75" width="0.1524" layer="91"/>
-<pinref part="R33" gate="G$1" pin="2"/>
-<wire x1="58.42" y1="31.75" x2="55.88" y2="31.75" width="0.1524" layer="91"/>
-</segment>
-</net>
-<net name="N$31" class="0">
-<segment>
-<pinref part="JP1" gate="A" pin="6"/>
-<wire x1="76.2" y1="34.29" x2="86.36" y2="34.29" width="0.1524" layer="91"/>
-<wire x1="86.36" y1="34.29" x2="86.36" y2="31.75" width="0.1524" layer="91"/>
-<pinref part="R34" gate="G$1" pin="1"/>
-<wire x1="86.36" y1="31.75" x2="88.9" y2="31.75" width="0.1524" layer="91"/>
-</segment>
-</net>
-<net name="N$32" class="0">
-<segment>
-<pinref part="JP1" gate="A" pin="2"/>
-<wire x1="76.2" y1="39.37" x2="86.36" y2="39.37" width="0.1524" layer="91"/>
-<wire x1="86.36" y1="39.37" x2="86.36" y2="41.91" width="0.1524" layer="91"/>
-<pinref part="R32" gate="G$1" pin="1"/>
-<wire x1="86.36" y1="41.91" x2="88.9" y2="41.91" width="0.1524" layer="91"/>
-</segment>
-</net>
 </nets>
 </sheet>
@@
 </segment>
 </net>
-<net name="OUT_RIGHT" class="0">
-<segment>
-<pinref part="R35" gate="G$1" pin="2"/>
-<wire x1="193.04" y1="128.27" x2="196.85" y2="128.27" width="0.1524" layer="91"/>
-<wire x1="196.85" y1="128.27" x2="196.85" y2="118.11" width="0.1524" layer="91"/>
-<pinref part="R37" gate="G$1" pin="2"/>
-<wire x1="196.85" y1="118.11" x2="196.85" y2="107.95" width="0.1524" layer="91"/>
-<wire x1="196.85" y1="107.95" x2="193.04" y2="107.95" width="0.1524" layer="91"/>
-<wire x1="196.85" y1="118.11" x2="204.47" y2="118.11" width="0.1524" layer="91"/>
-<junction x="196.85" y="118.11"/>
-<label x="204.47" y="118.11" size="2.54" layer="95" xref="yes"/>
-</segment>
-</net>
 <net name="V+" class="0">
 <segment>
@@
 </segment>
 </net>
+<net name="OUT_LEFT" class="0">
+<segment>
+<pinref part="R35" gate="G$1" pin="2"/>
+<wire x1="193.04" y1="128.27" x2="196.85" y2="128.27" width="0.1524" layer="91"/>
+<wire x1="196.85" y1="128.27" x2="196.85" y2="118.11" width="0.1524" layer="91"/>
+<pinref part="R37" gate="G$1" pin="2"/>
+<wire x1="196.85" y1="118.11" x2="196.85" y2="107.95" width="0.1524" layer="91"/>
+<wire x1="196.85" y1="107.95" x2="193.04" y2="107.95" width="0.1524" layer="91"/>
+<wire x1="196.85" y1="118.11" x2="204.47" y2="118.11" width="0.1524" layer="91"/>
+<junction x="196.85" y="118.11"/>
+<label x="204.47" y="118.11" size="2.54" layer="95" xref="yes"/>
+</segment>
+</net>
 <net name="ADJUSTED_RIGHT" class="0">
 <segment>
@@
 </segment>
 </net>
-<net name="OUT_LEFT" class="0">
+<net name="OUT_RIGHT" class="0">
 <segment>
 <pinref part="R38" gate="G$1" pin="2"/>
@@
 </segment>
 </net>
-<net name="ADJUSTED_RIGHT" class="0">
-<segment>
-<pinref part="JP3" gate="A" pin="5"/>
-<wire x1="109.22" y1="22.86" x2="83.82" y2="22.86" width="0.1524" layer="91"/>
-<wire x1="83.82" y1="22.86" x2="83.82" y2="21.59" width="0.1524" layer="91"/>
-<wire x1="83.82" y1="21.59" x2="73.66" y2="21.59" width="0.1524" layer="91"/>
-<label x="73.66" y="21.59" size="3.302" layer="95" rot="R180" xref="yes"/>
-</segment>
-</net>
 <net name="PREAMP_LEFT" class="0">
 <segment>
@@
 </segment>
 </net>
+<net name="ADJUSTED_RIGHT" class="0">
+<segment>
+<pinref part="JP3" gate="A" pin="5"/>
+<wire x1="109.22" y1="22.86" x2="83.82" y2="22.86" width="0.1524" layer="91"/>
+<wire x1="83.82" y1="22.86" x2="83.82" y2="21.59" width="0.1524" layer="91"/>
+<wire x1="83.82" y1="21.59" x2="73.66" y2="21.59" width="0.1524" layer="91"/>
+<label x="73.66" y="21.59" size="3.302" layer="95" rot="R180" xref="yes"/>
+</segment>
+</net>

Commit message: More fixups and cleaup.
Not too much changed here, but the airwires have been cleaned up.

Still need to make sure that the connector offset from the edge is good,
as well as go through each subsystem and redo functional/design checks.
After that, I think I can properly clean up and tidy up the routing.
Parts:
- removed U$10, U$12, U$4, U$8, U$9: FIDUCIAL-1MM, fiducials:FIDUCIAL-1MM
Other:
- note added: "Audio Clock Generation"
- note added: "We use a separate gain stage, from the output stage, following the Objective2 design. We've chosen to implement a 2X gain mode. We also route to line out before the gain stage, to allow line-level outputs."
- note added: "We're generating dual clocks to support 44.1-kHz and 48-kHz based sampling rates. We toggle which one is output with a simple analog switch."
- note removed: "We use a separate gain stage, from the output stage, following the Objective2 design. We've chosen to implement a 2X and 4X gain mode. We also route to line out before the gain stage, to allow line-level outputs."
- moved on the sheet: C91, C92, C93, C94, R24, R25, R26, R28, R29, R30, R33, R34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

Commit message: Start attributizing things to help develop tooling.
Parts:
- removed JP3: (no value), pin-headers:PINHD-1X7
- removed R15: 0, passives:RESISTOR-HORIZONTAL-0402
- removed U$1, U$11, U$13, U$2, U$3, U$5, U$6, U$7: FIDUCIAL-1MM, fiducials:FIDUCIAL-1MM
- added C123: 1uF, passives:CAPACITOR-0603
- added C124: 0.1uF, passives:CAPACITOR-0402
- added FID1, FID2, FID3, FID4, FID5, FID6: FIDUCIAL_100MIL, MF_Aesthetics:FIDUCIAL_100MIL
- added JP1: (no value), pin-headers:PINHD-1X10
- added R27: 10K, passives:RESISTOR-HORIZONTAL-0402
- added R31: 18K, passives:RESISTOR-0402
- C1, C13, C2, C26, C3, C4, C5, C6: MPN (none) -> EMVA250ADA470MF55G; PN EMVA250ADA470MF55G -> (none)
- C10, C23: value 22uF -> 47uF; MPN (none) -> EMVA250ADA470MF55G; PN 12063D226KAT2A -> (none)
- C100, C97: MPN (none) -> GRM1555C1H330JA01D; PN GRM1555C1H330JA01D -> (none)
- C101, C102: MPN (none) -> RSBCC4220Z310K; PN RSBCC4220Z310K -> (none)
- C103, C106, C109, C112, C116, C119, C12, C121, C122, C16, C25, C29, C37, C45, C48, C53, C56, C60, C61, C62, C63, C64, C65, C66, C67, C68, C69, C70, C71, C72, C73, C74, C75, C76, C77, C78, C79, C85, C87, C89, C95, C98: value 100nF -> 0.1uF
- C104, C107, C110, C113, C117, C120, C20, C22, C33, C34, C41, C58, C59, C9, C96, C99: value 10nF -> 0.01uF
- C105, C108, C111, C114: value 33pF -> 27pF; PN GRM1555C1H330JA01D -> (none)
- C14, C17, C18, C19, C27, C30, C31, C32, C35, C38, C39, C40, C43, C46, C51, C54, C80, C86, C88, C90: MPN (none) -> GRM21BR61E106KA73L; PN GRM21BR61E106KA73L -> (none)
- C21, C8: value 100nF -> 0.1uF; MPN (none) -> C0805C104K5RACTU; PN C0805C104K5RACTU -> (none)
- C42, C49, C50, C57: value 100nF -> 0.01uF; PN GRM155R71H104KE14D -> GRM15XR71C103KA86D
- C81, C82: MPN (none) -> GRM188R61C225KE15D; PN GRM188R61C225KE15D -> (none)
- C83, C84: MPN (none) -> C0402C222J3GACTU; PN C0402C222J3GACTU -> (none)
- C91, C92, C93, C94: MPN (none) -> GRM1555C1H221JA01J; PN GRM1555C1H221JA01J -> (none)
- D1: MPN (none) -> PMEG3050BEP,115; PN PMEG3050BEP,115 -> (none); TYPE (none) -> diode; VF (none) -> 0.45
- D2: MPN (none) -> P4SMA16CA; PN P4SMA16CA -> (none)
- D3, D4, D5, D6, D7, D8: MPN (none) -> 598-8070-107F; PN 598-8070-107F -> (none)
- F1: IMAX (none) -> 0.6; MPN (none) -> 2920L030DR; PN 2920L030DR -> (none); TYPE (none) -> fuse; VMAX (none) -> 60
- J1: CURRENT (none) -> 2.0; MPN (none) -> PJ-002A; PN PJ-002A -> (none); TYPE (none) -> pwrsource; VOLTAGE (none) -> 12.0
- J2: MPN (none) -> 292304-1; PN 292304-1 -> (none)
- J3: MPN (none) -> NRJ6HH; PN NRJ6HH -> (none)
- J4: MPN (none) -> PJRAN2X1U01AUX; PN PJRAN2X1U01AUX -> (none)
- J5: MPN (none) -> T1M-05-T-S-RA-TR; PN T1M-05-T-S-RA-TR -> (none)
- JP2: MPN (none) -> N2520-5002RB; PN N2520-5002RB -> (none)
- L1: MPN (none) -> VLP8040T-2R2N; PN VLP8040T-2R2N -> (none)
- L2: value 1.5uH -> 2.2uH; MPN (none) -> VLP8040T-2R2N; PN VLP8040T-1R5N -> (none)
- R1: MPN (none) -> RK73B1ETTP430J; PN RK73B1ETTP430J -> (none)
- R10: MPN (none) -> RC0402FR-079K76L; PN RC0402FR-079K76L -> (none)
- R11: MPN (none) -> RK73H1ETTP1154F; PN RK73H1ETTP1154F -> (none)
- R12: MPN (none) -> RC0402FR-07137KL; PN RC0402FR-07137KL -> (none)
- R14: MPN (none) -> RCS04024R70JNED; PN SG73P1ETTP4R7J -> (none)
- R19, R20: MPN (none) -> RK73B1ETTP330J; PN RK73B1ETTP330J -> (none)
- R2, R5: MPN (none) -> RC0402FR-0710KL; PN RC0402FR-0710KL -> (none)
- R22, R23: MPN (none) -> RG1005P-471-B-T5; PN RG1005P-471-B-T5 -> (none)
- R24, R28: value 243, 0.1% -> 270, 1%; device passives:RESISTOR-HORIZONTAL-0402 -> passives:RESISTOR-HORIZONTAL-0603; MPN (none) -> MCT06030C2700FP500; PN ERA-2AEB2430X -> (none)
- R25, R29: device passives:RESISTOR-0402 -> passives:RESISTOR-0603; MPN (none) -> MCT06030C1002FP500; PN ERA-2AEB103X -> (none)
- R26, R30: device passives:RESISTOR-HORIZONTAL-0402 -> passives:RESISTOR-HORIZONTAL-0603; MPN (none) -> MCT06030C1501FP500; PN RG1005P-152-B-T5 -> (none)
- R3: value 40.2K -> 40.2K, 1%; MPN (none) -> RK73H1ETTP4022F; PN RK73H1ETTP4022F -> (none)
- R33, R34: value 715, 0.1% -> 1K, 0.1%; device passives:RESISTOR-HORIZONTAL-0402 -> passives:RESISTOR-HORIZONTAL-0603; MPN (none) -> MCT06030C1001FP500; PN ERA-2AEB7150X -> (none)
- R35, R37, R38, R40: MPN (none) -> MCA12060C1008FP500; PN MCA12060C1008FP500 -> (none)
- R36, R39: MPN (none) -> RG1005P-4022-B-T5; PN RG1005P-4022-B-T5 -> (none)
- R4, R7: value 10K -> 10K, 1%; MPN (none) -> RC0402FR-0710KL; PN RC0402FR-0710KL -> (none)
- R46: value 10K, 0.1% -> 10K
- R47: MPN (none) -> RC0402FR-0749K9L; PN RC0402FR-0749K9L -> (none)
- R49, R50, R51, R52, R53: value 150 -> 220; PN SG73P1ETTP151J -> (none)
- R6: value 8.45K -> 9.53K, 1%; MPN (none) -> RC0402FR-079K53L; PN RC0402FR-078K45L -> (none)
- R9: MPN (none) -> RK73H1ETTP6652F; PN RK73H1ETTP6652F -> (none)
- RL1, RL2: MPN (none) -> TQ2-12V; PN TQ2-12V -> (none)
- U1: PN XUF208-256-TQ64-C10 -> (none)
- U10: MPN (none) -> TPS3702CX10DDCT; PN TPS3702CX10DDCT -> (none)
- U11: MPN (none) -> PCM5102APWR; PN PCM5102APWR -> (none)
- U12: MPN (none) -> SZNUD3124DMT1G; PN SZNUD3124DMT1G -> (none)
- U13: MPN (none) -> NJM2068M-TE1; PN NJM2068M-TE1 -> (none)
- U14, U15: MPN (none) -> NJM4556AM-TE1; PN NJM4556AM-TE1 -> (none)
- U16: MPN (none) -> TS5A3159DBVR; PN TS5A3159DBVR -> (none)
- U17: MPN (none) -> SN74LVC3G34DCUT; PN SN74LVC3G34DCUT -> (none)
- U18, U19: MPN (none) -> TPD2E007DCKR; PN TPD2E007DCKR -> (none)
- U2: MPN (none) -> TPD4E02B04DQAR; PN TPD4E02B04DQAR -> (none)
- U3: value TPS563200DDC -> TPS563201DDC; MPN (none) -> TPS5632001DCR; PN TPS563200DDCR -> (none); TYPE (none) -> switcher
- U4: MPN (none) -> TPS7A8300RGWR; PN TPS7A8300RGWR -> (none); TYPE (none) -> linear
- U5: value TPS563200DDC -> TPS563201DDC; MPN (none) -> TPS563201DDCR; PN TPS563200DDCR -> (none)
- U6, U7: MPN (none) -> TPS7A8300RGWR; PN TPS7A8300RGWR -> (none)
- U8: MPN (none) -> TPS7A4701RGWR; PN TPS7A4701RGWR -> (none)
- U9: MPN (none) -> TPS7A3301RGWR; PN TPS7A3301RGWR -> (none)
- X1: MPN (none) -> KC2520C24.0000C2LE00; PN KC2520C24.0000C2LE00 -> (none)
- X2: MPN (none) -> KC2520K22.5792C1GE00; PN KC2520K22.5792C1GE00 -> (none)
- X3: MPN (none) -> KC2520K24.5760C1GE00; PN KC2520K24.5760C1GE00 -> (none)
Connections:
- removed net N$33: R15.1, X1.CLK
- new net N$231: C123.1, C7.1, J2.VBUS, R27.1, R31.2, U2.IO4
- net +12V: now also JP1.1; no longer JP3.1
- net ADJUSTED_LEFT: now also JP1.6; no longer JP3.6
- net ADJUSTED_RIGHT: now also JP1.5; no longer JP3.5
- net AGND: now also C123.2, C124.2, JP1.2, JP1.7, R31.1; no longer JP3.2, JP3.7
- net CLK: now also X1.CLK; no longer R15.2
- net DVDD: now also JP1.8
- net I2C_SCL: now also JP1.9
- net I2C_SDA: now also JP1.10
- net PREAMP_LEFT: now also JP1.3; no longer JP3.4
- net PREAMP_RIGHT: now also JP1.4; no longer JP3.3
- net USB_VBUS: now also C124.1, R27.2; no longer C7.1, J2.VBUS, U2.IO4

Commit message: Lots of updates and tweaks.
This is the locked version for rev A of the volume control board.
Connections:
- net I2C_SCL: now also JP1.10; no longer JP1.9
- net I2C_SDA: now also JP1.9; no longer JP1.10

Commit message: Lots of cleanup.
Fixing up some incorrect MPNs and package sizes for bulk capacitance, and cleaning up DRC bits.  Also trying to move some bulk capacitance around the board to create a better supply plane.
Parts:
- removed C16, C29: 0.1uF, passives:CAPACITOR-0402
- added D9: 13.6V, diodes:SUPPRESSOR-DUAL-SMA
- C10, C23: device passives:CAPACITOR-1206 -> passives:CAPACITOR-1210
- C13, C26: value 47uF -> 22uF; device passives:CAPACITOR-1206 -> passives:CAPACITOR-1210; MPN EMVA250ADA470MF55G -> GCM32ER71A226ME12L
- C14, C27: value 10uF -> 22uF; device passives:CAPACITOR-0805 -> passives:CAPACITOR-1210; MPN GRM21BR61E106KA73L -> GCM32ER71A226ME12L
- U3: MPN TPS5632001DCR -> TPS563201DDC
- U5: MPN TPS563201DDCR -> TPS563201DDC
Connections:
- net +1V4: no longer C29.1
- net +4V0: no longer C16.1
- net AGND: now also D9.A; no longer C16.2, C29.2
- net N$8: now also D9.C
Other:
- moved on the sheet: D1, F1

Commit message: More DFM tune ups.
Just trying to simplify the BOM and make the sourcing easier.
Parts:
- C100, C97: value 33pF -> 27pF
- C17, C18, C19, C30, C31, C32, C35, C38, C39, C40: device passives:CAPACITOR-0805 -> passives:CAPACITOR-1206
Changed lines of the file:
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@@
 <attribute name="MPN" value="RC0402FR-0710KL"/>
 </part>
-<part name="C30" library="passives" deviceset="CAPACITOR" device="-0805" value="10uF">
-<attribute name="MPN" value="GRM21BR61E106KA73L"/>
-</part>
-<part name="C31" library="passives" deviceset="CAPACITOR" device="-0805" value="10uF">
-<attribute name="MPN" value="GRM21BR61E106KA73L"/>
-</part>
-<part name="C32" library="passives" deviceset="CAPACITOR" device="-0805" value="10uF">
+<part name="C30" library="passives" deviceset="CAPACITOR" device="-1206" value="10uF">
+<attribute name="MPN" value="GRM21BR61E106KA73L"/>
+</part>
+<part name="C31" library="passives" deviceset="CAPACITOR" device="-1206" value="10uF">
+<attribute name="MPN" value="GRM21BR61E106KA73L"/>
+</part>
+<part name="C32" library="passives" deviceset="CAPACITOR" device="-1206" value="10uF">
 <attribute name="MPN" value="GRM21BR61E106KA73L"/>
 </part>
@@
 <attribute name="MPN" value="RC0402FR-0710KL"/>
 </part>
-<part name="C17" library="passives" deviceset="CAPACITOR" device="-0805" value="10uF">
-<attribute name="MPN" value="GRM21BR61E106KA73L"/>
-</part>
-<part name="C18" library="passives" deviceset="CAPACITOR" device="-0805" value="10uF">
-<attribute name="MPN" value="GRM21BR61E106KA73L"/>
-</part>
-<part name="C19" library="passives" deviceset="CAPACITOR" device="-0805" value="10uF">
+<part name="C17" library="passives" deviceset="CAPACITOR" device="-1206" value="10uF">
+<attribute name="MPN" value="GRM21BR61E106KA73L"/>
+</part>
+<part name="C18" library="passives" deviceset="CAPACITOR" device="-1206" value="10uF">
+<attribute name="MPN" value="GRM21BR61E106KA73L"/>
+</part>
+<part name="C19" library="passives" deviceset="CAPACITOR" device="-1206" value="10uF">
 <attribute name="MPN" value="GRM21BR61E106KA73L"/>
 </part>
 <part name="AGND15" library="supplies" deviceset="AGND" device=""/>
 <part name="+4V03" library="supplies" deviceset="+4V0" device=""/>
-<part name="C35" library="passives" deviceset="CAPACITOR" device="-0805" value="10uF">
+<part name="C35" library="passives" deviceset="CAPACITOR" device="-1206" value="10uF">
 <attribute name="MPN" value="GRM21BR61E106KA73L"/>
 </part>
@@
 <attribute name="PN" value="RC0402FR-0710KL"/>
 </part>
-<part name="C38" library="passives" deviceset="CAPACITOR" device="-0805" value="10uF">
-<attribute name="MPN" value="GRM21BR61E106KA73L"/>
-</part>
-<part name="C39" library="passives" deviceset="CAPACITOR" device="-0805" value="10uF">
-<attribute name="MPN" value="GRM21BR61E106KA73L"/>
-</part>
-<part name="C40" library="passives" deviceset="CAPACITOR" device="-0805" value="10uF">
+<part name="C38" library="passives" deviceset="CAPACITOR" device="-1206" value="10uF">
+<attribute name="MPN" value="GRM21BR61E106KA73L"/>
+</part>
+<part name="C39" library="passives" deviceset="CAPACITOR" device="-1206" value="10uF">
+<attribute name="MPN" value="GRM21BR61E106KA73L"/>
+</part>
+<part name="C40" library="passives" deviceset="CAPACITOR" device="-1206" value="10uF">
 <attribute name="MPN" value="GRM21BR61E106KA73L"/>
 </part>
@@
 <attribute name="PN" value="GRM155R71H104KE14D"/>
 </part>
-<part name="C97" library="passives" deviceset="CAPACITOR" device="-0402" value="33pF">
+<part name="C97" library="passives" deviceset="CAPACITOR" device="-0402" value="27pF">
 <attribute name="MPN" value="GRM1555C1H330JA01D"/>
 </part>
@@
 <attribute name="PN" value="GRM155R71H104KE14D"/>
 </part>
-<part name="C100" library="passives" deviceset="CAPACITOR" device="-0402" value="33pF">
+<part name="C100" library="passives" deviceset="CAPACITOR" device="-0402" value="27pF">
 <attribute name="MPN" value="GRM1555C1H330JA01D"/>
 </part>

Commit message: Continuing to optimize the design for DFM.
Parts:
- C1, C2, C3, C4, C5, C6: MPN EMVA250ADA470MF55G -> (none)
- C123, C15, C28, C7: PN GRM188R61E105KA12D -> (none)
- C20, C22, C33, C9: PN GRM15XR71C103KA86D -> (none)
- C21, C8: device passives:CAPACITOR-HORIZONTAL-0805 -> passives:CAPACITOR-HORIZONTAL-0603; MPN C0805C104K5RACTU -> GCM188R71H104KA57J
