File: projects/usb-dac-amplifier-rev-b/smartstand-usb-dac-amplifier-rev-b.sch (EAGLE design)
At the start: 231 parts, among them J1 PJ-002A, J2 292304-1, J3 NRJ6HH, J4 PJRAN2X1U01AUX, J5 T1M-5POS, U1 XUF208-256-TQ64, U10 TPS3702, U11 PCM5102A, U12 SZNUD3124, U13 NJM2068M, U14 NJM4556AM, U15 NJM4556AM, U16 TS5A3159DBV, U17 SN74LVC3G34DCU, U18 TPD2E007DCK, U19 TPD2E007DCK, U2 TPD4E02B04DQA, U3 TPS563201DDC, U4 TPS7A8300RGW, U5 TPS563201DDC, U6 TPS7A8300RGW, U7 TPS7A8300RGW, U8 TPS7A4701RGW, U9 TPS7A3301RGW, X1 24MHz, X2 22.5792MHz, X3 24.576MHz

Commit message: start switching over to simplified bypassing
Parts:
- removed C17, C18, C30, C31: 10uF, passives:CAPACITOR-1206
- C10, C23: value 47uF -> 10uF; device passives:CAPACITOR-1210 -> passives:CAPACITOR-0603; MPN EMVA250ADA470MF55G -> ZRB18AR61E106ME01L
- C11, C24: value 1uF -> 10uF; MPN (none) -> ZRB18AR61E106ME01L; PN GRM188R61E105KA12D -> (none)
- C13, C14, C26, C27: device passives:CAPACITOR-1210 -> passives:CAPACITOR-0603; MPN GCM32ER71A226ME12L -> ZRB18AR61A226ME01L
- C15, C28: value 1uF -> 22uF; MPN (none) -> ZRB18AR61A226ME01L
- C19, C32: value 10uF -> 22uF; device passives:CAPACITOR-1206 -> passives:CAPACITOR-0603; MPN GRM21BR61E106KA73L -> ZRB18AR61A226ME01L
Connections:
- net +1V0: no longer C30.1, C31.1
- net AGND: no longer C17.2, C18.2, C30.2, C31.2
- net DVDD: no longer C17.1, C18.1
Other:
- moved on the sheet: C12, C13, C14, C15, C19, C20, C21, C22, C25, C26, C27, C28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
