File: projects/usb-dac-amplifier-rev-b/smartstand-usb-dac-amplifier-rev-b.sch (EAGLE design)
At the start: 227 parts, among them J1 PJ-002A, J2 292304-1, J3 NRJ6HH, J4 PJRAN2X1U01AUX, J5 T1M-5POS, U1 XUF208-256-TQ64, U10 TPS3702, U11 PCM5102A, U12 SZNUD3124, U13 NJM2068M, U14 NJM4556AM, U15 NJM4556AM, U16 TS5A3159DBV, U17 SN74LVC3G34DCU, U18 TPD2E007DCK, U19 TPD2E007DCK, U2 TPD4E02B04DQA, U3 TPS563201DDC, U4 TPS7A8300RGW, U5 TPS563201DDC, U6 TPS7A8300RGW, U7 TPS7A8300RGW, U8 TPS7A4701RGW, U9 TPS7A3301RGW, X1 24MHz, X2 22.5792MHz, X3 24.576MHz

Commit message: More BOM tweaking.
We had some caps that were not sized properly for their expected voltages, so we've fixed that up, and we've added MPNs where necessary.
Parts:
- removed C23, C24: 10uF, passives:CAPACITOR-0603
- removed C35, C38, C39: 10uF, passives:CAPACITOR-1206
- removed C36: 1uF, passives:CAPACITOR-0603
- removed C37: 0.1uF, passives:CAPACITOR-0402
- removed R5, R8: 10K, passives:RESISTOR-0402
- added C16: 22uF, passives:CAPACITOR-0805
- C10, C11: value 10uF -> 22uF; device passives:CAPACITOR-0603 -> passives:CAPACITOR-1812; MPN ZRB18AR61E106ME01L -> C4532X7R1E226M250KC
- C100, C97: MPN GRM1555C1H330JA01D -> (none)
- C13, C14, C15: device passives:CAPACITOR-0603 -> passives:CAPACITOR-0805; MPN ZRB18AR61A226ME01L -> GRM21BR61A226ME51L
- C40: value 10uF -> 22uF; device passives:CAPACITOR-1206 -> passives:CAPACITOR-0603; MPN GRM21BR61E106KA73L -> ZRB18AR61A226ME01L
Connections:
- removed net PG_1V0: R5.2, U6.PG
- removed net PG_AVDD: R8.2, U7.PG
- net +12V: no longer C23.1, C24.1
- net +1V0: no longer R5.1
- net +4V0: now also C16.1; no longer C35.1, C36.1, C37.1
- net AGND: now also C16.2; no longer C23.2, C24.2, C35.2, C36.2, C37.2, C38.2, C39.2
- net AVDD: no longer C38.1, C39.1, R8.1
Other:
- moved on the sheet: C11, C12, C25, C34, C40, C41, C42, C43, C44, C45, C46, C47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

Commit message: Cleaning up some of the power circuitry.
A lot of generic cleanup here:
- capacitor availability is painful, so reworking that
- no need to use the smallest via possible when fewer bigger ones will do
- use ranks to better allow flood pours to coexist
Parts:
- added C17, C18: 10uF, passives:CAPACITOR-0603
- C10, C11: value 22uF -> 10uF; device passives:CAPACITOR-1812 -> passives:CAPACITOR-0603; MPN C4532X7R1E226M250KC -> GRM188R6YA106MA73D
- C13, C14, C15, C16: device passives:CAPACITOR-0805 -> passives:CAPACITOR-0603; MPN GRM21BR61A226ME51L -> ZRB18AR61A226ME01L
- C43, C46, C51, C54: value 10uF -> 22uF; device passives:CAPACITOR-0805 -> passives:CAPACITOR-0603; MPN GRM21BR61E106KA73L -> GRM188R6YA106MA73D
Connections:
- net +12V: now also C17.1, C18.1
- net AGND: now also C17.2, C18.2
Other:
- moved on the sheet: C12, C16, C25, C40
